File: Audio/AmpModule.kicad_pcb (KiCad board)
At the start: 2 copper layers, 52.5 x 41.5 mm, 26 parts, among them J10 AMP_AUX_IN, J11 AMP_AUX_OUT, J9 AMP_PWR

Commit message: rework pcb
Parts:
- removed C22, C23: 0.1μF, Resistor_SMD:R_0603_1608Metric_Pad0.98x0.95mm_HandSolder
- removed C24: 0.1μF, Capacitor_THT:C_Rect_L7.2mm_W2.5mm_P5.00mm_FKS2_FKP2_MKS2_MKP2
- removed C25: 10μF, Capacitor_THT:CP_Radial_D5.0mm_P2.00mm
- removed H5, H6, H7, H8: MountingHole, MountingHole:MountingHole_3.2mm_M3
- removed R29: 50Ω, Resistor_SMD:R_0603_1608Metric_Pad0.98x0.95mm_HandSolder
- added C30: 0.1μF, Capacitor_THT:C_Rect_L7.2mm_W2.5mm_P5.00mm_FKS2_FKP2_MKS2_MKP2, F.Cu at (40.6, 104.1)
- added C31: 10μF, Capacitor_THT:CP_Radial_D5.0mm_P2.00mm, F.Cu at (40.6, 113.0)
- added C32: 470μF, Capacitor_THT:CP_Radial_D16.0mm_P7.50mm, F.Cu at (91.4, 72.4)
- added C33: 470μF, Capacitor_THT:CP_Radial_D16.0mm_P7.50mm, F.Cu at (91.4, 104.1)
- added H10: MountingHole, MountingHole:MountingHole_3.2mm_M3, F.Cu at (16.5, 128.3)
- added H11: MountingHole, MountingHole:MountingHole_3.2mm_M3, F.Cu at (16.5, 133.3)
- added H12: MountingHole, MountingHole:MountingHole_3.2mm_M3, F.Cu at (16.5, 138.4)
- added H9: MountingHole, MountingHole:MountingHole_3.2mm_M3, F.Cu at (16.5, 123.2)
- added R19: 220KΩ, R_1206_3216Metric_Pad1.30x1.75mm_HandSolder, F.Cu at (39.4, 81.3)
- C26: footprint Capacitor_THT:C_Rect_L7.2mm_W2.5mm_P5.00mm_FKS2_FKP2_MKS2_MKP2 -> C_1206_3216Metric_Pad1.33x1.80mm_HandSolder
- C27: value 10μF -> 0.1μF; footprint Capacitor_THT:CP_Radial_D5.0mm_P2.00mm -> C_1206_3216Metric_Pad1.33x1.80mm_HandSolder
- C28: value 470μF -> 0.1μF; footprint Capacitor_THT:CP_Radial_D16.0mm_P7.50mm -> Capacitor_THT:C_Rect_L7.2mm_W2.5mm_P5.00mm_FKS2_FKP2_MKS2_MKP2
- C29: value 470μF -> 10μF; footprint Capacitor_THT:CP_Radial_D16.0mm_P7.50mm -> Capacitor_THT:CP_Radial_D5.0mm_P2.00mm
- R20, R22, R23, R24, R26: footprint Resistor_SMD:R_0603_1608Metric_Pad0.98x0.95mm_HandSolder -> R_1206_3216Metric_Pad1.30x1.75mm_HandSolder; moved to F.Cu
- R21: value 220KΩ -> 10KΩ; footprint Resistor_SMD:R_0603_1608Metric_Pad0.98x0.95mm_HandSolder -> R_1206_3216Metric_Pad1.30x1.75mm_HandSolder; moved to F.Cu
- R25: value 10KΩ -> 47KΩ; footprint Resistor_SMD:R_0603_1608Metric_Pad0.98x0.95mm_HandSolder -> R_1206_3216Metric_Pad1.30x1.75mm_HandSolder; moved to F.Cu
- R27: value 47KΩ -> 47Ω; footprint Resistor_SMD:R_0603_1608Metric_Pad0.98x0.95mm_HandSolder -> R_1206_3216Metric_Pad1.30x1.75mm_HandSolder; moved to F.Cu
- R28: value 50Ω -> 47Ω; footprint Resistor_SMD:R_0603_1608Metric_Pad0.98x0.95mm_HandSolder -> R_1206_3216Metric_Pad1.30x1.75mm_HandSolder; moved to F.Cu
- moved J9 134.1 mm to (17.8, 35.6), turned to 0 degrees
- moved C26 122.1 mm to (33.0, 24.1), turned to 0 degrees
- moved C29 117.1 mm to (40.6, 69.8)
- moved C27 110.4 mm to (33.0, 48.3), turned to 0 degrees
- moved AMP1 107.3 mm to (40.6, 35.6)
- moved J10 92.6 mm to (26.7, 85.1), turned to 0 degrees
- moved R23 91.2 mm to (54.6, 59.7), turned to 180 degrees
- moved R22 87.6 mm to (53.3, 116.8), turned to 180 degrees
- moved C28 84.3 mm to (40.6, 61.0)
- moved R24 80.6 mm to (54.6, 99.1), turned to 90 degrees
- moved R20 78.0 mm to (39.4, 92.7), turned to 90 degrees
- moved R26 75.7 mm to (67.3, 99.1)
- moved R25 74.7 mm to (67.3, 82.5), turned to 90 degrees
- moved R21 72.9 mm to (53.3, 74.9), turned to 90 degrees
- moved R27 68.0 mm to (82.5, 72.4)
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Connections:
- C26 pad 1: Net-(AMP1B-+) -> (no net)
- C26 pad 2: /Rotary_L_OUT -> (no net)
- C27 pad 1: Net-(AMP1B-+) -> (no net)
- C27 pad 2: /Rotary_L_OUT -> (no net)
- C28 pad 1: Net-(C28-Pad1) -> Net-(AMP1A-+)
- C28 pad 2: /AmpModule/R_OUT -> /Rotary_R_OUT
- C29 pad 1: Net-(C29-Pad1) -> Net-(AMP1A-+)
- C29 pad 2: /AmpModule/L_OUT -> /Rotary_R_OUT
- J11 pad 1: /AmpModule/L_OUT -> /Rotary_R_OUT
- J11 pad 2: /AmpModule/R_OUT -> /Rotary_L_OUT
- R20 pad 1: /Rotary_R_OUT -> (no net)
- R20 pad 2: GND -> (no net)
- R21 pad 1: /Rotary_L_OUT -> (no net)
- R21 pad 2: GND -> (no net)
- R22 pad 1: GND -> (no net)
- R22 pad 2: Net-(AMP1A--) -> (no net)
- R23 pad 1: GND -> (no net)
- R23 pad 2: Net-(AMP1B-+) -> (no net)
- R24 pad 1: Net-(AMP1A-+) -> (no net)
- R24 pad 2: GND -> (no net)
- R25 pad 1: GND -> (no net)
- R25 pad 2: Net-(AMP1B--) -> (no net)
- R26 pad 1: Net-(AMP1A--) -> (no net)
- R26 pad 2: Net-(AMP1-Pad1) -> (no net)
- R27 pad 1: Net-(AMP1B--) -> (no net)
- R27 pad 2: Net-(AMP1-Pad7) -> (no net)
- R28 pad 1: Net-(AMP1-Pad1) -> (no net)
- R28 pad 2: Net-(C28-Pad1) -> (no net)
Routing:
- net /AmpModule/R_OUT: track 31.8 -> 0.00 mm, vias 1 -> 0
- net Net-(AMP1B-+): track 28.8 -> 0.00 mm
- net /Rotary_V-_OUT: track 23.2 -> 0.00 mm
- net /Rotary_L_OUT: track 20.8 -> 0.00 mm
- net /AmpModule/L_OUT: track 20.7 -> 0.00 mm
- net /Rotary_R_OUT: track 19.5 -> 0.00 mm
- net Net-(AMP1A-+): track 18.0 -> 0.00 mm
- net /Rotary_V+_OUT: track 14.1 -> 0.00 mm
- net Net-(C28-Pad1): track 11.9 -> 0.00 mm
- net Net-(AMP1-Pad1): track 11.2 -> 0.00 mm
- net Net-(AMP1B--): track 7.88 -> 0.00 mm
- net Net-(AMP1A--): track 6.71 -> 0.00 mm
- net Net-(C29-Pad1): track 6.49 -> 0.00 mm
- net Net-(AMP1-Pad7): track 6.00 -> 0.00 mm
- removed copper zone on B.Cu, net GND
