File: Audio/PowerModule.kicad_pcb (KiCad board)
At the start: 2 copper layers, 62 x 37 mm, 15 parts, among them J4 PWR_IN, J5 PWR_OUT

Commit message: rework pcb
Parts:
- removed C1: 47μF, Capacitor_THT:CP_Radial_D8.0mm_P3.50mm
- removed C2, C3: 4.7μF, Capacitor_THT:CP_Radial_D5.0mm_P2.00mm
- removed C4: 0.1μF, Resistor_SMD:R_0603_1608Metric_Pad0.98x0.95mm_HandSolder
- removed F1: 1A, Resistor_THT:R_Axial_DIN0411_L9.9mm_D3.6mm_P12.70mm_Horizontal
- removed U1: ~, Library:MCW03-12D15_SIP7_THT
- added C6: 4.7μF, Capacitor_THT:CP_Radial_D5.0mm_P2.00mm, F.Cu at (99.1, 36.8)
- added C7: 4.7μF, Capacitor_THT:CP_Radial_D5.0mm_P2.00mm, F.Cu at (99.1, 44.5)
- added C8: 0.1μF, C_1206_3216Metric_Pad1.33x1.80mm_HandSolder, F.Cu at (110.5, 36.8)
- added C9: 0.1μF, C_1206_3216Metric_Pad1.33x1.80mm_HandSolder, F.Cu at (110.5, 44.5)
- added F2: 1A, Resistor_THT:R_Axial_DIN0411_L9.9mm_D3.6mm_P12.70mm_Horizontal, F.Cu at (39.4, 44.5)
- added U2: , Library:MCW03-12D15_SIP7_THT, F.Cu at (64.8, 31.8)
- C5: value 0.1μF -> 47μF; footprint Resistor_SMD:R_0603_1608Metric_Pad0.98x0.95mm_HandSolder -> Capacitor_THT:CP_Radial_D8.0mm_P3.50mm
- moved H3 170.8 mm to (15.2, 68.6)
- moved H2 162.5 mm to (15.2, 63.5)
- moved C5 145.7 mm to (45.7, 40.6), turned to 0 degrees
- moved J4 121.9 mm to (27.9, 36.8)
- moved H4 119.9 mm to (15.2, 73.7)
- moved H1 112.7 mm to (15.2, 58.4)
- moved L1 109.0 mm to (83.8, 38.1), turned to -90 degrees
- moved L2 105.9 mm to (83.8, 43.2), turned to 90 degrees
- moved J5 84.5 mm to (133.3, 40.6), turned to 0 degrees
Connections:
- C5 pad 1: GND -> Net-(U1-+Vin)
- C5 pad 2: /Rotary_V-_IN -> /PowerModule/PD_GND_IN
- J5 pad 1: /Rotary_V+_IN -> /Rotary_V+_OUT
- J5 pad 3: /Rotary_V-_IN -> /Rotary_V-_OUT
- L1 pad 1: /Rotary_V+_IN -> Net-(U1--Vout)
- L1 pad 2: Net-(U1-+Vout) -> /Rotary_V-_IN
Routing:
- net /PowerModule/PD_GND_IN: track 39.3 -> 0.00 mm
- net Net-(U1-+Vin): track 36.8 -> 0.00 mm
- net /Rotary_V-_IN: track 29.6 -> 0.00 mm
- net /Rotary_V+_IN: track 28.9 -> 0.00 mm
- net Net-(U1-+Vout): track 15.4 -> 0.00 mm
- net Net-(U1--Vout): track 9.98 -> 0.00 mm
- net /PowerModule/+15_IN: track 6.61 -> 0.00 mm
- net GND: track 4.10 -> 0.00 mm, vias 2 -> 0
- removed copper zone on B.Cu, net GND
