File: Audio/AudioCase.kicad_pcb (KiCad board)
At the start: 2 copper layers, 262.1 x 203.6 mm, 126 parts, among them J10 AMP_AUX_IN, J11 AMP_AUX_OUT, J12 AMP1_PWR, J13 PD_IN, J14 AUDIO_IN, J15 AMP1_LR, J16 AMP2_PWR, J17 AMP2_LR, J18 AMP3_PWR, J19 AMP4_PWR, J20 AMP5_PWR, J21 AMP3_LR, J22 AMP4_LR, J23 AMP5_LR, J24 OLED_PIN, J4 PWR_IN, J5 PWR_OUT, J6 AUX_IN, J7 V_IN, J8 AUX_OUT, J9 AMP_PWR, K1 AZ850P2-x, K10 AZ850P2-x, K2 AZ850P2-x, K3 AZ850P2-x, K4 AZ850P2-x, K5 AZ850P2-x, K6 AZ850P2-x, K7 AZ850P2-x, K8 AZ850P2-x, K9 AZ850P2-x, SW1 RotaryEncoder_Switch, U1 MCW03, U2 NJM4558, U3 NJM4558, U4 BP5293-50, U5 ULN2803A, U6 ULN2803A, U7 ULN2803A

Commit message: step1
Parts:
- moved NT1 110.7 mm to (160.7, 211.8), turned to 180 degrees
- moved J13 106.9 mm to (169.0, 211.8), turned to 90 degrees
- moved F2 85.4 mm to (168.9, 201.0), turned to 90 degrees
- moved C31 72.8 mm to (163.2, 199.4)
- moved C30 71.5 mm to (163.7, 190.4)
- moved U4 50.1 mm to (163.0, 182.1), turned to 180 degrees
- moved C33 41.9 mm to (157.8, 170.5)
- moved C32 37.8 mm to (157.8, 163.3), turned to 180 degrees
- moved J24 29.2 mm to (115.9, 214.6)
- moved SW1 23.1 mm to (88.7, 210.8)
- moved J14 19.1 mm to (34.4, 104.9), turned to 180 degrees
- moved U6 16.7 mm to (83.2, 173.9), turned to -90 degrees
- moved U5 15.6 mm to (115.4, 174.1)
- moved J8 15.0 mm to (145.1, 22.1)
- moved U7 11.6 mm to (48.8, 173.6)
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Routing:
- net /Controll/5V_+: track 18.6 -> 182.1 mm
- net /Controll/PWR_RESET_GPIO_5: track 0.00 -> 52.9 mm
- net /Controll/PWR_SET_GPIO_5: track 0.00 -> 46.1 mm
- net /Controll/CTRL_GND: track 53.7 -> 91.4 mm, vias 5 -> 9
- net Net-(U3A--): track 18.5 -> 12.7 mm
- net /Controll/+15_IN: track 20.8 -> 15.8 mm
- net /EQModule/R_IN: track 82.3 -> 86.8 mm
- net /Controll/PD_GND_IN: track 35.7 -> 39.7 mm
- net /EQModule/L_IN: track 83.4 -> 86.7 mm
- net /Controll/AMP_V+_IN: track 107.3 -> 104.9 mm
- net /Controll/AMP_V-_IN: track 102.4 -> 100.2 mm
- net /Controll/R_IN: track 18.7 -> 16.9 mm
- net /Controll/L_IN: track 17.8 -> 19.5 mm
- net Net-(U4-VIN): track 33.0 -> 31.3 mm
- net GND: track 11.9 -> 10.7 mm
Other:
- outline, holes or cut-outs redrawn
