File: Audio/AudioCase.kicad_pcb (KiCad board)
At the start: 2 copper layers, 262.1 x 203.6 mm, 126 parts, among them J10 AMP_AUX_IN, J11 AMP_AUX_OUT, J12 AMP1_PWR, J13 PD_IN, J14 AUDIO_IN, J15 AMP1_LR, J16 AMP2_PWR, J17 AMP2_LR, J18 AMP3_PWR, J19 AMP4_PWR, J20 AMP5_PWR, J21 AMP3_LR, J22 AMP4_LR, J23 AMP5_LR, J24 OLED_PIN, J4 PWR_IN, J5 PWR_OUT, J6 AUX_IN, J7 V_IN, J8 AUX_OUT, J9 AMP_PWR, K1 AZ850P2-x, K10 AZ850P2-x, K2 AZ850P2-x, K3 AZ850P2-x, K4 AZ850P2-x, K5 AZ850P2-x, K6 AZ850P2-x, K7 AZ850P2-x, K8 AZ850P2-x, K9 AZ850P2-x, SW1 RotaryEncoder_Switch, U1 MCW03, U2 NJM4558, U3 NJM4558, U4 BP5293-50, U5 ULN2803A, U6 ULN2803A, U7 ULN2803A

Commit message: Controll基板のレイアウトを進め、AudioCase PCBと各シートを同期。
端子を上辺・入力左上・中央にリレー/ULN/Pico・下にUI・右に5Vとする配置へ更新。K1/K2のリレー接点配線とNetTieを含む回路図変更をPCBへ反映（PowerModuleの配線済み領域は維持）。

Co-authored-by: Cursor <cursoragent@cursor.com>
Parts:
- removed SW1: RotaryEncoder_Switch, Rotary_Encoder:RotaryEncoder_Alps_EC11E-Switch_Vertical_H20mm
- added J25: AMP5_LR, TerminalBlock_Phoenix:TerminalBlock_Phoenix_MKDS-1,5-2-5.08_1x02_P5.08mm_Horizontal, F.Cu at (165.6, 122.5)
- J13: value PD_IN -> ROTARY_SW; footprint TerminalBlock_Phoenix:TerminalBlock_Phoenix_MKDS-1,5-2-5.08_1x02_P5.08mm_Horizontal -> Connector_PinHeader_2.54mm:PinHeader_1x05_P2.54mm_Vertical
- J14: value AUDIO_IN -> PD_IN
- J15: value AMP1_LR -> AUDIO_IN
- J16: value AMP2_PWR -> OLED_PIN; footprint TerminalBlock_Phoenix:TerminalBlock_Phoenix_MKDS-1,5-2-5.08_1x02_P5.08mm_Horizontal -> Connector_PinHeader_2.54mm:PinHeader_1x04_P2.54mm_Vertical
- J17: value AMP2_LR -> AMP1_LR
- J18: value AMP3_PWR -> AMP2_PWR
- J19: value AMP4_PWR -> AMP2_LR
- J20: value AMP5_PWR -> AMP3_PWR
- J21: value AMP3_LR -> AMP4_PWR
- J22: value AMP4_LR -> AMP5_PWR
- J23: value AMP5_LR -> AMP3_LR
- J24: value OLED_PIN -> AMP4_LR; footprint Connector_PinHeader_2.54mm:PinHeader_1x04_P2.54mm_Vertical -> TerminalBlock_Phoenix:TerminalBlock_Phoenix_MKDS-1,5-2-5.08_1x02_P5.08mm_Horizontal
- moved J14 171.9 mm to (169.0, 211.8), turned to 90 degrees
- moved J16 164.6 mm to (41.7, 209.5), turned to 90 degrees
- moved J13 132.0 mm to (37.5, 200.5)
- moved J24 120.8 mm to (55.5, 110.0)
- moved U7 7.23 mm to (55.9, 171.9), turned to 90 degrees
- moved U6 4.62 mm to (87.5, 172.2), turned to 90 degrees
- moved A1 4.35 mm to (92.8, 191.5)
- moved U5 3.37 mm to (118.2, 172.2), turned to 90 degrees
Connections:
- J13 pad 1: /Controll/PD_GND_IN -> /Controll/ENC_A
- J13 pad 2: /Controll/+15_IN -> /Controll/ENC_B
- J14 pad 1: /Controll/R_IN -> /Controll/PD_GND_IN
- J14 pad 2: /Controll/L_IN -> /Controll/+15_IN
- J15 pad 1: /Controll/L_OUT -> /Controll/R_IN
- J15 pad 2: /Controll/R_OUT -> /Controll/L_IN
- J16 pad 1: /Controll/AMP_V+_OUT -> /Controll/CTRL_GND
- J16 pad 2: /Controll/AMP_V-_OUT -> /Controll/3V3
- J19 pad 1: /Controll/AMP_V+_OUT -> /Controll/L_OUT
- J19 pad 2: /Controll/AMP_V-_OUT -> /Controll/R_OUT
- J21 pad 1: /Controll/L_OUT -> /Controll/AMP_V+_OUT
- J21 pad 2: /Controll/R_OUT -> /Controll/AMP_V-_OUT
- J22 pad 1: /Controll/L_OUT -> /Controll/AMP_V+_OUT
- J22 pad 2: /Controll/R_OUT -> /Controll/AMP_V-_OUT
- J24 pad 1: /Controll/CTRL_GND -> /Controll/L_OUT
- J24 pad 2: /Controll/3V3 -> /Controll/R_OUT
- U5 pad 1: /Controll/AUDIO_SET_GPIO_1 -> /Controll/PWR_RESET_GPIO_2
- U5 pad 11: /Controll/PWR_RESET_RELAY_2 -> /Controll/PWR_SET_RELAY_2
- U5 pad 12: /Controll/PWR_SET_RELAY_2 -> /Controll/PWR_RESET_RELAY_2
- U5 pad 13: /Controll/AUDIO_RESET_RELAY_2 -> /Controll/AUDIO_SET_RELAY_2
- U5 pad 14: /Controll/AUDIO_SET_RELAY_2 -> /Controll/AUDIO_RESET_RELAY_2
- U5 pad 15: /Controll/PWR_RESET_RELAY_1 -> /Controll/PWR_SET_RELAY_1
- U5 pad 16: /Controll/PWR_SET_RELAY_1 -> /Controll/PWR_RESET_RELAY_1
- U5 pad 17: /Controll/AUDIO_RESET_RELAY_1 -> /Controll/AUDIO_SET_RELAY_1
- U5 pad 18: /Controll/AUDIO_SET_RELAY_1 -> /Controll/AUDIO_RESET_RELAY_1
- U5 pad 2: /Controll/AUDIO_RESET_GPIO_1 -> /Controll/PWR_SET_GPIO_2
- U5 pad 3: /Controll/PWR_SET_GPIO_1 -> /Controll/AUDIO_RESET_GPIO_2
- U5 pad 4: /Controll/PWR_RESET_GPIO_1 -> /Controll/AUDIO_SET_GPIO_2
- U5 pad 5: /Controll/AUDIO_SET_GPIO_2 -> /Controll/PWR_RESET_GPIO_1
- U5 pad 6: /Controll/AUDIO_RESET_GPIO_2 -> /Controll/PWR_SET_GPIO_1
- U5 pad 7: /Controll/PWR_SET_GPIO_2 -> /Controll/AUDIO_RESET_GPIO_1
- U5 pad 8: /Controll/PWR_RESET_GPIO_2 -> /Controll/AUDIO_SET_GPIO_1
- U6 pad 1: /Controll/AUDIO_SET_GPIO_3 -> /Controll/PWR_RESET_GPIO_4
- U6 pad 11: /Controll/PWR_RESET_RELAY_4 -> /Controll/AUDIO_SET_RELAY_3
- U6 pad 12: /Controll/PWR_SET_RELAY_4 -> /Controll/AUDIO_RESET_RELAY_3
- U6 pad 13: /Controll/AUDIO_RESET_RELAY_4 -> /Controll/PWR_SET_RELAY_3
- U6 pad 14: /Controll/AUDIO_SET_RELAY_4 -> /Controll/PWR_RESET_RELAY_3
- U6 pad 15: /Controll/PWR_RESET_RELAY_3 -> /Controll/AUDIO_SET_RELAY_4
- U6 pad 16: /Controll/PWR_SET_RELAY_3 -> /Controll/AUDIO_RESET_RELAY_4
- U6 pad 17: /Controll/AUDIO_RESET_RELAY_3 -> /Controll/PWR_SET_RELAY_4
- U6 pad 18: /Controll/AUDIO_SET_RELAY_3 -> /Controll/PWR_RESET_RELAY_4
- U6 pad 2: /Controll/AUDIO_RESET_GPIO_3 -> /Controll/PWR_SET_GPIO_4
- U6 pad 3: /Controll/PWR_SET_GPIO_3 -> /Controll/AUDIO_RESET_GPIO_4
- U6 pad 4: /Controll/PWR_RESET_GPIO_3 -> /Controll/AUDIO_SET_GPIO_4
- U6 pad 5: /Controll/AUDIO_SET_GPIO_4 -> /Controll/PWR_RESET_GPIO_3
- U6 pad 6: /Controll/AUDIO_RESET_GPIO_4 -> /Controll/PWR_SET_GPIO_3
- U6 pad 7: /Controll/PWR_SET_GPIO_4 -> /Controll/AUDIO_RESET_GPIO_3
- U6 pad 8: /Controll/PWR_RESET_GPIO_4 -> /Controll/AUDIO_SET_GPIO_3
- U7 pad 1: /Controll/AUDIO_SET_GPIO_5 -> /Controll/PWR_RESET_GPIO_5
- U7 pad 15: /Controll/PWR_RESET_RELAY_5 -> /Controll/AUDIO_SET_RELAY_5
- U7 pad 16: /Controll/PWR_SET_RELAY_5 -> /Controll/AUDIO_RESET_RELAY_5
- U7 pad 17: /Controll/AUDIO_RESET_RELAY_5 -> /Controll/PWR_SET_RELAY_5
- U7 pad 18: /Controll/AUDIO_SET_RELAY_5 -> /Controll/PWR_RESET_RELAY_5
- U7 pad 2: /Controll/AUDIO_RESET_GPIO_5 -> /Controll/PWR_SET_GPIO_5
- U7 pad 3: /Controll/PWR_SET_GPIO_5 -> /Controll/AUDIO_RESET_GPIO_5
- U7 pad 4: /Controll/PWR_RESET_GPIO_5 -> /Controll/AUDIO_SET_GPIO_5
Routing:
- net /Controll/5V_+: track 182.1 -> 45.5 mm
- net /Controll/PWR_RESET_GPIO_5: track 52.9 -> 0.00 mm
- net /Controll/PWR_SET_GPIO_5: track 46.1 -> 0.00 mm
- net /Controll/R_IN: track 16.9 -> 17.8 mm
- net /Controll/L_OUT: track 28.2 -> 27.3 mm

Commit message: AudioCaseを製造用に4基板へ分割
KiKitで切り出した個別PCBとGerber/ドリル出力を追加し、JLCPCB向けに各基板を個別発注できる形にします。

Co-authored-by: Cursor <cursoragent@cursor.com>
Parts:
- added J26: AMP5_LR, TerminalBlock_Phoenix:TerminalBlock_Phoenix_MKDS-1,5-2-5.08_1x02_P5.08mm_Horizontal, F.Cu at (47.5, 25.8)
- C22, C23: footprint Resistor_SMD:R_0603_1608Metric_Pad0.98x0.95mm_HandSolder -> Capacitor_SMD:C_1206_3216Metric_Pad1.33x1.80mm_HandSolder
- J14: value PD_IN -> AMP_PWR_IN
- J15: value AUDIO_IN -> PD_IN
- J16: value OLED_PIN -> AUDIO_IN; footprint Connector_PinHeader_2.54mm:PinHeader_1x04_P2.54mm_Vertical -> TerminalBlock_Phoenix:TerminalBlock_Phoenix_MKDS-1,5-2-5.08_1x02_P5.08mm_Horizontal
- J17: value AMP1_LR -> OLED_PIN; footprint TerminalBlock_Phoenix:TerminalBlock_Phoenix_MKDS-1,5-2-5.08_1x02_P5.08mm_Horizontal -> Connector_PinHeader_2.54mm:PinHeader_1x04_P2.54mm_Vertical
- J18: value AMP2_PWR -> AMP1_LR
- J19: value AMP2_LR -> AMP2_PWR
- J20: value AMP3_PWR -> AMP2_LR
- J21: value AMP4_PWR -> AMP3_PWR
- J22: value AMP5_PWR -> AMP4_PWR
- J23: value AMP3_LR -> AMP5_PWR
- J24: value AMP4_LR -> AMP3_LR
- J25: value AMP5_LR -> AMP4_LR
- R19, R20, R21, R22, R23, R24, R25, R26, R27, R28: footprint Resistor_SMD:R_0603_1608Metric_Pad0.98x0.95mm_HandSolder -> Resistor_SMD:R_1206_3216Metric_Pad1.30x1.75mm_HandSolder
- moved H14 231.0 mm to (178.8, 22.4)
- moved J14 207.5 mm to (32.5, 55.5), turned to -90 degrees
- moved H15 196.5 mm to (178.8, 113.6)
- moved J16 196.3 mm to (110.7, 25.8), turned to 180 degrees
- moved J25 134.1 mm to (72.7, 25.8), turned to 180 degrees
- moved J20 132.5 mm to (148.6, 25.8)
- moved H13 127.2 mm to (22.8, 22.4)
- moved J19 117.5 mm to (161.2, 25.8)
- moved J13 113.8 mm to (107.4, 110.7)
- moved H7 113.1 mm to (118.4, 174.8)
- moved H8 113.1 mm to (45.9, 174.8)
- moved C20 112.7 mm to (115.4, 133.4)
- moved R12 112.7 mm to (112.4, 154.8)
- moved R14 112.7 mm to (87.8, 141.8)
- moved R18 112.7 mm to (115.5, 140.8)
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Connections:
- J14 pad 1: /Controll/PD_GND_IN -> /Controll/AMP_V+_IN
- J14 pad 2: /Controll/+15_IN -> /Controll/AMP_V-_IN
- J15 pad 1: /Controll/R_IN -> /Controll/PD_GND_IN
- J15 pad 2: /Controll/L_IN -> /Controll/+15_IN
- J16 pad 1: /Controll/CTRL_GND -> /Controll/R_IN
- J16 pad 2: /Controll/3V3 -> /Controll/L_IN
- J17 pad 1: /Controll/L_OUT -> /Controll/CTRL_GND
- J17 pad 2: /Controll/R_OUT -> /Controll/3V3
- J18 pad 1: /Controll/AMP_V+_OUT -> /Controll/L_OUT
- J18 pad 2: /Controll/AMP_V-_OUT -> /Controll/R_OUT
- J19 pad 1: /Controll/L_OUT -> /Controll/AMP_V+_OUT
- J19 pad 2: /Controll/R_OUT -> /Controll/AMP_V-_OUT
- J20 pad 1: /Controll/AMP_V+_OUT -> /Controll/L_OUT
- J20 pad 2: /Controll/AMP_V-_OUT -> /Controll/R_OUT
- J23 pad 1: /Controll/L_OUT -> /Controll/AMP_V+_OUT
- J23 pad 2: /Controll/R_OUT -> /Controll/AMP_V-_OUT
- U7 pad 1: /Controll/PWR_RESET_GPIO_5 -> /Controll/AUDIO_RESET_GPIO_5
- U7 pad 15: /Controll/AUDIO_SET_RELAY_5 -> /Controll/PWR_SET_RELAY_5
- U7 pad 16: /Controll/AUDIO_RESET_RELAY_5 -> /Controll/PWR_RESET_RELAY_5
- U7 pad 17: /Controll/PWR_SET_RELAY_5 -> /Controll/AUDIO_SET_RELAY_5
- U7 pad 18: /Controll/PWR_RESET_RELAY_5 -> /Controll/AUDIO_RESET_RELAY_5
- U7 pad 2: /Controll/PWR_SET_GPIO_5 -> /Controll/AUDIO_SET_GPIO_5
- U7 pad 3: /Controll/AUDIO_RESET_GPIO_5 -> /Controll/PWR_RESET_GPIO_5
- U7 pad 4: /Controll/AUDIO_SET_GPIO_5 -> /Controll/PWR_SET_GPIO_5
Routing:
- net /Controll/5V_+: track 45.5 -> 489.2 mm, vias 0 -> 5
- net /Controll/AMP_V-_OUT: track 23.2 -> 301.7 mm, vias 0 -> 13
- net /Controll/AMP_V+_OUT: track 13.9 -> 206.5 mm, vias 0 -> 9
- net /Controll/R_IN: track 17.8 -> 184.4 mm, vias 0 -> 5
- net /Controll/AMP_V-_IN: track 100.2 -> 226.5 mm
- net /Controll/AMP_V+_IN: track 104.9 -> 224.4 mm
- net /Controll/R_OUT: track 22.2 -> 136.4 mm
- net /Controll/L_IN: track 19.5 -> 133.4 mm
- net /Controll/L_OUT: track 27.3 -> 103.9 mm, vias 0 -> 2
- net /Controll/AUDIO_SET_GPIO_5: track 0.00 -> 55.6 mm, vias 0 -> 2
- net /Controll/AUDIO_RESET_GPIO_5: track 0.00 -> 50.8 mm
- net /Controll/AUDIO_RESET_RELAY_5: track 0.00 -> 50.7 mm
- net /Controll/CTRL_GND: track 91.4 -> 40.8 mm, vias 9 -> 3
- net /Controll/AUDIO_SET_RELAY_5: track 0.00 -> 46.1 mm
- net /Controll/AUDIO_RESET_RELAY_2: track 0.00 -> 45.7 mm
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Other:
- board size 262.1 x 203.6 mm -> 258.2 x 159.4 mm

Commit message: ノイズ対策と製造データ整備: デカップリング追加・GNDベタ強化・シルク整理
- 5V_+ラインにデカップリング/バルク(C34-C37)を追加し、リレー切替時の電源変動を抑制
- F.CuにCTRL_GND/GNDベタを追加し、ステッチングビアで表裏GNDを補強(DC-DC周辺含む)
- 端子台ラベル等のシルク重なりを解消(J11/J14/J6/J4/L1/L2ほか)
- masterから4基板を再split、Gerber/zipを再生成

Co-authored-by: Cursor <cursoragent@cursor.com>
Parts:
- added C34: 0.1μF, Capacitor_SMD:C_1206_3216Metric_Pad1.33x1.80mm_HandSolder, B.Cu at (125.0, 106.4)
- added C35: 0.1μF, Capacitor_SMD:C_1206_3216Metric_Pad1.33x1.80mm_HandSolder, B.Cu at (76.0, 73.3)
- added C36: 0.1μF, Capacitor_SMD:C_1206_3216Metric_Pad1.33x1.80mm_HandSolder, B.Cu at (102.6, 73.4)
- added C37: 0.1μF, Capacitor_SMD:C_1206_3216Metric_Pad1.33x1.80mm_HandSolder, B.Cu at (128.4, 73.8)
- moved J6 0.80 mm to (60.2, 128.9)
- moved J11 0.70 mm to (270.5, 98.4)
- moved J10 0.55 mm to (222.8, 91.5)
- moved H8 0.26 mm to (46.2, 174.8)
- moved H5 0.25 mm to (46.2, 125.2)
- moved J8 0.23 mm to (106.4, 128.1)
Routing:
- net /Controll/5V_+: track 489.2 -> 503.2 mm
- net /Controll/L_OUT: track 103.9 -> 102.2 mm
- net Net-(AMP1-Pad7): track 8.82 -> 7.75 mm
- net Net-(AMP1A--): track 7.76 -> 6.86 mm
- net /Controll/R_OUT: track 136.4 -> 137.2 mm
- net /EQModule/R_IN: track 86.1 -> 85.5 mm
- net /AmpModule/R_OUT: track 14.3 -> 13.6 mm
- net /AmpModule/L_OUT: track 18.8 -> 18.1 mm
- net /EQModule/L_IN: track 86.7 -> 86.2 mm
- net GND: vias 4 -> 10
- net /Controll/CTRL_GND: vias 3 -> 30
- added copper zone on F.Cu, net /Controll/CTRL_GND
- added copper zone on F.Cu, net GND
Other:
- outline, holes or cut-outs redrawn
