File: Audio/AmpModule.kicad_sch (KiCad schematic)
At the start: 26 parts, among them J10 AMP_AUX_IN, J11 AMP_AUX_OUT, J9 AMP_PWR

Commit message: EQ update
Parts:
- renumbered C22 to C28, C23 to C29, C24 to C30, C25 to C31, C26 to C32, C27 to C33, C28 to C34, C29 to C35, R19 to R25, R20 to R26, R21 to R27, R22 to R28, R23 to R29, R24 to R30, R25 to R31, R26 to R32, R27 to R33, R28 to R34
Changed lines of the file:
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@@
 		(in_pos_files yes)
 		(dnp no)
-		(property "Reference" "C27"
+		(property "Reference" "C33"
 			(at 38.1 110.49 0)
 			(show_name no)
@@
 			(project "AudioCase"
 				(path "/760b9589-09e7-434e-9ca2-6e4136e3b7a2/477be123-54b6-4d91-ae02-fb2ccb128622"
-					(reference "C27")
+					(reference "C33")
 					(unit 1)
 				)
@@
 		(in_pos_files yes)
 		(dnp no)
-		(property "Reference" "R21"
+		(property "Reference" "R27"
 			(at 54.61 77.47 90)
 			(show_name no)
@@
 			(project "AudioCase"
 				(path "/760b9589-09e7-434e-9ca2-6e4136e3b7a2/477be123-54b6-4d91-ae02-fb2ccb128622"
-					(reference "R21")
+					(reference "R27")
 					(unit 1)
 				)
@@
 		(in_pos_files yes)
 		(dnp no)
-		(property "Reference" "R23"
+		(property "Reference" "R29"
 			(at 57.15 59.69 90)
 			(show_name no)
@@
 			(project "AudioCase"
 				(path "/760b9589-09e7-434e-9ca2-6e4136e3b7a2/477be123-54b6-4d91-ae02-fb2ccb128622"
-					(reference "R23")
+					(reference "R29")
 					(unit 1)
 				)
@@
 		(in_pos_files yes)
 		(dnp no)
-		(property "Reference" "R20"
+		(property "Reference" "R26"
 			(at 40.64 95.25 90)
 			(show_name no)
@@
 			(project "AudioCase"
 				(path "/760b9589-09e7-434e-9ca2-6e4136e3b7a2/477be123-54b6-4d91-ae02-fb2ccb128622"
-					(reference "R20")
+					(reference "R26")
 					(unit 1)
 				)
@@
 		(in_pos_files yes)
 		(dnp no)
-		(property "Reference" "C24"
+		(property "Reference" "C30"
 			(at 35.56 58.42 90)
 			(show_name no)
@@
 			(project "AudioCase"
 				(path "/760b9589-09e7-434e-9ca2-6e4136e3b7a2/477be123-54b6-4d91-ae02-fb2ccb128622"
-					(reference "C24")
+					(reference "C30")
 					(unit 1)
 				)
@@
 		(in_pos_files yes)
 		(dnp no)
-		(property "Reference" "R22"
+		(property "Reference" "R28"
 			(at 55.88 116.84 90)
 			(show_name no)
@@
 			(project "AudioCase"
 				(path "/760b9589-09e7-434e-9ca2-6e4136e3b7a2/477be123-54b6-4d91-ae02-fb2ccb128622"
-					(reference "R22")
+					(reference "R28")
 					(unit 1)
 				)
@@
 		(in_pos_files yes)
 		(dnp no)
-		(property "Reference" "C29"
+		(property "Reference" "C35"
 			(at 88.9 105.41 0)
 			(show_name no)
@@
 			(project "AudioCase"
 				(path "/760b9589-09e7-434e-9ca2-6e4136e3b7a2/477be123-54b6-4d91-ae02-fb2ccb128622"
-					(reference "C29")
+					(reference "C35")
 					(unit 1)
 				)
@@
 		(in_pos_files yes)
 		(dnp no)
-		(property "Reference" "C26"
+		(property "Reference" "C32"
 			(at 38.1 102.87 0)
 			(show_name no)
@@
 			(project "AudioCase"
 				(path "/760b9589-09e7-434e-9ca2-6e4136e3b7a2/477be123-54b6-4d91-ae02-fb2ccb128622"
-					(reference "C26")
+					(reference "C32")
 					(unit 1)
 				)
@@
 		(in_pos_files yes)
 		(dnp no)
-		(property "Reference" "R27"
+		(property "Reference" "R33"
 			(at 78.74 71.12 0)
 			(show_name no)
@@
 			(project "AudioCase"
 				(path "/760b9589-09e7-434e-9ca2-6e4136e3b7a2/477be123-54b6-4d91-ae02-fb2ccb128622"
-					(reference "R27")
+					(reference "R33")
 					(unit 1)
 				)
@@
 		(in_pos_files yes)
 		(dnp no)
-		(property "Reference" "C23"
+		(property "Reference" "C29"
 			(at 30.48 53.34 90)
 			(show_name no)
@@
 			(project "AudioCase"
 				(path "/760b9589-09e7-434e-9ca2-6e4136e3b7a2/477be123-54b6-4d91-ae02-fb2ccb128622"
-					(reference "C23")
+					(reference "C29")
 					(unit 1)
 				)
@@
 		(in_pos_files yes)
 		(dnp no)
-		(property "Reference" "C28"
+		(property "Reference" "C34"
 			(at 88.9 73.66 0)
 			(show_name no)
@@
 			(project "AudioCase"
 				(path "/760b9589-09e7-434e-9ca2-6e4136e3b7a2/477be123-54b6-4d91-ae02-fb2ccb128622"
-					(reference "C28")
+					(reference "C34")
 					(unit 1)
 				)
@@
 		(in_pos_files yes)
 		(dnp no)
-		(property "Reference" "R25"
+		(property "Reference" "R31"
 			(at 66.04 80.01 90)
 			(show_name no)
@@
 			(project "AudioCase"
 				(path "/760b9589-09e7-434e-9ca2-6e4136e3b7a2/477be123-54b6-4d91-ae02-fb2ccb128622"
-					(reference "R25")
+					(reference "R31")
 					(unit 1)
 				)
@@
 		(in_pos_files yes)
 		(dnp no)
-		(property "Reference" "R24"
+		(property "Reference" "R30"
 			(at 55.88 101.6 90)
 			(show_name no)
@@
 			(project "AudioCase"
 				(path "/760b9589-09e7-434e-9ca2-6e4136e3b7a2/477be123-54b6-4d91-ae02-fb2ccb128622"
-					(reference "R24")
+					(reference "R30")
 					(unit 1)
 				)
@@
 		(in_pos_files yes)
 		(dnp no)
-		(property "Reference" "C22"
+		(property "Reference" "C28"
 			(at 39.37 24.13 0)
 			(show_name no)
@@
 			(project "AudioCase"
 				(path "/760b9589-09e7-434e-9ca2-6e4136e3b7a2/477be123-54b6-4d91-ae02-fb2ccb128622"
-					(reference "C22")
+					(reference "C28")
 					(unit 1)
 				)
@@
 		(in_pos_files yes)
 		(dnp no)
-		(property "Reference" "C25"
+		(property "Reference" "C31"
 			(at 35.56 72.39 90)
 			(show_name no)
@@
 			(project "AudioCase"
 				(path "/760b9589-09e7-434e-9ca2-6e4136e3b7a2/477be123-54b6-4d91-ae02-fb2ccb128622"
-					(reference "C25")
+					(reference "C31")
 					(unit 1)
 				)
@@
 		(in_pos_files yes)
 		(dnp no)
-		(property "Reference" "R28"
+		(property "Reference" "R34"
 			(at 78.74 102.87 0)
 			(show_name no)
@@
 			(project "AudioCase"
 				(path "/760b9589-09e7-434e-9ca2-6e4136e3b7a2/477be123-54b6-4d91-ae02-fb2ccb128622"
-					(reference "R28")
+					(reference "R34")
 					(unit 1)
 				)
@@
 		(in_pos_files yes)
 		(dnp no)
-		(property "Reference" "R26"
+		(property "Reference" "R32"
 			(at 67.31 96.52 90)
 			(show_name no)
@@
 			(project "AudioCase"
 				(path "/760b9589-09e7-434e-9ca2-6e4136e3b7a2/477be123-54b6-4d91-ae02-fb2ccb128622"
-					(reference "R26")
+					(reference "R32")
 					(unit 1)
 				)
@@
 		(in_pos_files yes)
 		(dnp no)
-		(property "Reference" "R19"
+		(property "Reference" "R25"
 			(at 40.64 83.82 90)
 			(show_name no)
@@
 			(project "AudioCase"
 				(path "/760b9589-09e7-434e-9ca2-6e4136e3b7a2/477be123-54b6-4d91-ae02-fb2ccb128622"
-					(reference "R19")
-					(unit 1)
-				)
+					(reference "R25")
+					(unit 1)
+				)
