File: Audio/AmpModule.kicad_sch (KiCad schematic)
At the start: 26 parts, among them J10 AMP_AUX_IN, J11 AMP_AUX_OUT, J9 AMP_PWR

Commit message: AmpModuleのIC配置・配線を整理し、周辺の作業ファイルも合わせて反映する。
AmpModuleはNE5532のピン配置に合わせてIC(AMP1)を90°回転させ、L/Rチャンネルを
上下の行に揃えて左右の配線差を縮小。0.1µFの結合コンデンサ2個をSMD化してIC直近
まで寄せ、出力段(R33/R34→C34/C35→J11)の配線も整頓。マウントホールを基板外形内
に戻し、余計なスタブ・重複配線を削除。DRCは違反0件を確認済み。

そのほか、MeasurementADCの回路図更新とBOM整理、SPICEシミュレーション結果、
部品リファレンス資料(ASFL1/LT1763/Pico2ファームウェア)を追加。
Parts:
- C30, C32: footprint Capacitor_THT:C_Rect_L7.2mm_W2.5mm_P5.00mm_FKS2_FKP2_MKS2_MKP2 -> Capacitor_SMD:C_1206_3216Metric_Pad1.33x1.80mm_HandSolder
Changed lines of the file:
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@@
 			)
 		)
-		(property "Footprint" "Capacitor_THT:C_Rect_L7.2mm_W2.5mm_P5.00mm_FKS2_FKP2_MKS2_MKP2"
+		(property "Footprint" "Capacitor_SMD:C_1206_3216Metric_Pad1.33x1.80mm_HandSolder"
 			(at 36.83 59.9948 0)
 			(hide yes)
@@
 			)
 		)
-		(property "Footprint" "Capacitor_THT:C_Rect_L7.2mm_W2.5mm_P5.00mm_FKS2_FKP2_MKS2_MKP2"
+		(property "Footprint" "Capacitor_SMD:C_1206_3216Metric_Pad1.33x1.80mm_HandSolder"
 			(at 36.83 103.1748 0)
 			(hide yes)
