File: Audio/AmpModule.kicad_sch (KiCad schematic)
At the start: 26 parts, among them J10 AMP_AUX_IN, J11 AMP_AUX_OUT, J9 AMP_PWR

Commit message: AmpModuleの±15V入口にOS-CON 120µF/35Vバルクを追加し、参照番号を400番台へ振り直す。
Co-authored-by: Cursor <cursoragent@cursor.com>
Parts:
- added C401, C403: 120μF, Capacitor_THT:CP_Radial_D10.0mm_P5.00mm, symbol Device:C_Polarized
- renumbered AMP1 to AMP401, C28 to C402, C29 to C404, C30 to C405, C31 to C406, C34 to C407, C32 to C408, C35 to C409, C33 to C410, H9 to H401, H10 to H402, H11 to H403, H12 to H404, J9 to J401, J10 to J402, J11 to J403, R29 to R401, R33 to R402, R27 to R403, R25 to R404, R31 to R405, R26 to R406, R30 to R407, R32 to R408, R34 to R409, R28 to R410
Connections:
- net A_GND: now also C401.2, C403.1
- net V+_IN: now also C401.1
- net V-_IN: now also C403.2

Commit message: ヘッドホン出力と切替を追加し、S式検査をコミット前に走らせる。
Amp 後段を PHONE/MUTE/LINE に分け、NJM4556A の電流バッファとパッド付きボリュームを載せる。括弧崩れで回路図が開けなくなるのを check_sexpr と pre-commit で止める。

Co-authored-by: Cursor <cursoragent@cursor.com>
Other:
- moved on the sheet: C401, C403
