File: Audio/EQModule.kicad_sch (KiCad schematic)
At the start: 46 parts, among them J6 AUX_IN, J7 V_IN, J8 AUX_OUT, U2 NJM4558, U3 NJM4558

Commit message: Update audio KiCad project wiring.
Co-authored-by: Cursor <cursoragent@cursor.com>
Connections:
- net L BAX OUT renamed L_BAX_SUM
- net R BAX OUT renamed R_BAX_SUM
Changed lines of the file:
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@@
 		)
 	)
-	(label "L BAX OUT"
+	(label "L_BAX_SUM"
 		(at 81.28 144.78 180)
 		(effects
@@
 		)
 	)
-	(label "R BAX OUT"
+	(label "R_BAX_SUM"
 		(at 44.45 57.15 180)
 		(effects
@@
 		)
 	)
-	(label "L BAX OUT"
+	(label "L_BAX_SUM"
 		(at 72.39 101.6 180)
 		(effects
@@
 		)
 	)
-	(label "L BAX OUT"
+	(label "L_BAX_SUM"
 		(at 67.31 54.61 180)
 		(effects
@@
 		)
 	)
-	(label "R BAX OUT"
+	(label "R_BAX_SUM"
 		(at 49.53 104.14 180)
 		(effects
@@
 		)
 	)
-	(label "R BAX OUT"
+	(label "R_BAX_SUM"
 		(at 58.42 147.32 180)
 		(effects
@@
 		)
 	)
-	(label "L BAX OUT"
+	(label "L_BAX_SUM"
 		(at 115.57 137.16 180)
 		(effects
@@
 		)
 	)
-	(label "R BAX OUT"
+	(label "R_BAX_SUM"
 		(at 115.57 113.03 180)
 		(effects
