File: Audio/EQModule.kicad_sch (KiCad schematic)
At the start: 46 parts, among them J6 AUX_IN, J7 V_IN, J8 AUX_OUT, U2 NJM4558, U3 NJM4558

Commit message: EQ update
Connections:
- net at C13.1, R11.1: now also C15.1, RV2.5; no longer RV2.6
- net at R9.1, RV3.4: now also C16.2; no longer C17.2
- net at C17.1, RV3.5: now also C16.1, R12.1; no longer C16.2
- net at R5.1, RV1.4: now also C11.2; no longer C12.2
- net at R7.1, RV2.4: now also C13.2; no longer C15.2
- net at C11.1, R10.1: now also C12.2, RV1.5; no longer RV1.6
- new net: C17.2, RV3.6
- new net: C15.2, RV2.6
- new net: C12.1, RV1.6
Other:
- moved on the sheet: R10, R11, R12, R3, R5, R6

Commit message: EQ update
Parts:
- added C18, C20, C26, C27: 0.1μF, Capacitor_SMD:C_1206_3216Metric_Pad1.33x1.80mm_HandSolder, symbol Device:C
- added C19, C21: 10μF, Capacitor_THT:CP_Radial_D5.0mm_P2.00mm, symbol Device:C_Polarized
- added R13, R14: 0Ω, Resistor_SMD:R_1206_3216Metric_Pad1.30x1.75mm_HandSolder, symbol Device:R
- added R15, R16: 47kΩ, Resistor_SMD:R_1206_3216Metric_Pad1.30x1.75mm_HandSolder, symbol Device:R
- added R17, R18: 47Ω, Resistor_SMD:R_1206_3216Metric_Pad1.30x1.75mm_HandSolder, symbol Device:R
- added U2: NJM4558, Package_DIP:DIP-8_W7.62mm_Socket, symbol Amplifier_Operational:NJM4558
- renumbered C11 to C10, C10 to C11, C13 to C12, C12 to C13, C16 to C15, C15 to C16, C18 to C22, C19 to C23, C20 to C24, C21 to C25, R8 to R10, R9 to R11, R13 to R19, R14 to R20, R15 to R21, R16 to R22, R17 to R23, R18 to R24, R6 to R4, R4 to R5, R5 to R6, R10 to R8, R11 to R9, U2 to U3, U3 to U4
Connections:
- net A_GND: now also C26.2, C27.1, R15.2, R16.2
- net L_IN: now also C20.1, C20.2, C21.1, C21.2, R16.1, U2.3 (+); no longer R11.2, R6.2, R7.2
- net R_IN: now also C18.1, C18.2, C19.1, C19.2, R15.1, U2.5 (+); no longer R1.1, R2.1, R5.1
- net V+_IN: now also C26.1, U2.8 (V+)
- net V-_IN: now also C27.2, U2.4 (V-)
- new net: R14.2, U2.6 (-)
- new net: R14.1, R18.2, U2.7
- new net: R13.1, R17.2, U2.1
- new net: R13.2, U2.2 (-)
- new net L_BUFF: R11.2, R17.1, R6.2, R7.2
- new net R_BUFF: R1.1, R18.1, R2.1, R5.1
Other:
- moved on the sheet: J6, J8, R19, R20, R21, R22, R23, R24, U3A, U3B, U4A, U4B
