File: Audio/Controll.kicad_sch (KiCad schematic)
At the start: 44 parts, among them J12 AMP1_PWR, J13 ROTARY_SW, J14 AMP_PWR_IN, J15 PD_IN, J16 AUDIO_IN, J17 OLED_PIN, J18 AMP1_LR, J19 AMP2_PWR, J20 AMP2_LR, J21 AMP3_PWR, J22 AMP4_PWR, J23 AMP5_PWR, J24 AMP3_LR, J25 AMP4_LR, J26 AMP5_LR, K1 AZ850P2-x, K10 AZ850P2-x, K2 AZ850P2-x, K3 AZ850P2-x, K4 AZ850P2-x, K5 AZ850P2-x, K6 AZ850P2-x, K7 AZ850P2-x, K8 AZ850P2-x, K9 AZ850P2-x, U4 BP5293-50, U5 ULN2803A, U6 ULN2803A, U7 ULN2803A

Commit message: EQ update
Parts:
- renumbered C30 to C36, C31 to C37, C34 to C38, C32 to C39, C33 to C40, C37 to C41, C36 to C42, C35 to C43, U4 to U5, U5 to U6, U6 to U7, U7 to U8
Changed lines of the file:
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@@
 		(in_pos_files yes)
 		(dnp no)
-		(property "Reference" "C36"
+		(property "Reference" "C42"
 			(at 185.42 110.49 90)
 			(show_name no)
@@
 			(project "AudioCase"
 				(path "/760b9589-09e7-434e-9ca2-6e4136e3b7a2/e19c5b2a-a625-4260-8099-fc122fec1c7e"
-					(reference "C36")
+					(reference "C42")
 					(unit 1)
 				)
@@
 		(in_pos_files yes)
 		(dnp no)
-		(property "Reference" "C32"
+		(property "Reference" "C39"
 			(at 109.22 71.12 90)
 			(show_name no)
@@
 			(project "AudioCase"
 				(path "/760b9589-09e7-434e-9ca2-6e4136e3b7a2/e19c5b2a-a625-4260-8099-fc122fec1c7e"
-					(reference "C32")
+					(reference "C39")
 					(unit 1)
 				)
@@
 		(dnp no)
 		(fields_autoplaced yes)
-		(property "Reference" "U5"
+		(property "Reference" "U6"
 			(at 175.26 67.31 0)
 			(show_name no)
@@
 			(project "AudioCase"
 				(path "/760b9589-09e7-434e-9ca2-6e4136e3b7a2/e19c5b2a-a625-4260-8099-fc122fec1c7e"
-					(reference "U5")
+					(reference "U6")
 					(unit 1)
 				)
@@
 		(in_pos_files yes)
 		(dnp no)
-		(property "Reference" "C37"
+		(property "Reference" "C41"
 			(at 185.42 68.58 90)
 			(show_name no)
@@
 			(project "AudioCase"
 				(path "/760b9589-09e7-434e-9ca2-6e4136e3b7a2/e19c5b2a-a625-4260-8099-fc122fec1c7e"
-					(reference "C37")
+					(reference "C41")
 					(unit 1)
 				)
@@
 		(dnp no)
 		(fields_autoplaced yes)
-		(property "Reference" "U4"
+		(property "Reference" "U5"
 			(at 101.6 59.69 0)
 			(show_name no)
@@
 			(project "AudioCase"
 				(path "/760b9589-09e7-434e-9ca2-6e4136e3b7a2/e19c5b2a-a625-4260-8099-fc122fec1c7e"
-					(reference "U4")
+					(reference "U5")
 					(unit 1)
 				)
@@
 		(in_pos_files yes)
 		(dnp no)
-		(property "Reference" "C34"
+		(property "Reference" "C38"
 			(at 101.6 157.48 90)
 			(show_name no)
@@
 			(project "AudioCase"
 				(path "/760b9589-09e7-434e-9ca2-6e4136e3b7a2/e19c5b2a-a625-4260-8099-fc122fec1c7e"
-					(reference "C34")
+					(reference "C38")
 					(unit 1)
 				)
@@
 		(dnp no)
 		(fields_autoplaced yes)
-		(property "Reference" "U7"
+		(property "Reference" "U8"
 			(at 176.53 143.51 0)
 			(show_name no)
@@
 			(project "AudioCase"
 				(path "/760b9589-09e7-434e-9ca2-6e4136e3b7a2/e19c5b2a-a625-4260-8099-fc122fec1c7e"
-					(reference "U7")
+					(reference "U8")
 					(unit 1)
 				)
@@
 		(in_pos_files yes)
 		(dnp no)
-		(property "Reference" "C35"
+		(property "Reference" "C43"
 			(at 185.42 144.78 90)
 			(show_name no)
@@
 			(project "AudioCase"
 				(path "/760b9589-09e7-434e-9ca2-6e4136e3b7a2/e19c5b2a-a625-4260-8099-fc122fec1c7e"
-					(reference "C35")
+					(reference "C43")
 					(unit 1)
 				)
@@
 		(in_pos_files yes)
 		(dnp no)
-		(property "Reference" "C30"
+		(property "Reference" "C36"
 			(at 80.01 71.12 90)
 			(show_name no)
@@
 			(project "AudioCase"
 				(path "/760b9589-09e7-434e-9ca2-6e4136e3b7a2/e19c5b2a-a625-4260-8099-fc122fec1c7e"
-					(reference "C30")
+					(reference "C36")
 					(unit 1)
 				)
@@
 		(in_pos_files yes)
 		(dnp no)
-		(property "Reference" "C31"
+		(property "Reference" "C37"
 			(at 95.25 71.12 0)
 			(show_name no)
@@
 			(project "AudioCase"
 				(path "/760b9589-09e7-434e-9ca2-6e4136e3b7a2/e19c5b2a-a625-4260-8099-fc122fec1c7e"
-					(reference "C31")
+					(reference "C37")
 					(unit 1)
 				)
@@
 		(in_pos_files yes)
 		(dnp no)
-		(property "Reference" "C33"
+		(property "Reference" "C40"
 			(at 127 71.12 0)
 			(show_name no)
@@
 			(project "AudioCase"
 				(path "/760b9589-09e7-434e-9ca2-6e4136e3b7a2/e19c5b2a-a625-4260-8099-fc122fec1c7e"
-					(reference "C33")
+					(reference "C40")
 					(unit 1)
 				)
@@
 		(dnp no)
 		(fields_autoplaced yes)
-		(property "Reference" "U6"
+		(property "Reference" "U7"
 			(at 176.53 109.22 0)
 			(show_name no)
@@
 			(project "AudioCase"
 				(path "/760b9589-09e7-434e-9ca2-6e4136e3b7a2/e19c5b2a-a625-4260-8099-fc122fec1c7e"
-					(reference "U6")
+					(reference "U7")
 					(unit 1)
 				)
