File: Audio/AudioCase.kicad_sch (KiCad schematic)
At the start: 3 parts, among them J1 PD給電, J2 入力ジャック, J3 出力ジャック

Commit message: RVConvert基板を追加し、分割Gerber生成を5基板対応にする。
Co-authored-by: Cursor <cursoragent@cursor.com>
Other:
- added sheet RVConvert (RVConvert.kicad_sch)
Changed lines of the file:
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@@
+		)
+	)
+	(sheet
+		(at 144.78 60.96)
+		(size 12.7 11.43)
+		(exclude_from_sim no)
+		(in_bom yes)
+		(on_board yes)
+		(dnp no)
+		(fields_autoplaced yes)
+		(stroke
+			(width 0.1524)
+			(type solid)
+		)
+		(fill
+			(color 0 0 0 0)
+		)
+		(property "Sheetname" "RVConvert"
+			(at 144.78 60.2484 0)
+			(show_name no)
+			(do_not_autoplace no)
+			(effects
+				(font
+					(size 1.27 1.27)
+				)
+				(justify left bottom)
+			)
+		)
+		(property "Sheetfile" "RVConvert.kicad_sch"
+			(at 144.78 72.9746 0)
+			(show_name no)
+			(do_not_autoplace no)
+			(effects
+				(font
+					(size 1.27 1.27)
+				)
+				(justify left top)
+			)
+		)
+		(instances
+			(project "AudioCase"
+				(path "/760b9589-09e7-434e-9ca2-6e4136e3b7a2"
+					(page "6")
+				)
+			)
 		)
 	)
