File: Audio/MeasurementADC1804_Module.kicad_sch (KiCad schematic)
At the start: 3 parts, among them J1 PD給電, J2 入力ジャック, J3 出力ジャック

Commit message: MeasurementADC階層を追加し、基準計測用の電源・シンボルと進捗メモを整える。
KiCad 10向けにADC1804モジュール回路を移植し、親シート接続・Extrasライブラリ・ASFLフットプリント・ERCスナップショットを含める。

Co-authored-by: Cursor <cursoragent@cursor.com>
Parts:
- removed J1: PD給電, TerminalBlock_Phoenix:TerminalBlock_Phoenix_MKDS-1,5-2-5.08_1x02_P5.08mm_Horizontal, symbol Connector:Screw_Terminal_01x02
- removed J2: 入力ジャック, TerminalBlock_Phoenix:TerminalBlock_Phoenix_MKDS-1,5-2-5.08_1x02_P5.08mm_Horizontal, symbol Connector_Audio:AudioJack2_Ground
- removed J3: 出力ジャック, TerminalBlock_Phoenix:TerminalBlock_Phoenix_MKDS-1,5-2-5.08_1x02_P5.08mm_Horizontal, symbol Connector_Audio:AudioJack2_Ground
- added A2: ADC1804_F_MODULE, symbol MeasurementADC1804:ADC1804_F_MODULE
- added A3: Pico2, symbol MCU_Module:RaspberryPi_Pico
- added C44, C45, C60, C62: 100nF, symbol Device:C
- added C46, C47, C48, C49, C50, C51: 10uF 25V, symbol Device:C_Polarized
- added C52, C53, C54, C55: 0.1uF film, symbol Device:C
- added C56, C57, C58, C59: 1.8nF C0G/film, symbol Device:C
- added C61, C63: 10uF, symbol Device:C_Polarized
- added C64: 10uF IN, symbol Device:C
- added C65: 10uF, symbol Device:C
- added C66, C67: 0.1u CT, symbol Device:C
- added C68, C69: 10uF OUT, symbol Device:C
- added LCDDisplay1: WAVESHARE-29318, symbol MeasurementADC_Extras:WAVESHARE-29318
- added Q1: AO3401A, Package_TO_SOT_SMD:SOT-23, symbol Transistor_FET:AO3401A
- added R35, R36, R37, R38: 4.7k 0.1%, symbol Device:R
- added R39, R40, R41, R42: 3.3k 0.1%, symbol Device:R
- added R43, R44, R45, R46: 1k 0.1%, symbol Device:R
- added R47, R48, R49, R50: 47, symbol Device:R
- added R51: 100k, symbol Device:R
- added R52: 10k OD pullup, symbol Device:R
- added R53: 33 MCLK, symbol Device:R
- added U10, U11, U9: OPA1656, symbol MeasurementADC1804:OPA1656
- added U12: BP5293-50, symbol BP5293_ROHM:BP5293-50
- added U13: MBC2596-01, symbol MeasurementADC_Extras:MBC2596-01
- added U14: LT1763-3.3, symbol MeasurementADC_Extras:LT1763-3.3
- added U15: TPS3808 3V3, symbol Power_Supervisor:TPS3808DBV
- added U16: LT1763-5, symbol MeasurementADC_Extras:LT1763-5
- added U17: TPS3808 5V, symbol Power_Supervisor:TPS3808DBV
- added Y1: ASFL1-12.288MHZ-EC-T, symbol MeasurementADC_Extras:ASFL1-12.288MHZ
Connections:
- new net: C55.2, U11.3 (INA+)
- new net: C47.2, R38.1, U9.7 (OUTB)
- new net: R36.1, R38.2, U9.6 (INB-)
- new net: C57.1, R44.1, R48.2, U10.7 (OUTB)
- new net: C57.2, R42.1, R44.2, U10.6 (INB-)
- new net: C56.2, R41.1, R43.2, U10.2 (INA-)
- new net: C49.1, R41.2
- new net: C59.1, R46.1, R50.2, U11.7 (OUTB)
- new net: C59.2, R40.1, R46.2, U11.6 (INB-)
- new net: C50.1, R42.2
- new net: C48.1, R40.2
- new net: Q1.1 (G), R51.2
- new net: C58.1, R45.1, R49.2, U11.1 (OUTA)
- new net: C58.2, R39.1, R45.2, U11.2 (INA-)
- new net: R35.1, R37.2, U9.2 (INA-)
- new net: C49.2, R37.1, U9.1 (OUTA)
- new net: C56.1, R43.1, R47.2, U10.1 (OUTA)
- new net: C52.2, U10.3 (INA+)
- new net: C53.2, U10.5 (INB+)
- new net: C47.1, R39.2
- new net: C54.2, U11.5 (INB+)
- new net +15V_A: C44.1, C46.1, U10.8 (V+), U11.8 (V+), U9.8 (V+)
- new net +3V3_A: A2.12 (+5V), C60.1, C61.1, C62.1, C63.1, R52.1, U14.1 (OUT), U14.2 (SENSE), U15.3 (~{MR}), U15.5 (SENSE), U15.6 (VDD), U16.1 (OUT), U16.2 (SENSE), U16.5 (SHDN), U17.3 (~{MR}), U17.5 (SENSE), U17.6 (VDD), Y1.1 (ST), Y1.4 (VDD)
- new net +5V_D: A3.39 (VSYS), Q1.2 (S), U12.3 (VOUT)
- new net +6V7_PRE: C60.2, C61.2, C62.2, C63.2, U13.3 (OUT+), U13.4 (OUT-), U14.3 (GND), U14.5 (SHDN), U14.7 (GND), U14.8 (IN), U16.3 (GND), U16.7 (GND), U16.8 (IN)
- new net -15V_A: C45.2, C51.2, U10.4 (V-), U11.4 (V-), U9.4 (V-)
- new net ADC_BCK: A2.9 (BCK), A3.2 (GPIO1)
- new net ADC_DATA: A2.10 (DATA), A3.1 (GPIO0)
- new net ADC_GND_IN: A3.13 (GND), A3.18 (GND), A3.23 (GND), A3.28 (GND), A3.3 (GND), A3.38 (GND), A3.8 (GND), LCDDisplay1.2 (GND), U12.2 (GND), U13.2 (IN-)
- new net ADC_LRCK: A2.8 (LRCK), A3.4 (GPIO2)
- new net ADC_MCLK: A2.7 (SCKI), R53.2
- new net ADC_V_IN: U12.1 (VIN), U13.1 (IN+)
- new net ADC_nRST: A2.11 (RST), C66.2, C67.2, R52.2, U15.1 (~{RESET}), U15.4 (CT), U17.1 (~{RESET}), U17.4 (CT)
- new net AUDIO_L_IN: C50.2, R35.2
- new net AUDIO_R_IN: C48.2, R36.2
- new net A_GND: C44.2, C45.1, C46.2, C51.1, C66.1, C67.1, U15.2 (GND), U17.2 (GND), U9.3 (INA+), U9.5 (INB+), Y1.2 (GND)
- new net LCD_CS: A3.7 (GPIO5), LCDDisplay1.5 (LCD_CS)
- new net LCD_DC: A3.9 (GPIO6), LCDDisplay1.6 (LCD_DC)
- new net LCD_EN: A3.11 (GPIO8), R51.1
- new net LCD_MOSI: A3.6 (GPIO4), LCDDisplay1.3 (LCD_DIN)
- new net LCD_RST: A3.10 (GPIO7), LCDDisplay1.7 (LCD_RST)
- new net LCD_SCK: A3.5 (GPIO3), LCDDisplay1.4 (LCD_CLK)
- new net LCD_VCC: LCDDisplay1.1 (VCC), LCDDisplay1.8 (LCD_BL), Q1.3 (D)
- new net MCLK_RAW: R53.1, Y1.3 (OUT)
- new net PICO_3V3: A3.30 (RUN), A3.35 (ADC_VREF), A3.36 (3V3), A3.37 (3V3_EN)
- new net TP_INT: A3.16 (GPIO12), LCDDisplay1.11 (TP_INT)
- new net TP_RST: A3.17 (GPIO13), LCDDisplay1.12 (TP_RST)
- new net TP_SCL: A3.15 (GPIO11), LCDDisplay1.10 (TP_SCL)
- new net TP_SDA: A3.14 (GPIO10), LCDDisplay1.9 (TP_SDA)
- new net VCOML: A2.2 (VCOML), C52.1, C53.1
- new net VCOMR: A2.5 (VCOMR), C54.1, C55.1
- new net VINL+: A2.1 (VINL+), R48.1
- new net VINL-: A2.3 (VINL-), R47.1
- new net VINR+: A2.6 (VINR+), R50.1
- new net VINR-: A2.4 (VINR-), R49.1
- no-connect marks 0 -> 15
Other:
- removed sheet AmpModule
- removed sheet Controll
- removed sheet EQModule
- removed sheet MeasurementADC
- removed sheet PowerModule
- removed sheet RVConvert
- note added: "A3 Pico2: VSYS=+5V_D GND=A_GND | GP0=ADC_DATA GP1=ADC_BCK GP2=ADC_LRCK | GP3=LCD_SCK GP4=LCD_MOSI GP5=LCD_CS GP6=LCD_DC GP7=LCD_RST GP8=LCD_EN | GP10=TP_SDA GP11=TP_SCL GP12=TP_INT GP13=TP_RST. Wire labels to pins in EESchema."
- note added: "ADC/LCD のデジタル戻り電流を A_GND 入力トレースから遠ざける。GND はモジュール上の管理された一点で接続。"
- note added: "ADC1804_F には PCM1804 のデカップリングとジャンパが内蔵済み。本シートは外部コネクタのみをモデル化。"
- note added: "ADC1804_F モジュール / デジタル・インターフェース"
- note added: "ADC_V_IN ├─ BP5293-50 → +5V_D（Pico/LCD） └─ MBC2596 → ~6.6V ├─ LT1763-5 → +5V_A （ADC） └─ LT1763-3.3 → +3V3_A （ADC）"
- note added: "FE_PATCH_V1"
- note added: "JP1F でマスタ/スレーブ、I2S フォーマット、OSR、HPF をモジュールマニュアルに従い設定。"
- note added: "LRCK/BCK の向きは ADC マスタモード想定。スレーブ時は階層ピンの方向を合わせて変更すること。"
- note added: "OPA1656 の各電源ペアに 100nF を配置。バルクコンデンサはアナログフロントエンドの電源入口付近に。"
- note added: "OPA2134 からの OPA1656 置き換えは暫定。試作で安定性とフルスケール・レベルを確認すること。"
- note added: "PATCH_V1"
- note added: "PATCH_V2"
- note added: "POWER/DIGITAL: ADC_VIN->U15(6.6-6.8V)->U14(+3V3_A) then U13(+5V_A EN=+3V3_A). U12=+5V_D. Y1 ASFL1->R55->ADC_MCLK. U16/U17 SV wire-AND->ADC_nRST>=20ms. Q1 LCD load-SW; precision mode LCD off."
- note added: "PWRWIRE_V2"
- note added: "Q1 P-FET: LCD_EN low=ON. Precision: LCD_EN high cuts LCD/touch."
- note added: "U13 EN=+3V3_A (3V3-first). AbsMax VCC-VDD protection."
- note added: "U14 EN=+6V7_PRE. FB~3.3V (R51/R52). Place FB network to OUT/FB/GND."
- note added: "U16/U17: SENSE dividers for rails; CT delay >=20ms; OD ~RESET wire-AND to ADC_nRST."
- note added: "チャンネルあたりの公式リファレンス構成: 入力インバータ + ADC VCOM 基準の反転 LPF ドライバ×2。"
- note added: "右チャンネル"
- note added: "階層ポート / 左チャンネル"
- note removed: "MeasurementADC: ADC_V_IN+ADC_GND_IN=raw PD pair. AUDIO from Amp L/R_OUT. +/-15V_A from PowerModule."
- company: (none) -> AudioCase project
- title: (none) -> 計測モジュール - OPA1656 + ADC1804_F + Pico2 + LCD

Commit message: MeasurementADCのQ1ロードSW配線とスーパーバイザ周りを整理する。
LCD電源スイッチ近傍のラベル配置を直し、TPS3808埋め込みシンボルとコンデンサ参照を更新する。

Co-authored-by: Cursor <cursoragent@cursor.com>
Parts:
- renumbered C67 to C66, C68 to C67, C69 to C68, C66 to C69
Connections:
- net +3V3_A: no longer U15.5 (SENSE), U17.5 (SENSE)
- net ADC_nRST: no longer U15.4 (CT), U17.4 (CT)
Other:
- moved on the sheet: R51
Changed lines of the file:
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@@
 	(wire
 		(pts
-			(xy 328.93 143.51) (xy 331.47 143.51)
+			(xy 325.12 143.51) (xy 326.39 143.51)
 		)
 		(stroke
@@
 	(wire
 		(pts
+			(xy 334.01 143.51) (xy 340.36 143.51)
+		)
+		(stroke
+			(width 0)
+			(type default)
+		)
+	)
+	(wire
+		(pts
 			(xy 92.71 68.58) (xy 92.71 63.5)
 		)
@@
 	(wire
 		(pts
+			(xy 347.98 149.86) (xy 347.98 148.59)
+		)
+		(stroke
+			(width 0)
+			(type default)
+		)
+	)
+	(wire
+		(pts
 			(xy 82.55 25.4) (xy 83.82 25.4)
 		)
@@
 	(wire
 		(pts
-			(xy 347.98 148.59) (xy 347.98 151.13)
+			(xy 346.71 149.86) (xy 347.98 149.86)
 		)
 		(stroke
@@
 	(wire
 		(pts
-			(xy 339.09 143.51) (xy 340.36 143.51)
-		)
-		(stroke
-			(width 0)
-			(type default)
-		)
-	)
-	(wire
-		(pts
 			(xy 113.03 29.21) (xy 121.92 29.21)
 		)
@@
 	(wire
 		(pts
-			(xy 347.98 134.62) (xy 347.98 138.43)
-		)
-		(stroke
-			(width 0)
-			(type default)
-		)
-	)
-	(wire
-		(pts
 			(xy 45.72 40.64) (xy 36.83 40.64)
 		)
@@
 	(wire
 		(pts
+			(xy 347.98 137.16) (xy 347.98 138.43)
+		)
+		(stroke
+			(width 0)
+			(type default)
+		)
+	)
+	(wire
+		(pts
 			(xy 248.92 182.88) (xy 248.32 182.85)
 		)
@@
 	(wire
 		(pts
+			(xy 346.71 137.16) (xy 347.98 137.16)
+		)
+		(stroke
+			(width 0)
+			(type default)
+		)
+	)
+	(wire
+		(pts
 			(xy 222.25 161.29) (xy 224.79 161.29)
 		)
@@
 	)
 	(label "+5V_A"
-		(at 186.69 107.95 90)
+		(at 186.69 107.95 180)
 		(effects
 			(font
 				(size 1.27 1.27)
 			)
-			(justify left)
+			(justify right)
 		)
 	)
@@
 	)
 	(label "+5V_A"
-		(at 204.47 107.95 90)
+		(at 204.47 107.95 180)
 		(effects
 			(font
 				(size 1.27 1.27)
 			)
-			(justify left)
+			(justify right)
 		)
 	)
@@
 	)
 	(label "LCD_VCC"
-		(at 347.98 134.62 180)
+		(at 346.71 137.16 180)
 		(effects
 			(font
@@
 	)
 	(label "+5V_D"
-		(at 347.98 151.13 180)
+		(at 346.71 149.86 180)
 		(effects
 			(font
@@
 	)
 	(label "LCD_EN"
-		(at 328.93 143.51 180)
+		(at 325.12 143.51 180)
 		(effects
 			(font
@@
 		(in_pos_files yes)
 		(dnp no)
-		(property "Reference" "C68"
+		(property "Reference" "C67"
 			(at 430.53 27.94 0)
 			(show_name no)
@@
 			(project "AudioCase"
 				(path "/760b9589-09e7-434e-9ca2-6e4136e3b7a2/6d49c70d-b40d-4b21-ac6e-fba63bdae03e"
-					(reference "C68")
+					(reference "C67")
 					(unit 1)
 				)
@@
 		(in_pos_files yes)
 		(dnp no)
-		(property "Reference" "C66"
+		(property "Reference" "C69"
 			(at 440.69 142.24 0)
 			(show_name no)
@@
 			(project "AudioCase"
 				(path "/760b9589-09e7-434e-9ca2-6e4136e3b7a2/6d49c70d-b40d-4b21-ac6e-fba63bdae03e"
-					(reference "C66")
+					(reference "C69")
 					(unit 1)
 				)
@@
 	(symbol
 		(lib_id "Device:R")
-		(at 335.28 143.51 90)
+		(at 330.2 143.51 90)
 		(unit 1)
 		(body_style 1)
@@
 		(dnp no)
 		(property "Reference" "R51"
-			(at 332.74 142.24 90)
+			(at 327.66 142.24 90)
 			(show_name no)
 			(do_not_autoplace no)
@@
 		)
 		(property "Value" "100k"
-			(at 337.82 144.78 90)
+			(at 332.74 144.78 90)
 			(show_name no)
 			(do_not_autoplace no)
@@
 		)
 		(property "Footprint" ""
-			(at 335.28 143.51 0)
+			(at 330.2 143.51 0)
 			(hide yes)
 			(show_name no)
@@
 		)
 		(property "Datasheet" ""
-			(at 335.28 143.51 0)
+			(at 330.2 143.51 0)
 			(hide yes)
 			(show_name no)
@@
 		)
 		(property "Description" ""
-			(at 335.28 143.51 0)
+			(at 330.2 143.51 0)
 			(hide yes)
 			(show_name no)
@@
 	)
 	(symbol
+		(lib_name "TPS3808DBV_1")
 		(lib_id "Power_Supervisor:TPS3808DBV")
 		(at 405 130 0)
@@
 		(dnp no)
 		(property "Reference" "U17"
-			(at 405 127.46 0)
+			(at 399.92 123.65 0)
 			(show_name no)
 			(do_not_autoplace no)
@@
 		)
 		(property "Value" "TPS3808 5V"
-			(at 405 124.92 0)
+			(at 411.35 123.65 0)
 			(show_name no)
 			(do_not_autoplace no)
@@
 		(in_pos_files yes)
 		(dnp no)
-		(property "Reference" "C67"
+		(property "Reference" "C66"
 			(at 407.7 121.92 0)
 			(show_name no)
@@
 			(project "AudioCase"
 				(path "/760b9589-09e7-434e-9ca2-6e4136e3b7a2/6d49c70d-b40d-4b21-ac6e-fba63bdae03e"
-					(reference "C67")
+					(reference "C66")
 					(unit 1)
 				)
@@
 		(dnp no)
 		(property "Reference" "U15"
-			(at 395 109.22 0)
+			(at 389.412 105.156 0)
 			(show_name no)
 			(do_not_autoplace no)
@@
 		)
 		(property "Value" "TPS3808 3V3"
-			(at 395 106.68 0)
+			(at 402.112 105.41 0)
 			(show_name no)
 			(do_not_autoplace no)
@@
 		(in_pos_files yes)
 		(dnp no)
-		(property "Reference" "C69"
+		(property "Reference" "C68"
 			(at 436.88 72.39 0)
 			(show_name no)
@@
 			(project "AudioCase"
 				(path "/760b9589-09e7-434e-9ca2-6e4136e3b7a2/6d49c70d-b40d-4b21-ac6e-fba63bdae03e"
-					(reference "C69")
+					(reference "C68")
 					(unit 1)
 				)

Commit message: MeasurementADCをChatGPTレビュー指摘に合わせて直し、進捗メモを更新する。
VCOM直結・LDO型番・TPS3808 OCシンボル・OPA電源デカップなど初号NOGO要因を解消し、STATUSをレビュー追跡形式にする。

Co-authored-by: Cursor <cursoragent@cursor.com>
Parts:
- removed C51: 10uF 25V, symbol Device:C_Polarized
- removed C53, C55: 0.1uF film, symbol Device:C
- removed C66, C69: 0.1u CT, symbol Device:C
- removed C67, C68: 10uF OUT, symbol Device:C
- removed U16: LT1763-5, symbol MeasurementADC_Extras:LT1763-5
- removed U17: TPS3808 5V, symbol Power_Supervisor:TPS3808DBV
- added C47: 10uF 25V, symbol Device:C_Polarized
- added C48, C49, C56, C57, C65: 100nF, symbol Device:C
- added C58, C59: 0.1uF film, symbol Device:C
- added C70, C71, C74, C75: 10uF, symbol Device:C
- added C73, C76, C77: 10nF, symbol Device:C
- added C78, C79: 0.1uF VDD, symbol Device:C
- added NT22: NetTie_2, symbol Device:NetTie_2
- added U15: LT1763-5, Package_SO:SOIC-8_3.9x4.9mm_P1.27mm, symbol MeasurementADC_Extras:LT1763-5
- added U17: TPS3808G50DBVR, Package_TO_SOT_SMD:SOT-23-6, symbol MeasurementADC_Extras:TPS3808G50DBVR
- C64: value 10uF IN -> 100nF
- C72: renamed from C65; value 10uF -> 10nF
- LCDDisplay1: footprint (none) -> Connector_PinHeader_2.54mm:PinHeader_1x15_P2.54mm_Vertical
- U14: footprint (none) -> Package_SO:SOIC-8_3.9x4.9mm_P1.27mm
- U16: renamed from U15; value TPS3808 3V3 -> TPS3808G33DBVR; footprint (none) -> Package_TO_SOT_SMD:SOT-23-6; symbol Power_Supervisor:TPS3808DBV -> MeasurementADC_Extras:TPS3808G33DBVR
- renumbered C47 to C50, C48 to C51, C49 to C52, C50 to C53, C52 to C55, C56 to C60, C57 to C61, C58 to C62, C59 to C63, C60 to C66, C61 to C67, C62 to C68, C63 to C69, R53 to R52, R52 to R53
Connections:
- net +15V_A: now also C64.1, C48.1, C56.1
- net +3V3_A: now also A2.13 (+3V3), C72.1, U16.5 (SENSE), C74.1, C76.2, C78.1, U15.5 (SHDN); no longer A2.12 (+5V), C66.1, C67.1
- net +6V7_PRE: now also C70.1, C71.1, U15.8 (IN); no longer C66.2, C67.2, C68.2, C69.2, U13.4 (OUT-), U14.3 (GND), U14.7 (GND)
- net -15V_A: now also C47.2, C49.2, C57.2, C65.2
- net ADC_GND_IN: now also NT22.1; no longer A3.13 (GND), A3.18 (GND), A3.23 (GND), A3.28 (GND), A3.3 (GND), A3.38 (GND), A3.8 (GND), LCDDisplay1.2 (GND)
- net ADC_nRST: now also U17.1 (~{RESET})
- net A_GND: now also C54.2, C55.2, C64.2, C47.1, C48.2, C49.1, C56.2, C57.1, C58.2, C59.2, C65.1; no longer U16.2 (GND), Y1.2 (GND)
- net LCD_CS: now also LCDDisplay1.8 (LCD_CS); no longer LCDDisplay1.5 (LCD_CS)
- net LCD_DC: now also LCDDisplay1.9 (LCD_DC); no longer LCDDisplay1.6 (LCD_DC)
- net LCD_MOSI: now also LCDDisplay1.5 (MOSI); no longer LCDDisplay1.3 (LCD_DIN)
- net LCD_RST: now also LCDDisplay1.10 (LCD_RST); no longer LCDDisplay1.7 (LCD_RST)
- net LCD_SCK: now also LCDDisplay1.6 (SCLK); no longer LCDDisplay1.4 (LCD_CLK)
- net LCD_VCC: now also LCDDisplay1.11 (LCD_BL); no longer LCDDisplay1.8 (LCD_BL)
- net TP_INT: now also LCDDisplay1.14 (TP_INT); no longer LCDDisplay1.11 (TP_INT)
- net TP_RST: now also LCDDisplay1.15 (TP_RST); no longer LCDDisplay1.12 (TP_RST)
- net TP_SCL: now also LCDDisplay1.13 (TP_SCL); no longer LCDDisplay1.10 (TP_SCL)
- net TP_SDA: now also LCDDisplay1.12 (TP_SDA); no longer LCDDisplay1.9 (TP_SDA)
- net VCOML: now also C54.1, U10.3 (INA+), U10.5 (INB+)
- net VCOMR: now also U11.3 (INA+), U11.5 (INB+), C58.1, C59.1; no longer C54.1
- net ADC_GND: now reaches A2.14 (GND)
- net ADC_GND: now also C66.2, C67.2, C68.2, C69.2, U13.4 (OUT-), U14.3 (GND), U14.6 (GND), U14.7 (GND), U16.2 (GND), Y1.2 (GND), C70.2, C71.2, C74.2, C75.2, C76.1, C77.1, C78.2, C79.2, U15.3 (GND), U15.6 (GND), U15.7 (GND), U17.2 (GND)
- net at U14.4 (BYP): now also C72.2
- net MCLK_RAW: no longer names the net of R52.1, Y1.3 (OUT)
- new net: C73.2, U15.4 (BYP)
- new net +5V_A: A2.12 (+5V), C66.1, C67.1, C73.1, C75.1, C77.2, C79.1, U15.1 (OUT), U15.2 (SENSE), U17.5 (SENSE), U17.6 (VDD)
- new net D_GND: A3.13 (GND), A3.18 (GND), A3.23 (GND), A3.28 (GND), A3.3 (GND), A3.38 (GND), A3.8 (GND), LCDDisplay1.3 (GND), NT22.2
- no-connect marks 15 -> 21
Other:
- note added: "POWER/DIGITAL: ADC_VIN->U15(6.6-6.8V)->U14(+3V3_A) then U13(+5V_A EN=+3V3_A). U12=+5V_D. Y1 ASFL1->R55->ADC_MCLK. U16/U17 OD wire-AND->ADC_nRST (CT~0.57s). Q1 LCD load-SW; precision mode LCD off."
- note added: "U16=G33(+3V3_A) U17=G50(+5V_A); SENSE=rail; CT 0.1uF~0.57s (open~20ms); OD ~RESET wire-AND+R53; VDD 0.1uF local."
- note removed: "POWER/DIGITAL: ADC_VIN->U15(6.6-6.8V)->U14(+3V3_A) then U13(+5V_A EN=+3V3_A). U12=+5V_D. Y1 ASFL1->R55->ADC_MCLK. U16/U17 SV wire-AND->ADC_nRST>=20ms. Q1 LCD load-SW; precision mode LCD off."
- note removed: "U16/U17: SENSE dividers for rails; CT delay >=20ms; OD ~RESET wire-AND to ADC_nRST."
- moved on the sheet: A2, C55, C72, R51, R52, R53, U13, U16, Y1

Commit message: MeasurementADCシートの部品番号を700番台に振り直す。
階層シート内の参照衝突を避けるためのアノテーションのみ。他モジュールのネットは変更しない。

Co-authored-by: Cursor <cursoragent@cursor.com>
Parts:
- renumbered A2 to A701, A3 to A702, C44 to C701, C45 to C702, C46 to C703, C47 to C704, C48 to C705, C49 to C706, C50 to C707, C51 to C708, C52 to C709, C53 to C710, C54 to C711, C55 to C712, C56 to C713, C57 to C714, C58 to C715, C59 to C716, C60 to C717, C61 to C718, C62 to C719, C63 to C720, C64 to C721, C65 to C722, C66 to C723, C67 to C724, C68 to C725, C69 to C726, C70 to C727, C71 to C728, C72 to C729, C73 to C730, C74 to C731, C75 to C732, C76 to C733, C77 to C734, C78 to C735, C79 to C736, LCDDisplay1 to LCDDisplay701, NT22 to NT701, Q1 to Q701, R35 to R701, R36 to R702, R37 to R703, R38 to R704, R39 to R705, R40 to R706, R41 to R707, R42 to R708, R43 to R709, R44 to R710, R45 to R711, R46 to R712, R47 to R713, R48 to R714, R49 to R715, R50 to R716, R51 to R717, R52 to R718, R53 to R719, U9 to U701, U10 to U702, U11 to U703, U12 to U704, U13 to U705, U14 to U706, U15 to U707, U16 to U708, U17 to U709, Y1 to Y701

Commit message: MeasurementADCのGND星点・コンデンサ値・フットプリントを整える。
Option A（NT701/NT702）を明示し、高分子相当のバルクと1206系FPを割り当ててPCB化準備を進める。

Co-authored-by: Cursor <cursoragent@cursor.com>
Parts:
- removed C712: 0.1uF film, symbol Device:C
- removed C723, C725: 100nF, symbol Device:C
- removed C724, C726: 10uF, symbol Device:C_Polarized
- added C714: 47uF, Capacitor_THT:CP_Radial_D8.0mm_P3.50mm, symbol Device:C_Polarized
- added C729, C730, C736, C737, C738: 100nF, Capacitor_SMD:C_1206_3216Metric_Pad1.33x1.80mm_HandSolder, symbol Device:C
- added C735: 22uF, Capacitor_THT:CP_Radial_D6.3mm_P2.50mm, symbol Device:C_Polarized
- added J701, J702: Screw_Terminal_01x02, TerminalBlock_Phoenix:TerminalBlock_Phoenix_MKDS-1,5-2-5.08_1x02_P5.08mm_Horizontal, symbol Connector:Screw_Terminal_01x02
- added J703: Screw_Terminal_01x03, TerminalBlock_Phoenix:TerminalBlock_Phoenix_MKDS-1,5-3-5.08_1x03_P5.08mm_Horizontal, symbol Connector:Screw_Terminal_01x03
- added NT701: A_GND-ADC_GND, NetTie:NetTie-2_THT_Pad1.0mm, symbol Device:NetTie_2
- A702: footprint (none) -> Module:RaspberryPi_Pico_Common_Unspecified
- C701, C702, C705, C706, C721, C722: footprint (none) -> Capacitor_SMD:C_1206_3216Metric_Pad1.33x1.80mm_HandSolder
- C703, C704: value 10uF 25V -> 10uF 50V; footprint (none) -> Capacitor_THT:CP_Radial_D5.0mm_P2.00mm
- C707, C708, C709, C710: footprint (none) -> Capacitor_THT:CP_Radial_D5.0mm_P2.00mm
- C711, C715, C716: value 0.1uF film -> 100nF; footprint (none) -> Capacitor_SMD:C_1206_3216Metric_Pad1.33x1.80mm_HandSolder
- C712: renamed from C713; footprint (none) -> Capacitor_SMD:C_1206_3216Metric_Pad1.33x1.80mm_HandSolder
- C713: renamed from C714; footprint (none) -> Capacitor_SMD:C_1206_3216Metric_Pad1.33x1.80mm_HandSolder
- C717, C718, C719, C720: value 1.8nF C0G/film -> 1.8nF C0G; footprint (none) -> Capacitor_SMD:C_1206_3216Metric_Pad1.33x1.80mm_HandSolder
- C723: renamed from C727; value 10uF -> 10uF 16V X7R; footprint (none) -> Capacitor_SMD:C_1206_3216Metric_Pad1.33x1.80mm_HandSolder
- C724: renamed from C728; value 10uF -> 10uF 16V X7R; footprint (none) -> Capacitor_SMD:C_1206_3216Metric_Pad1.33x1.80mm_HandSolder
- C725: renamed from C729; footprint (none) -> Capacitor_SMD:C_1206_3216Metric_Pad1.33x1.80mm_HandSolder
- C726: renamed from C730; footprint (none) -> Capacitor_SMD:C_1206_3216Metric_Pad1.33x1.80mm_HandSolder
- C727: renamed from C731; value 10uF -> 10uF 10V X7R; footprint (none) -> Capacitor_SMD:C_1206_3216Metric_Pad1.33x1.80mm_HandSolder
- C728: renamed from C732; value 10uF -> 10uF 16V X7R; footprint (none) -> Capacitor_SMD:C_1206_3216Metric_Pad1.33x1.80mm_HandSolder
- C731: renamed from C733; footprint (none) -> Capacitor_SMD:C_1206_3216Metric_Pad1.33x1.80mm_HandSolder
- C732: renamed from C734; footprint (none) -> Capacitor_SMD:C_1206_3216Metric_Pad1.33x1.80mm_HandSolder
- C733: renamed from C735; value 0.1uF VDD -> 100nF; footprint (none) -> Capacitor_SMD:C_1206_3216Metric_Pad1.33x1.80mm_HandSolder
- C734: renamed from C736; value 0.1uF VDD -> 100nF; footprint (none) -> Capacitor_SMD:C_1206_3216Metric_Pad1.33x1.80mm_HandSolder
- NT702: renamed from NT701; value NetTie_2 -> ADC_GND_IN-D_GND; footprint (none) -> NetTie:NetTie-2_THT_Pad1.0mm
- R701: renamed from R702; footprint (none) -> Resistor_SMD:R_1206_3216Metric_Pad1.30x1.75mm_HandSolder
- R702: renamed from R701; footprint (none) -> Resistor_SMD:R_1206_3216Metric_Pad1.30x1.75mm_HandSolder
- R703: renamed from R704; footprint (none) -> Resistor_SMD:R_1206_3216Metric_Pad1.30x1.75mm_HandSolder
- R704: renamed from R703; footprint (none) -> Resistor_SMD:R_1206_3216Metric_Pad1.30x1.75mm_HandSolder
- R705, R706, R707, R708, R709, R710, R711, R712, R713, R714, R715, R716, R717, R718, R719: footprint (none) -> Resistor_SMD:R_1206_3216Metric_Pad1.30x1.75mm_HandSolder
- U701, U702, U703: footprint (none) -> Package_SO:SOIC-8_3.9x4.9mm_P1.27mm
- U704: footprint (none) -> Library:BP5293-50_ROHM_SIP-3
- U705: footprint (none) -> Connector_PinHeader_2.54mm:PinHeader_1x04_P2.54mm_Vertical
- Y701: footprint (none) -> Library:Oscillator_SMD_Abracon_ASFL-4Pin_5.0x3.2mm_HandSoldering
Connections:
- net +15V_A: now also J703.1 (Pin_1)
- net +3V3_A: now also C729.1
- net +5V_A: now also C730.1
- net +5V_D: now also C716.1, C714.1
- net -15V_A: now also J703.3 (Pin_3)
- net ADC_GND: now also C711.1, C715.1, C729.2, C730.2, C737.2, C738.2, NT701.1
- net ADC_GND_IN: now also J702.1 (Pin_1)
- net ADC_V_IN: now also J702.2 (Pin_2)
- net AUDIO_L_IN: now also J701.1 (Pin_1)
- net AUDIO_R_IN: now also J701.2 (Pin_2)
- net A_GND: now also J703.2 (Pin_2), NT701.2; no longer C711.2, C715.2, C716.2
- net D_GND: now also C716.2, C714.2, C735.2, C736.1
- net LCD_VCC: now also C735.1, C736.2
- net VCOML: now also C711.2; no longer C711.1
- net VCOMR: now also C715.2; no longer C715.1, C716.1
- net +6V7_PRE: no longer names the net of C723.1, C724.1, U705.3 (OUT+), U706.5 (SHDN), U706.8 (IN), U707.8 (IN)
- net +6V7_PRE: now also C737.1, C738.1
Other:
- note added: "A3 Pico2: VSYS=+5V_D GND=D_GND | GP0=ADC_DATA GP1=ADC_BCK GP2=ADC_LRCK | GP3=LCD_SCK GP4=LCD_MOSI GP5=LCD_CS GP6=LCD_DC GP7=LCD_RST GP8=LCD_EN | GP10=TP_SDA GP11=TP_SCL GP12=TP_INT GP13=TP_RST. Wire labels to pins in EESchema."
- note added: "GND: NT702=A_GND─ADC_GND（A701近傍・アナログ星点）。NT701=ADC_GND_IN─D_GND（PD入口）。Pico/LCD は D_GND のみ。D_GND は太く短く、アナログ入力から離す。計測経路は PD 基準（非絶縁完成）。"
- note removed: "A3 Pico2: VSYS=+5V_D GND=A_GND | GP0=ADC_DATA GP1=ADC_BCK GP2=ADC_LRCK | GP3=LCD_SCK GP4=LCD_MOSI GP5=LCD_CS GP6=LCD_DC GP7=LCD_RST GP8=LCD_EN | GP10=TP_SDA GP11=TP_SCL GP12=TP_INT GP13=TP_RST. Wire labels to pins in EESchema."
- note removed: "ADC/LCD のデジタル戻り電流を A_GND 入力トレースから遠ざける。GND はモジュール上の管理された一点で接続。"
- moved on the sheet: C701, C702, C703, C704, C705, C706, C707, C708, C709, C710, C712, C713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
