File: Audio/split/AudioCase_5_rv_convert.kicad_pcb (KiCad board)
At the start: 2 copper layers, 8.8 x 15.5 mm, 2 parts

Commit message: 分割Gerberを再生成し、05のzip名をスクリプト表記に揃える。
初号向け再出力を取り込み、旧05_rv_conv.zipを05_rv_convert.zipへ置き換える。

Co-authored-by: Cursor <cursoragent@cursor.com>
Parts:
- removed BAX, RV: Conn_01x06_Pin, Connector_PinHeader_2.54mm:PinHeader_2x03_P2.54mm_Vertical
- added J29: Conn_01x06_Pin, Connector_PinHeader_2.54mm:PinHeader_2x03_P2.54mm_Vertical, F.Cu at (146.0, 24.4)
- added J30: Conn_01x06_Pin, Connector_PinHeader_2.54mm:PinHeader_2x03_P2.54mm_Vertical, F.Cu at (146.0, 33.7)
Changed lines of the file:
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@@
 	(footprint "Connector_PinHeader_2.54mm:PinHeader_2x03_P2.54mm_Vertical"
 		(layer "F.Cu")
-		(at 145.96 24.44 90)
+		(at 145.995 33.69 90)
 		(descr "Through hole straight pin header, 2x03, 2.54mm pitch, double rows")
 		(tags "Through hole pin header THT 2x03 2.54mm double row")
-		(property "Reference" "BAX"
-			(at -2.46 -0.01 0)
+		(property "Reference" "J30"
+			(at 1.27 -2.38 90)
 			(unlocked yes)
 			(layer "F.SilkS")
@@
 		)
 		(property "Value" "Conn_01x06_Pin"
-			(at 5.665 2.44 0)
+			(at 1.27 7.46 90)
 			(unlocked yes)
 			(layer "F.Fab")
@@
 			)
 		)
-		(property "Description" ""
+		(property "Description" "Generic connector, single row, 01x06, script generated"
 			(at 0 0 90)
 			(layer "F.Fab")
@@
 				(font
 					(size 1.27 1.27)
-				)
-			)
-		)
-		(property "KiLib_Generator" "connector/pin_header_socket"
-			(at 0 0 90)
-			(layer "F.SilkS")
-			(hide yes)
-			(effects
-				(font
-					(size 1 1)
-					(thickness 0.15)
 				)
 			)
@@
 			(layers "*.Cu" "*.Mask")
 			(remove_unused_layers no)
-			(net "Net-(J29-Pin_1)")
+			(net "Net-(J29-Pin_3)")
 			(pinfunction "Pin_1_1")
 			(pintype "passive")
@@
 			(layers "*.Cu" "*.Mask")
 			(remove_unused_layers no)
-			(net "Net-(J29-Pin_3)")
+			(net "Net-(J29-Pin_1)")
 			(pinfunction "Pin_3_3")
 			(pintype "passive")
@@
 			(layers "*.Cu" "*.Mask")
 			(remove_unused_layers no)
-			(net "Net-(J29-Pin_4)")
+			(net "Net-(J29-Pin_6)")
 			(pinfunction "Pin_4_4")
 			(pintype "passive")
@@
 			(layers "*.Cu" "*.Mask")
 			(remove_unused_layers no)
-			(net "Net-(J29-Pin_6)")
+			(net "Net-(J29-Pin_4)")
 			(pinfunction "Pin_6_6")
 			(pintype "passive")
@@
 	(footprint "Connector_PinHeader_2.54mm:PinHeader_2x03_P2.54mm_Vertical"
 		(layer "F.Cu")
-		(at 145.975 33.73 90)
+		(at 145.975 24.44 90)
 		(descr "Through hole straight pin header, 2x03, 2.54mm pitch, double rows")
 		(tags "Through hole pin header THT 2x03 2.54mm double row")
-		(property "Reference" "RV"
-			(at 4.99 4.965 0)
+		(property "Reference" "J29"
+			(at 1.27 -2.38 90)
 			(unlocked yes)
 			(layer "F.SilkS")
@@
 		)
 		(property "Value" "Conn_01x06_Pin"
-			(at -3.31 2.265 0)
+			(at 1.27 7.46 90)
 			(unlocked yes)
 			(layer "F.Fab")
@@
 			)
 		)
-		(property "Description" ""
+		(property "Description" "Generic connector, single row, 01x06, script generated"
 			(at 0 0 90)
 			(layer "F.Fab")
@@
 				(font
 					(size 1.27 1.27)
-				)
-			)
-		)
-		(property "KiLib_Generator" "connector/pin_header_socket"
-			(at 0 0 90)
-			(layer "F.SilkS")
-			(hide yes)
-			(effects
-				(font
-					(size 1 1)
-					(thickness 0.15)
 				)
 			)
@@
 			(layers "*.Cu" "*.Mask")
 			(remove_unused_layers no)
-			(net "Net-(J29-Pin_3)")
+			(net "Net-(J29-Pin_1)")
 			(pinfunction "Pin_1_1")
 			(pintype "passive")
@@
 			(layers "*.Cu" "*.Mask")
 			(remove_unused_layers no)
-			(net "Net-(J29-Pin_1)")
+			(net "Net-(J29-Pin_3)")
 			(pinfunction "Pin_3_3")
 			(pintype "passive")
@@
 			(layers "*.Cu" "*.Mask")
 			(remove_unused_layers no)
-			(net "Net-(J29-Pin_6)")
+			(net "Net-(J29-Pin_4)")
 			(pinfunction "Pin_4_4")
 			(pintype "passive")
@@
 			(layers "*.Cu" "*.Mask")
 			(remove_unused_layers no)
-			(net "Net-(J29-Pin_4)")
+			(net "Net-(J29-Pin_6)")
 			(pinfunction "Pin_6_6")
 			(pintype "passive")
@@
 	)
 	(segment
-		(start 147.275 32.505)
-		(end 148.5 33.73)
-		(width 0.2)
-		(layer "F.Cu")
-		(net "Net-(J29-Pin_1)")
-	)
-	(segment
-		(start 147.275 25.77)
-		(end 147.275 32.505)
-		(width 0.2)
-		(layer "F.Cu")
-		(net "Net-(J29-Pin_1)")
-	)
-	(segment
-		(start 145.945 24.44)
-		(end 147.275 25.77)
-		(width 0.2)
-		(layer "F.Cu")
-		(net "Net-(J29-Pin_1)")
-	)
-	(segment
-		(start 145.945 21.9)
-		(end 144.7 23.145)
-		(width 0.2)
-		(layer "F.Cu")
-		(net "Net-(J29-Pin_2)")
-	)
-	(segment
-		(start 144.7 23.145)
-		(end 144.7 29.93)
-		(width 0.2)
-		(layer "F.Cu")
-		(net "Net-(J29-Pin_2)")
-	)
-	(segment
-		(start 144.7 29.93)
-		(end 145.96 31.19)
-		(width 0.2)
-		(layer "F.Cu")
-		(net "Net-(J29-Pin_2)")
+		(start 148.475 26.975)
+		(end 148.475 24.45)
+		(width 0.2)
+		(layer "F.Cu")
+		(net "Net-(J29-Pin_3)")
+	)
+	(segment
+		(start 148.475 24.45)
+		(end 148.485 24.44)
+		(width 0.2)
+		(layer "F.Cu")
+		(net "Net-(J29-Pin_3)")
 	)
 	(segment
 		(start 147.925 27.525)
 		(end 148.475 26.975)
-		(width 0.2)
-		(layer "F.Cu")
-		(net "Net-(J29-Pin_3)")
-	)
-	(segment
-		(start 148.475 24.45)
-		(end 148.485 24.44)
-		(width 0.2)
-		(layer "F.Cu")
-		(net "Net-(J29-Pin_3)")
-	)
-	(segment
-		(start 148.475 26.975)
-		(end 148.475 24.45)
 		(width 0.2)
 		(layer "F.Cu")
@@
 	)
 	(segment
+		(start 145.96 33.715)
+		(end 145.96 33.73)
+		(width 0.2)
+		(layer "B.Cu")
+		(net "Net-(J29-Pin_3)")
+	)
+	(segment
 		(start 147.275 28.175)
 		(end 147.275 32.4)
@@
 	)
 	(segment
-		(start 145.96 33.715)
-		(end 145.96 33.73)
-		(width 0.2)
-		(layer "B.Cu")
-		(net "Net-(J29-Pin_3)")
-	)
-	(segment
 		(start 147.925 27.525)
 		(end 147.275 28.175)
@@
 	)
 	(segment
-		(start 149.8 29.95)
-		(end 151.04 31.19)
-		(width 0.2)
-		(layer "F.Cu")
-		(net "Net-(J29-Pin_4)")
-	)
-	(segment
-		(start 149.8 23.215)
-		(end 149.8 29.95)
-		(width 0.2)
-		(layer "F.Cu")
-		(net "Net-(J29-Pin_4)")
-	)
-	(segment
-		(start 148.485 21.9)
-		(end 149.8 23.215)
-		(width 0.2)
-		(layer "F.Cu")
-		(net "Net-(J29-Pin_4)")
-	)
-	(segment
-		(start 149.775 30.05)
-		(end 149.775 32.45)
-		(width 0.2)
-		(layer "B.Cu")
-		(net "Net-(J29-Pin_5)")
-	)
-	(segment
-		(start 151.04 24.44)
-		(end 151.04 28.785)
-		(width 0.2)
-		(layer "B.Cu")
-		(net "Net-(J29-Pin_5)")
-	)
-	(segment
-		(start 149.775 32.45)
-		(end 151.055 33.73)
-		(width 0.2)
-		(layer "B.Cu")
-		(net "Net-(J29-Pin_5)")
-	)
-	(segment
-		(start 151.04 28.785)
-		(end 149.775 30.05)
-		(width 0.2)
-		(layer "B.Cu")
-		(net "Net-(J29-Pin_5)")
+		(start 145.945 21.9)
+		(end 144.7 23.145)
+		(width 0.2)
+		(layer "F.Cu")
+		(net "Net-(J29-Pin_2)")
+	)
+	(segment
+		(start 144.7 23.145)
+		(end 144.7 29.93)
+		(width 0.2)
+		(layer "F.Cu")
+		(net "Net-(J29-Pin_2)")
+	)
+	(segment
+		(start 144.7 29.93)
+		(end 145.96 31.19)
+		(width 0.2)
+		(layer "F.Cu")
+		(net "Net-(J29-Pin_2)")
+	)
+	(segment
+		(start 147.275 32.505)
+		(end 148.5 33.73)
+		(width 0.2)
+		(layer "F.Cu")
+		(net "Net-(J29-Pin_1)")
+	)
+	(segment
+		(start 147.275 25.77)
+		(end 147.275 32.505)
+		(width 0.2)
+		(layer "F.Cu")
+		(net "Net-(J29-Pin_1)")
+	)
+	(segment
+		(start 145.945 24.44)
+		(end 147.275 25.77)
+		(width 0.2)
+		(layer "F.Cu")
+		(net "Net-(J29-Pin_1)")
 	)
 	(segment
@@
 	)
 	(segment
+		(start 149.8 23.125)
+		(end 149.8 27.55)
+		(width 0.2)
+		(layer "B.Cu")
+		(net "Net-(J29-Pin_6)")
+	)
+	(segment
 		(start 149.8 27.55)
 		(end 148.5 28.85)
@@
 	)
 	(segment
-		(start 149.8 23.125)
-		(end 149.8 27.55)
-		(width 0.2)
-		(layer "B.Cu")
-		(net "Net-(J29-Pin_6)")
-	)
-	(segment
 		(start 151.025 21.9)
 		(end 149.8 23.125)
@@
 		(net "Net-(J29-Pin_6)")
 	)
+	(segment
+		(start 149.775 32.45)
+		(end 151.055 33.73)
+		(width 0.2)
+		(layer "B.Cu")
+		(net "Net-(J29-Pin_5)")
+	)
+	(segment
+		(start 151.04 28.785)
+		(end 149.775 30.05)
+		(width 0.2)
+		(layer "B.Cu")
+		(net "Net-(J29-Pin_5)")
+	)
+	(segment
+		(start 151.04 24.44)
+		(end 151.04 28.785)
+		(width 0.2)
+		(layer "B.Cu")
+		(net "Net-(J29-Pin_5)")
+	)
+	(segment
+		(start 149.775 30.05)
+		(end 149.775 32.45)
+		(width 0.2)
+		(layer "B.Cu")
+		(net "Net-(J29-Pin_5)")
+	)
+	(segment
+		(start 149.8 29.95)
+		(end 151.04 31.19)
+		(width 0.2)
+		(layer "F.Cu")
+		(net "Net-(J29-Pin_4)")
+	)
+	(segment
+		(start 149.8 23.215)
+		(end 149.8 29.95)
+		(width 0.2)
+		(layer "F.Cu")
+		(net "Net-(J29-Pin_4)")
+	)
+	(segment
+		(start 148.485 21.9)
+		(end 149.8 23.215)
+		(width 0.2)
+		(layer "F.Cu")
+		(net "Net-(J29-Pin_4)")
+	)
 	(embedded_fonts no)
