File: Audio/split/AudioCase_6_measurement_adc.kicad_pcb (KiCad board)
At the start: 2 copper layers, 182.6 x 83.7 mm, 87 parts, among them J701 AUDIO, J702 V_IN, J703 15_V_IN, U701 OPA1656, U702 OPA1656, U703 OPA1656, U704 BP5293-50, U705 MBC2596-01, U706 LT1763-3.3, U707 LT1763-5, U708 XC8107AC20MR-G, U709 TPS3808G33DBVR, U710 TPS3808G50DBVR, Y701 ASFL1-12.288MHZ-EC-T

Commit message: fix(MeasurementADC): Takman RLC25S を実寸シルクのフットプリントへ
DIN0309(9×φ3.2)は本体が大きすぎるため、RLC25SFY実寸(3.3×φ1.7)の
カスタム軸型FPに差し替え。パッドピッチ12.70mmは既存配線を維持。

Co-authored-by: m_arino <indare@users.noreply.github.com>
Parts:
- R713, R714, R715, R716, R719: footprint Resistor_THT:R_Axial_DIN0309_L9.0mm_D3.2mm_P12.70mm_Horizontal -> Library:R_Axial_Takman_RLC25S_L3.3mm_D1.7mm_P12.70mm_Horizontal
