File: AudioV2/ControlPanel.kicad_sch (KiCad schematic)
At the start: 16 parts, among them SW1 PWR SW, U1 Pico 2 / RP2350, U2 PT2314 tone, U3 PGA2310 HP, U4 PGA2310 LINE, U5 BP5293-50 +5V, U6 OLED ctrl I2C

Commit message: fix(AudioV2): PT2314 C1 を 100n に修正（R=2.4k と区別）
Parts:
- C1: value 2.4k PT2314 -> 100n PT2314
Changed lines of the file:
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@@
 			)
 		)
-		(property "Value" "2.4k PT2314"
-			(at 152.4 132.54 0)
+		(property "Value" "100n PT2314"
 			(show_name no)
 			(do_not_autoplace no)

Commit message: feat(AudioV2): CIRCUIT_DESIGNに沿って回路配置・配線（Control/Power/親）
- wire_circuit_design.py: PT2314 周辺 C/R、PGA2310 SPI/電源、7809、親バス
- PowerModule/ControlPanel/AudioV2Case を配線付きで再生成
- CIRCUIT_DESIGN.md チェックリスト更新

ERC は Relay/Output 未配線・親バス調整残り
Parts:
- removed C1: 100n PT2314, symbol Device:C
- removed R1: 2.4k PT2314, symbol Device:R
- added C201: 0.1u, symbol Device:C
- added C202, C203, C211, C212: 2.2u, symbol Device:C
- added C204: 22u, symbol Device:C
- added C205, C206, C207, C208: 100n, symbol Device:C
- added C209, C210: 2.7n, symbol Device:C
- added R201: 5.6k, symbol Device:R
- added R202, R203, R204, R205, R208, R209: 2.4k, symbol Device:R
- added R210, R211: 4.7k, symbol Device:R
- added R220: 10k, symbol Device:R
- U2: value PT2314 tone -> PT2314
Other:
- note added: "ControlPanel — CIRCUIT_DESIGN wired (§10 + §3) PT2314 @9V / PGA2310PA×2 / Pico2 / ENC×6 TONE_L/R → Amp inputs (off-sheet). AMP_SEL ← selected Amp output"
- note removed: "ControlPanel — DRAFT (§10) Pico 2 / ENC×6 GPIO direct / SSD1306 I2C0 PT2314 tone / PGA2310PA×2 SPI daisy / BP5293 +5V PWR SW + 12V LED on PD_12V (§9)"
