File: AudioV2/ControlPanel.kicad_sch (KiCad schematic)
At the start: 36 parts, among them SW1 PWR SW, U1 Pico 2 / RP2350, U2 PT2314, U3 PGA2310 HP, U4 PGA2310 LINE, U5 BP5293-50 +5V, U6 OLED ctrl I2C

Commit message: refactor(AudioV2): KiCad標準libへ置換（PGA2310/ULN2803/ENC） (#20)
- Audio:PGA2310PA, Transistor_Array:ULN2803A, Device:RotaryEncoder_Switch
- 配線スクリプトの PGA2310 ピン座標を標準シンボルに合わせて更新
- AudioV2.kicad_sym から PGA2310PA カスタム定義を削除
- PT2314 / DKMW20F-12 / CH224 モジュールは標準 lib 無しのため維持
- CIRCUIT_DESIGN.md に lib 方針表を追加

Co-authored-by: Cursor Agent <cursoragent@cursor.com>
Parts:
- removed J_ENC1: ENC_CH GP0/1/12, symbol Connector:Conn_01x05_Pin
- removed J_ENC2: ENC_HP GP2/3/13, symbol Connector:Conn_01x05_Pin
- removed J_ENC3: ENC_LINE GP4/5/14, symbol Connector:Conn_01x05_Pin
- removed J_ENC4: ENC_DEST GP6/7/15, symbol Connector:Conn_01x05_Pin
- removed J_ENC5: ENC_BASS GP8/9/26, symbol Connector:Conn_01x05_Pin
- removed J_ENC6: ENC_TREBLE GP10/11/27, symbol Connector:Conn_01x05_Pin
- removed U3: PGA2310 HP, symbol AudioV2:PGA2310PA
- removed U4: PGA2310 LINE, symbol AudioV2:PGA2310PA
- added ENC1: EC11 ENC_CH GP0/1/12, symbol Device:RotaryEncoder_Switch
- added ENC2: EC11 ENC_HP GP2/3/13, symbol Device:RotaryEncoder_Switch
- added ENC3: EC11 ENC_LINE GP4/5/14, symbol Device:RotaryEncoder_Switch
- added ENC4: EC11 ENC_DEST GP6/7/15, symbol Device:RotaryEncoder_Switch
- added ENC5: EC11 ENC_BASS GP8/9/26, symbol Device:RotaryEncoder_Switch
- added ENC6: EC11 ENC_TREBLE GP10/11/27, symbol Device:RotaryEncoder_Switch
- added U3: PGA2310PA HP, symbol Audio:PGA2310PA
- added U4: PGA2310PA LINE, symbol Audio:PGA2310PA
Changed lines of the file:
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@@
 	)
 	(symbol
-		(lib_id "AudioV2:PGA2310PA")
+		(lib_id "Audio:PGA2310PA")
 		(at 127.0 78.0 0)
 		(unit 1)
@@
 			)
 		)
-		(property "Value" "PGA2310 HP"
+		(property "Value" "PGA2310PA HP"
 			(at 127.0 80.54 0)
 			(show_name no)
@@
 	)
 	(symbol
-		(lib_id "AudioV2:PGA2310PA")
+		(lib_id "Audio:PGA2310PA")
 		(at 127.0 95.0 0)
 		(unit 1)
@@
 			)
 		)
-		(property "Value" "PGA2310 LINE"
+		(property "Value" "PGA2310PA LINE"
 			(at 127.0 97.54 0)
 			(show_name no)
@@
 	)
 	(symbol
-		(lib_id "Connector:Conn_01x05_Pin")
+		(lib_id "Device:RotaryEncoder_Switch")
 		(at 35.56 40.64 0)
 		(unit 1)
@@
 		(dnp no)
 		(fields_autoplaced yes)
-		(property "Reference" "J_ENC1"
+		(property "Reference" "ENC1"
 			(at 35.56 38.1 0)
 			(show_name no)
@@
 			)
 		)
-		(property "Value" "ENC_CH GP0/1/12"
+		(property "Value" "EC11 ENC_CH GP0/1/12"
 			(at 35.56 43.18 0)
 			(show_name no)
@@
 			(project "AudioV2Case"
 				(path "/a1000001-0001-4001-8001-000000000001/a1000006-0006-4006-8006-000000000006"
-					(reference "J_ENC1")
+					(reference "ENC1")
 					(unit 1)
 				)
@@
 	)
 	(symbol
-		(lib_id "Connector:Conn_01x05_Pin")
+		(lib_id "Device:RotaryEncoder_Switch")
 		(at 35.56 55.88 0)
 		(unit 1)
@@
 		(dnp no)
 		(fields_autoplaced yes)
-		(property "Reference" "J_ENC2"
+		(property "Reference" "ENC2"
 			(at 35.56 53.34 0)
 			(show_name no)
@@
 			)
 		)
-		(property "Value" "ENC_HP GP2/3/13"
+		(property "Value" "EC11 ENC_HP GP2/3/13"
 			(at 35.56 58.42 0)
 			(show_name no)
@@
 			(project "AudioV2Case"
 				(path "/a1000001-0001-4001-8001-000000000001/a1000006-0006-4006-8006-000000000006"
-					(reference "J_ENC2")
+					(reference "ENC2")
 					(unit 1)
 				)
@@
 	)
 	(symbol
-		(lib_id "Connector:Conn_01x05_Pin")
+		(lib_id "Device:RotaryEncoder_Switch")
 		(at 35.56 71.12 0)
 		(unit 1)
@@
 		(dnp no)
 		(fields_autoplaced yes)
-		(property "Reference" "J_ENC3"
+		(property "Reference" "ENC3"
 			(at 35.56 68.58 0)
 			(show_name no)
@@
 			)
 		)
-		(property "Value" "ENC_LINE GP4/5/14"
+		(property "Value" "EC11 ENC_LINE GP4/5/14"
 			(at 35.56 73.66000000000001 0)
 			(show_name no)
@@
 			(project "AudioV2Case"
 				(path "/a1000001-0001-4001-8001-000000000001/a1000006-0006-4006-8006-000000000006"
-					(reference "J_ENC3")
+					(reference "ENC3")
 					(unit 1)
 				)
@@
 	)
 	(symbol
-		(lib_id "Connector:Conn_01x05_Pin")
+		(lib_id "Device:RotaryEncoder_Switch")
 		(at 35.56 86.36 0)
 		(unit 1)
@@
 		(dnp no)
 		(fields_autoplaced yes)
-		(property "Reference" "J_ENC4"
+		(property "Reference" "ENC4"
 			(at 35.56 83.82 0)
 			(show_name no)
@@
 			)
 		)
-		(property "Value" "ENC_DEST GP6/7/15"
+		(property "Value" "EC11 ENC_DEST GP6/7/15"
 			(at 35.56 88.9 0)
 			(show_name no)
@@
 			(project "AudioV2Case"
 				(path "/a1000001-0001-4001-8001-000000000001/a1000006-0006-4006-8006-000000000006"
-					(reference "J_ENC4")
+					(reference "ENC4")
 					(unit 1)
 				)
@@
 	)
 	(symbol
-		(lib_id "Connector:Conn_01x05_Pin")
+		(lib_id "Device:RotaryEncoder_Switch")
 		(at 35.56 101.6 0)
 		(unit 1)
@@
 		(dnp no)
 		(fields_autoplaced yes)
-		(property "Reference" "J_ENC5"
+		(property "Reference" "ENC5"
 			(at 35.56 99.05999999999999 0)
 			(show_name no)
@@
 			)
 		)
-		(property "Value" "ENC_BASS GP8/9/26"
+		(property "Value" "EC11 ENC_BASS GP8/9/26"
 			(at 35.56 104.14 0)
 			(show_name no)
@@
 			(project "AudioV2Case"
 				(path "/a1000001-0001-4001-8001-000000000001/a1000006-0006-4006-8006-000000000006"
-					(reference "J_ENC5")
+					(reference "ENC5")
 					(unit 1)
 				)
@@
 	)
 	(symbol
-		(lib_id "Connector:Conn_01x05_Pin")
+		(lib_id "Device:RotaryEncoder_Switch")
 		(at 35.56 116.84 0)
 		(unit 1)
@@
 		(dnp no)
 		(fields_autoplaced yes)
-		(property "Reference" "J_ENC6"
+		(property "Reference" "ENC6"
 			(at 35.56 114.3 0)
 			(show_name no)
@@
 			)
 		)
-		(property "Value" "ENC_TREBLE GP10/11/27"
+		(property "Value" "EC11 ENC_TREBLE GP10/11/27"
 			(at 35.56 119.38000000000001 0)
 			(show_name no)
@@
 			(project "AudioV2Case"
 				(path "/a1000001-0001-4001-8001-000000000001/a1000006-0006-4006-8006-000000000006"
-					(reference "J_ENC6")
+					(reference "ENC6")
 					(unit 1)
 				)
@@
 	(wire
 		(pts
-			(xy 50.0 131.0) (xy 137.16 72.92)
+			(xy 50.0 131.0) (xy 132.08 105.94)
 		)
 		(stroke
@@
 	(wire
 		(pts
-			(xy 50.0 133.0) (xy 137.16 70.38)
+			(xy 50.0 133.0) (xy 132.08 50.06)
 		)
 		(stroke
@@
 	(wire
 		(pts
-			(xy 50.0 125.0) (xy 116.84 67.84)
+			(xy 50.0 125.0) (xy 114.3 95.78)
 		)
 		(stroke
@@
 	(wire
 		(pts
-			(xy 50.0 125.0) (xy 137.16 78.0)
+			(xy 50.0 125.0) (xy 114.3 60.22)
 		)
 		(stroke
@@
 	(wire
 		(pts
-			(xy 50.0 115.0) (xy 116.84 78.0)
+			(xy 50.0 115.0) (xy 121.92 105.94)
 		)
 		(stroke
@@
 	(wire
 		(pts
-			(xy 50.0 128.0) (xy 116.84 75.46)
+			(xy 50.0 128.0) (xy 121.92 50.06)
 		)
 		(stroke
@@
 	(wire
 		(pts
-			(xy 50.0 115.0) (xy 116.84 85.62)
+			(xy 50.0 115.0) (xy 114.3 83.08)
 		)
 		(stroke
@@
 	(wire
 		(pts
-			(xy 86.2 83.0) (xy 116.84 72.92)
+			(xy 86.2 83.0) (xy 114.3 80.54)
 		)
 		(stroke
@@
 	(wire
 		(pts
-			(xy 86.2 80.5) (xy 116.84 80.54)
+			(xy 86.2 80.5) (xy 114.3 78.0)
 		)
 		(stroke
@@
 	(wire
 		(pts
-			(xy 86.2 78.0) (xy 116.84 83.08)
+			(xy 86.2 78.0) (xy 114.3 75.46)
 		)
 		(stroke
@@
 	(wire
 		(pts
-			(xy 137.16 85.62) (xy 116.84 97.54)
+			(xy 114.3 70.38) (xy 114.3 95.0)
 		)
 		(stroke
@@
 	(wire
 		(pts
-			(xy 86.2 85.5) (xy 137.16 83.08)
+			(xy 86.2 85.5) (xy 114.3 85.62)
 		)
 		(stroke
@@
 	(wire
 		(pts
-			(xy 116.84 70.38) (xy 195.0 130.0)
+			(xy 139.7 93.24) (xy 195.0 130.0)
 		)
 		(stroke
@@
 	(wire
 		(pts
-			(xy 137.16 75.46) (xy 195.0 132.54)
+			(xy 139.7 62.76) (xy 195.0 132.54)
 		)
 		(stroke
@@
 	(wire
 		(pts
-			(xy 50.0 105.0) (xy 116.84 82.3)
+			(xy 50.0 105.0) (xy 114.3 107.7)
 		)
 		(stroke
@@
 	(wire
 		(pts
-			(xy 50.0 107.0) (xy 137.16 97.54)
+			(xy 50.0 107.0) (xy 114.3 82.3)
 		)
 		(stroke
@@
 	(wire
 		(pts
-			(xy 116.84 87.38) (xy 195.0 135.08)
+			(xy 139.7 110.24) (xy 195.0 135.08)
 		)
 		(stroke
@@
 	(wire
 		(pts
-			(xy 137.16 92.46) (xy 195.0 137.62)
+			(xy 139.7 79.76) (xy 195.0 137.62)
 		)
 		(stroke
