File: AudioV2/PowerModule.kicad_sch (KiCad schematic)
At the start: 7 parts, among them J1 USB-C PD in, J202 ±12+A_GND out, U1 DKMW20F-12, U2 50224_CH224, U3 LM7809 +9V

Commit message: feat(AudioV2): CIRCUIT_DESIGNに沿って回路配置・配線（Control/Power/親）
- wire_circuit_design.py: PT2314 周辺 C/R、PGA2310 SPI/電源、7809、親バス
- PowerModule/ControlPanel/AudioV2Case を配線付きで再生成
- CIRCUIT_DESIGN.md チェックリスト更新

ERC は Relay/Output 未配線・親バス調整残り
Parts:
- removed U3: LM7809 +9V, symbol Regulator_Linear:AP1117-33
- added C301: 10u, symbol Device:C
- added C302: 0.1u, symbol Device:C
- added U3: LM7809 +9V, symbol Regulator_Linear:LM7809_TO220
- J202: value ±12+A_GND out -> +12/-12/A_GND
Other:
- note added: "AudioV2 PowerModule — CIRCUIT_DESIGN wired U1 DKMW20F-12 / U2 50224 / F1 3A slow / U3 LM7809 +9V See CIRCUIT_DESIGN.md §4"
- note removed: "AudioV2 PowerModule — DRAFT (§8/§9) U1 DKMW20F-12 ±12V / U2 50224 CH224 USB-C PD F1 → DKMW20 +Vin. PD_12V → panel PWR SW → PD_12V_SW U3 LM7809 +9V → VCC_TONE (PT2314 typ 9V, see CIRCUIT_DESIGN.md)"
