File: AudioV2/PowerModule.kicad_sch (KiCad schematic)
At the start: 14 parts, among them J201 +15/-15/A_GND out, J202 PD module in (1=GND 2=+12V), J203 VCC_TONE OUT (1=A_GND 2=9V), U201 DKMW20F-15, U202 LM7809 +9V

Commit message: AudioV2: PowerModule の DC-DC を REC10K-2415DAW/H2 へ差し替え
ユーザーが KiCad で差し替え、こちらで検証と文書追随を行った。

ネットリストで全6ピンの接続が機能どおりであることを確認:
  1=+Vin  -> Net-(U203-+Vin)（F201 3A slow 経由、C205 47u / C206 0.1u 付き）
  2=-Vin  -> /PD_GND
  3=CTRL  -> unconnected（オープン=ON。DKMW の R.C. と同極性で配線変更不要）
  4=-Vout -> /-15V
  5=COM   -> /A_GND
  6=+Vout -> /+15V
不一致 0 件。旧 U201 は残っていない。

差し替えの再採番で U201 -> U203 に変わった。生成コード側は U201/DKMW20F-15 の
ままなので drift の差は広がったが、手編集所有なので想定内。

検証: check_sexpr 9/0、ERC 60件で変化なし（新規違反ゼロ）、
drift 生成コード所有 2/2 一致、gen_parts_bom --check rc=0。

文書の追随:
- CIRCUIT_DESIGN.md の信号経路・シンボル一覧・カスタム部品表
- DECISIONS.md の電源レール要約行と、8 の電流マージン節（DKMW20F-15 の
  ±660mA 前提の計算に、±333mA でも負荷率 62% で結論不変である旨を追記）
- AGENT_HANDOFF 2.10 を「差し替え済み」に更新し、穴位置と機能の対応表を残した

.gitattributes が効いて PowerModule の差分は 227 行に収まった（従来なら
改行コードだけで数千行の見せかけ差分になっていた）。

Co-Authored-By: Claude Opus 5 <noreply@anthropic.com>
Parts:
- removed U201: DKMW20F-15, symbol AudioV2:DKMW20F-15
- added U203: REC10K-2415DAW/H2, Library:REC10K-AW_1in_THT, symbol AudioV2:REC10K-2415DAW
Connections:
- net +15V: now also U203.6 (+Vout)
- net -15V: now also U203.4 (-Vout)
- net A_GND: now also U203.5 (COM)
- net PD_GND: now also U203.2 (-Vin)
- net at C205.2, C206.2, F201.2: now also U203.1 (+Vin)
Changed lines of the file:
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@@
-	)
-	(symbol
-		(lib_id "AudioV2:DKMW20F-15")
-		(at 111.76 76.2 0)
-		(unit 1)
-		(body_style 1)
-		(exclude_from_sim no)
-		(in_bom yes)
-		(on_board yes)
-		(in_pos_files yes)
-		(dnp no)
-		(property "Reference" "U201"
-			(at 111.76 74.93 0)
-			(show_name no)
-			(do_not_autoplace no)
-			(effects
-				(font
-					(size 1.27 1.27)
-				)
-			)
-		)
-		(property "Value" "DKMW20F-15"
-			(at 111.76 77.47 0)
-			(show_name no)
-			(do_not_autoplace no)
-			(effects
-				(font
-					(size 1.27 1.27)
-				)
-			)
-		)
-		(property "Footprint" ""
-			(at 2.54 22.86 0)
-			(hide yes)
-			(show_name no)
-			(do_not_autoplace no)
-			(effects
-				(font
-					(size 1.27 1.27)
-				)
-			)
-		)
-		(property "Datasheet" ""
-			(at 2.54 22.86 0)
-			(hide yes)
-			(show_name no)
-			(do_not_autoplace no)
-			(effects
-				(font
-					(size 1.27 1.27)
-				)
-			)
-		)
-		(property "Description" ""
-			(at 2.54 22.86 0)
-			(hide yes)
-			(show_name no)
-			(do_not_autoplace no)
-			(effects
-				(font
-					(size 1.27 1.27)
-				)
-			)
-		)
-		(pin "1"
-		)
-		(pin "2"
-		)
-		(pin "3"
-		)
-		(pin "4"
-		)
-		(pin "5"
-		)
-		(pin "6"
-		)
-		(instances
-			(project "AudioV2Case"
-				(path "/a1000001-0001-4001-8001-000000000001/a1000002-0002-4002-8002-000000000002"
-					(reference "U201")
-					(unit 1)
-				)
-			)
-		)
 	)
 	(symbol
@@
 					(unit 1)
 				)
+			)
+		)
+	)
+	(symbol
+		(lib_id "AudioV2:REC10K-2415DAW")
+		(at 111.76 76.2 0)
+		(unit 1)
+		(body_style 1)
+		(exclude_from_sim no)
+		(in_bom yes)
+		(on_board yes)
+		(in_pos_files yes)
+		(dnp no)
+		(fields_autoplaced yes)
+		(property "Reference" "U203"
+			(at 111.76 73.66 0)
+			(show_name no)
+			(do_not_autoplace no)
+			(effects
+				(font
+					(size 1.27 1.27)
+				)
+			)
+		)
+		(property "Value" "REC10K-2415DAW/H2"
+			(at 111.76 76.2 0)
+			(show_name no)
+			(do_not_autoplace no)
+			(effects
+				(font
+					(size 1.27 1.27)
+				)
+			)
+		)
+		(property "Footprint" "Library:REC10K-AW_1in_THT"
+			(at 113.03 72.39 0)
+			(hide yes)
+			(show_name no)
+			(do_not_autoplace no)
+			(effects
+				(font
+					(size 1.27 1.27)
+				)
+			)
+		)
+		(property "Datasheet" "https://recom-power.com/pdf/Econoline/REC10K-AW.pdf"
+			(at 112.268 74.422 0)
+			(hide yes)
+			(show_name no)
+			(do_not_autoplace no)
+			(effects
+				(font
+					(size 1.27 1.27)
+				)
+			)
+		)
+		(property "Description" "Mean Well DKMW20F-15 isolated DC/DC, 9-36Vin, ±15V/±660mA, DIP 1in x 1in, Cout 650uF/rail; DS datasheets/MeanWell_SKMW20_DKMW20.pdf"
+			(at 111.76 76.2 0)
+			(hide yes)
+			(show_name no)
+			(do_not_autoplace no)
+			(effects
+				(font
+					(size 1.27 1.27)
+				)
+			)
+		)
+		(property "Manufacturer" "MEAN WELL"
+			(at 111.76 76.2 0)
+			(hide yes)
+			(show_name no)
+			(do_not_autoplace no)
+			(effects
+				(font
+					(size 1.27 1.27)
+				)
+			)
+		)
+		(property "MPN" "DKMW20F-15"
+			(at 111.76 76.2 0)
+			(hide yes)
+			(show_name no)
+			(do_not_autoplace no)
+			(effects
+				(font
+					(size 1.27 1.27)
+				)
+			)
+		)
+		(pin "5"
+		)
+		(pin "6"
+		)
+		(pin "4"
+		)
+		(pin "3"
+		)
+		(pin "2"
+		)
+		(pin "1"
+		)
+		(instances
+			(project "AudioV2Case"
+				(path "/a1000001-0001-4001-8001-000000000001/a1000002-0002-4002-8002-000000000002"
+					(reference "U203")
+					(unit 1)
+				)

Commit message: AudioV2: 再アノテーション（PowerModule の DC-DC を U201 へ戻す）
ユーザーが KiCad で再アノテーション。DC-DC 差し替えの際に U203 へ動いていた
参照を U201 に戻した。副次的に AmpChannel 内の参照割り当ても入れ替わった
（集合は同じで 320 箇所の再割り当て。例: 220k は R603/R608/R611/R612 ->
R603/R605/R609/R611）。

Description はシンボルのプロパティなので部品に付いたまま動いており、
入出力プルダウンの L/R 対応は保たれている（BOM の 220k 行で確認）。
文書側はネット名・機能名で書いてあるため影響を受けない
（SOURCE_OF_TRUTH.md 3 の方針どおり）。

検証:
- check_sexpr 9ファイル / 問題0
- ネットリストで DC-DC 全6ピンが機能どおり:
  1=+Vin -> Net-(U201-+Vin)、2=-Vin -> /PD_GND、3=CTRL -> 未接続、
  4=-Vout -> /-15V、5=COM -> /A_GND、6=+Vout -> /+15V（不一致 0 件）
- AmpChannel の出力プルダウン 20/20 が OUT_L/OUT_R -> A_GND
- ERC 60件で変化なし
- drift 生成コード所有 2/2 一致
- PARTS.md の BOM を再生成（--check rc=0）

Co-Authored-By: Claude Opus 5 <noreply@anthropic.com>
Parts:
- renumbered U203 to U201
Changed lines of the file:
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@@
 		(dnp no)
 		(fields_autoplaced yes)
-		(property "Reference" "U203"
+		(property "Reference" "U201"
 			(at 111.76 73.66 0)
 			(show_name no)
@@
 			(project "AudioV2Case"
 				(path "/a1000001-0001-4001-8001-000000000001/a1000002-0002-4002-8002-000000000002"
-					(reference "U203")
+					(reference "U201")
 					(unit 1)
 				)
