File: AudioV2/OutputStage.kicad_sch (KiCad schematic)
At the start: 6 parts, among them K1 DEST LINE, K2 DEST PHONE, K3 DEST MUTE, U1 ULN spare/TODO

Commit message: refactor(AudioV2): KiCad標準libへ置換（PGA2310/ULN2803/ENC） (#20)
- Audio:PGA2310PA, Transistor_Array:ULN2803A, Device:RotaryEncoder_Switch
- 配線スクリプトの PGA2310 ピン座標を標準シンボルに合わせて更新
- AudioV2.kicad_sym から PGA2310PA カスタム定義を削除
- PT2314 / DKMW20F-12 / CH224 モジュールは標準 lib 無しのため維持
- CIRCUIT_DESIGN.md に lib 方針表を追加

Co-authored-by: Cursor Agent <cursoragent@cursor.com>
Parts:
- removed U1: ULN spare/TODO, symbol ULN2803A:ULN2803A
- added U1: ULN spare/TODO, symbol Transistor_Array:ULN2803A
Changed lines of the file:
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@@
 	)
 	(symbol
-		(lib_id "ULN2803A:ULN2803A")
+		(lib_id "Transistor_Array:ULN2803A")
 		(at 63.5 50.8 0)
 		(unit 1)
