File: AudioV2/OutputStage.kicad_sch (KiCad schematic)
At the start: 6 parts, among them SW601 DEST L (PHONE/MUTE/LINE), SW602 DEST R (PHONE/MUTE/LINE)

Commit message: update
Parts:
- added J_RAIL601: RAIL IN, symbol Connector:Screw_Terminal_01x03
Connections:
- net AMP_SEL_L: now also J_RAIL601.1 (Pin_1)
- net AMP_SEL_R: now also J_RAIL601.3 (Pin_3)
- net A_GND: now also J_RAIL601.2 (Pin_2)
- net MUTE_NC_L: no longer names the net of SW601.2
- net MUTE_NC_R: no longer names the net of SW602.2
- no-connect marks 0 -> 2
Other:
- moved on the sheet: J_HP601, J_LINE601, RV602, SW601, SW602
