File: AudioV2/OutputStage.kicad_sch (KiCad schematic)
At the start: 7 parts, among them SW601 DEST L (PHONE/MUTE/LINE), SW602 DEST R (PHONE/MUTE/LINE)

Commit message: AudioV2: AmpCh2手直しに伴う所有権更新、電源コンバータ代替調査、発注リスト追加
AmpBank/AmpChannelはユーザーがKiCadでAmpCh2を手直ししたため生成コード所有
から手編集所有へ卒業（wire_circuit_design.pyのHAND_EDITED/GENERATED更新、
driftで確認）。バルクコンデンサ周りの未接続配線をユーザーが修正、ERC 60件に復帰。

DECISIONS.md §11.1に電流マージンの実測ベース数値根拠を追記（±15V化後の実負荷、
オペアンプ差し替え最悪ケース）。PowerModuleの絶縁型DC-DCコンバータ(DKMW20F-15)
のコスト代替調査を開始し、AGENT_HANDOFF.md §2.10に途中経過と次のアクションを
記録（dc_dc.csvはDigiKeyのフィルタ済みエクスポート）。

AudioV2全体の発注リスト(PROCUREMENT.xlsx)を新規作成。

Co-Authored-By: Claude Sonnet 5 <noreply@anthropic.com>
Parts:
- renumbered J_HP601 to J_HP501, J_LINE601 to J_LINE501, J_RAIL601 to J_RAIL501, RV601 to RV501, RV602 to RV502, SW601 to SW501, SW602 to SW502
Changed lines of the file:
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@@
 		(in_pos_files yes)
 		(dnp no)
-		(property "Reference" "J_LINE601"
+		(property "Reference" "J_LINE501"
 			(at 173.99 53.34 0)
 			(show_name no)
@@
 			(project "AudioV2Case"
 				(path "/a1000001-0001-4001-8001-000000000001/a1000007-0007-4007-8007-000000000007"
-					(reference "J_LINE601")
+					(reference "J_LINE501")
 					(unit 1)
 				)
@@
 		(in_pos_files yes)
 		(dnp no)
-		(property "Reference" "RV601"
+		(property "Reference" "RV501"
 			(at 127 31.75 0)
 			(show_name no)
@@
 			(project "AudioV2Case"
 				(path "/a1000001-0001-4001-8001-000000000001/a1000007-0007-4007-8007-000000000007"
-					(reference "RV601")
+					(reference "RV501")
 					(unit 1)
 				)
@@
 		(in_pos_files yes)
 		(dnp no)
-		(property "Reference" "SW601"
+		(property "Reference" "SW501"
 			(at 62.23 43.18 0)
 			(show_name no)
@@
 			(project "AudioV2Case"
 				(path "/a1000001-0001-4001-8001-000000000001/a1000007-0007-4007-8007-000000000007"
-					(reference "SW601")
+					(reference "SW501")
 					(unit 1)
 				)
@@
 		(in_pos_files yes)
 		(dnp no)
-		(property "Reference" "J_HP601"
+		(property "Reference" "J_HP501"
 			(at 173.99 38.1 0)
 			(show_name no)
@@
 			(project "AudioV2Case"
 				(path "/a1000001-0001-4001-8001-000000000001/a1000007-0007-4007-8007-000000000007"
-					(reference "J_HP601")
+					(reference "J_HP501")
 					(unit 1)
 				)
@@
 		(in_pos_files yes)
 		(dnp no)
-		(property "Reference" "RV602"
+		(property "Reference" "RV502"
 			(at 127 63.5 0)
 			(show_name no)
@@
 			(project "AudioV2Case"
 				(path "/a1000001-0001-4001-8001-000000000001/a1000007-0007-4007-8007-000000000007"
-					(reference "RV602")
+					(reference "RV502")
 					(unit 1)
 				)
@@
 		(in_pos_files yes)
 		(dnp no)
-		(property "Reference" "J_RAIL601"
+		(property "Reference" "J_RAIL501"
 			(at 36.83 45.72 0)
 			(show_name no)
@@
 			(project "AudioV2Case"
 				(path "/a1000001-0001-4001-8001-000000000001/a1000007-0007-4007-8007-000000000007"
-					(reference "J_RAIL601")
+					(reference "J_RAIL501")
 					(unit 1)
 				)
@@
 		(in_pos_files yes)
 		(dnp no)
-		(property "Reference" "SW602"
+		(property "Reference" "SW502"
 			(at 62.23 59.69 0)
 			(show_name no)
@@
 			(project "AudioV2Case"
 				(path "/a1000001-0001-4001-8001-000000000001/a1000007-0007-4007-8007-000000000007"
-					(reference "SW602")
-					(unit 1)
-				)
+					(reference "SW502")
+					(unit 1)
+				)
