File: AudioV2/RelayBoard.kicad_sch (KiCad schematic)
At the start: 10 parts, among them K1 AZ850 CH1 audio, K2 AZ850 CH1 pwr, K3 AZ850 CH2 audio, K4 AZ850 CH2 pwr, K5 AZ850 CH3 audio, U1 MCP23017 addr0x20, U2 ULN2803A

Commit message: refactor(AudioV2): KiCad標準libへ置換（PGA2310/ULN2803/ENC） (#20)
- Audio:PGA2310PA, Transistor_Array:ULN2803A, Device:RotaryEncoder_Switch
- 配線スクリプトの PGA2310 ピン座標を標準シンボルに合わせて更新
- AudioV2.kicad_sym から PGA2310PA カスタム定義を削除
- PT2314 / DKMW20F-12 / CH224 モジュールは標準 lib 無しのため維持
- CIRCUIT_DESIGN.md に lib 方針表を追加

Co-authored-by: Cursor Agent <cursoragent@cursor.com>
Parts:
- removed U2: ULN2803A, symbol ULN2803A:ULN2803A
- added U2: ULN2803A, symbol Transistor_Array:ULN2803A
Changed lines of the file:
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@@
 	)
 	(symbol
-		(lib_id "ULN2803A:ULN2803A")
+		(lib_id "Transistor_Array:ULN2803A")
 		(at 88.9 50.8 0)
 		(unit 1)
