File: AudioV2/RelayBoard.kicad_sch (KiCad schematic)
At the start: 10 parts, among them K1 AZ850 CH1 audio, K2 AZ850 CH1 pwr, K3 AZ850 CH2 audio, K4 AZ850 CH2 pwr, K5 AZ850 CH3 audio, U1 MCP23017 addr0x20, U2 ULN2803A

Commit message: AudioV2: embed lib_symbols on all child schematics (KiCad 10)
ControlPanel, RelayBoard, and OutputStage had empty lib_symbols and
legacy symbol_inst without pin UUIDs — same pads-only issue as PowerModule.

- Extend sch_helpers: SYMBOL_SOURCES aliases, auto pin_numbers_for,
  BP5293 from Audio/, sanitize (type solid), sub-symbol rename on alias
- Regenerate all sheets via wire_circuit_design.py (power/control/relay/output)
- Fix Pico lib_id to MCU_Module:RaspberryPi_Pico (KiCad 10 name)
- SSD1306-128x64 embeds ER_OLEDM0.91 graphic under alias name
Connections:
- net 3V3: now also J_I2C.3 (Pin_3)
- net D_GND: now also J_I2C.4 (Pin_4)
- net I2C_SCL: now also J_I2C.2 (Pin_2)
- net I2C_SDA: now also J_I2C.1 (Pin_1)
- new net: K2.3, K4.10
- new net: K1.3, K3.10
- new net: K3.3, K5.10
- new net: K1.7, K5.1
