File: AudioV2/RelayBoard.kicad_sch (KiCad schematic)
At the start: 32 parts, among them K301 CH1 AUDIO, K302 CH1 POWER, K303 CH2 AUDIO, K304 CH2 POWER, K305 CH3 AUDIO, K306 CH3 POWER, K307 CH4 AUDIO, K308 CH4 POWER, K309 CH5 AUDIO, K310 CH5 POWER, U301 MCP23017, U302 ULN2803A, U303 ULN2803A

Commit message: AudioV2: 全シートを再アノテーション、参照変更を生成スクリプトと文書へ反映
KiCad で再アノテーションし、参照の重複と未付番を解消（計58件が変更）。

- ControlPanel の C201-C208 が PowerModule と重複していたため 5xx 台へ移動
- 未付番だった J_OLED を J_OLED501 に
- RelayBoard で U301(MCP23017) と U302(ULN2803A SET側) が入れ替わり
  → MCP23017 は U302、SET側 ULN が U301。接続トポロジは変更なし
- OutputStage が 6xx 台へ、AmpModule の C7xx/R7xx が L/R 対称に整列
- これにより netlist 出力時の「注釈のエラー」警告が解消

wire_circuit_design.py は旧参照をハードコードしており、再生成すると
アノテーションが巻き戻る状態だった。生成関数の行範囲でスコープを切って
86箇所を同時置換（U1 が PowerModule と ControlPanel で別部品のため）。
サンドボックスで再生成して実図と突き合わせ、AmpModule / ControlPanel /
RelayBoard / AudioV2Case は参照・値とも完全一致することを確認。
変更前後どちらの生成物も ERC 80件で、本修正は ERC 中立。

文書側も 7ファイル52箇所を更新。PARTS.md の「R705-708」等の範囲表記は
振り直し後に連番でなくなるため書き直し、OutputStage の表は SW_SP3T×2 の
実ピン（ネット名で照合）に合わせた。DECISIONS.md の D1/D2/D3 は決定ID、
旧 Audio/ SW101 参照は別プロジェクト指定のため意図的に据え置き。

既知の未同期: PowerModule はスクリプトが一世代古い（USB-C+CH224 の PD
前段を生成するが実図は PD モジュール外付け）。参照対応が一意に決まらない
ため F1→F201 / U1→U201 / U3→U202 / J202→J201 のみ修正し、コンデンサ群は
未着手。OutputStage の J_RAIL601 も生成対象外。

ERC は実図 54件で変化なし。

Co-Authored-By: Claude Opus 5 <noreply@anthropic.com>
Parts:
- renumbered U302 to U301, U301 to U302
Changed lines of the file:
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@@
 		(dnp no)
 		(fields_autoplaced yes)
-		(property "Reference" "U302"
+		(property "Reference" "U301"
 			(at 140.97 43.18 0)
 			(show_name no)
@@
 			(project "AudioV2Case"
 				(path "/a1000001-0001-4001-8001-000000000001/a1000004-0004-4004-8004-000000000004"
-					(reference "U302")
+					(reference "U301")
 					(unit 1)
 				)
 				(path "/a1000001-0001-4001-8001-000000000001/a1000005-0005-4005-8005-000000000005"
-					(reference "U402")
+					(reference "U401")
 					(unit 1)
 				)
@@
 		(in_pos_files yes)
 		(dnp no)
-		(property "Reference" "U301"
+		(property "Reference" "U302"
 			(at 88.9 73.66 0)
 			(show_name no)
@@
 			(project "AudioV2Case"
 				(path "/a1000001-0001-4001-8001-000000000001/a1000004-0004-4004-8004-000000000004"
-					(reference "U301")
+					(reference "U302")
 					(unit 1)
 				)
 				(path "/a1000001-0001-4001-8001-000000000001/a1000005-0005-4005-8005-000000000005"
-					(reference "U401")
-					(unit 1)
-				)
+					(reference "U402")
+					(unit 1)
+				)
