File: AudioV2/AmpBank.kicad_sch (KiCad schematic)
At the start: 8 parts

Commit message: AudioV2: D22/D23 を回路図へ実装（出力のみ MUX ＋ 入力 A案）
AmpChannel（1ch、これで両版共通になった）:
- TMUX7612 を外した。1 IC = 2ch なので per-channel シートには置けない
- 入力の 10µF 電解 ×2 と 220k プルダウン ×2 を撤去
- 結合C 100nF film -> 1uF film（P5.00 には入らないので 10mm ピッチの MKT へ）
- バイアス 1k -> 100k
- 階層ピン: SEL を削除、AMP_SEL_L/R -> OUT_L/OUT_R（ch ごとに独立）
- 部品 24 -> 19

AmpBank（切替段を引き受ける）:
- TMUX7612 ×5（U311-U315）と 100nF ×10（C311-C320）を追加
- 各 IC が 2ch を担当。S 側が ch ごと、D 側が共通バス
- 10 インスタンスのシートピンを新しい AmpChannel へ追随
- 出力ラベルを AMP_SEL_L/R -> CHn_OUT_L/R に改名（20件）

**書き起こし直さず、残す部分の手描き配線をそのまま置いた。** アンプ本体（AMP601 と
帰還・出力段）は座標も配線も無傷。sch_edit.py（新規）で部品単位の編集をする。

検証（ネットリスト）:
- /TONE_L に 10ch 分の結合Cが直付け（C602/C702/.../C1502）＝ブロードキャスト成立
- ch1 の + 入力 = {AMP601.3, C602.2, R601.2} ＝ A案そのもの
- /AMP_SEL_L に 5個の TMUX の D1/D3 が全部乗った（18 nodes）
- CHn_OUT_L = {結合C, 220k プルダウン, TMUX の S ピン}
- SEL_CHn = {TMUX の SEL 2本, MCP23017}
- 100k ×20 / 1uF film ×20 / 10µF は 3 個まで減（残りは別シート）
- 部品 362 個すべてユニーク（重複0）

ERC 56 -> 51。**AmpCh1〜10 は違反ゼロ**になった（各 ch にあった TMUX の
ground_pin_not_ground が、AmpBank の 5 個ぶんに集約されたため）。

途中で1件やらかして直した: TMUX7612 は元々 AmpChannel 側にいたので AmpBank の
lib_symbols に無く、入れ忘れたら **5個の TMUX がネットリストから丸ごと消えた**。
母板で娘基板コネクタを足したときと同じ罠。今回はネットリストの中身を見て気付いた。

⚠ build_ampchannel.py / build_ampbank.py は一度きりの移行スクリプトで冪等ではない。
変換済みのシートを食わせると書き込む前に落ちる（そう作ってある）。

⚠ 娘基板は 5ch×2枚（D19）なので、いまの「10ch 1枚・TMUX 5個」は最終形ではない。
1枚 5ch＝TMUX 3個 ×2枚への分割は別ステップ。

Co-Authored-By: Claude Opus 5 <noreply@anthropic.com>
Parts:
- added C311, C312, C313, C314, C315, C316, C317, C318, C319, C320: 100nF, Capacitor_SMD:C_1206_3216Metric_Pad1.33x1.80mm_HandSolder, symbol Device:C
- added U311, U312, U313, U314, U315: TMUX7612, Package_SO:TSSOP-16_4.4x5mm_P0.65mm, symbol AudioV2:TMUX7612
Connections:
- net +15V: now also C311.1, C313.1, C315.1, C317.1, C319.1, U311.13 (VDD), U312.13 (VDD), U313.13 (VDD), U314.13 (VDD), U315.13 (VDD)
- net -15V: now also C312.1, C314.1, C316.1, C318.1, C320.1, U311.4 (VSS), U312.4 (VSS), U313.4 (VSS), U314.4 (VSS), U315.4 (VSS)
- net AMP_SEL_L: now also U311.10 (D3), U311.2 (D1), U312.10 (D3), U312.2 (D1), U313.10 (D3), U313.2 (D1), U314.10 (D3), U314.2 (D1), U315.10 (D3), U315.2 (D1)
- net AMP_SEL_R: now also U311.15 (D2), U311.7 (D4), U312.15 (D2), U312.7 (D4), U313.15 (D2), U313.7 (D4), U314.15 (D2), U314.7 (D4), U315.15 (D2), U315.7 (D4)
- net A_GND: now also C311.2, C312.2, C313.2, C314.2, C315.2, C316.2, C317.2, C318.2, C319.2, C320.2, U311.5 (GND), U312.5 (GND), U313.5 (GND), U314.5 (GND), U315.5 (GND)
- net SEL_CH1: now also U311.1 (SEL1), U311.16 (SEL2)
- net SEL_CH10: now also U315.8 (SEL4), U315.9 (SEL3)
- net SEL_CH2: now also U311.8 (SEL4), U311.9 (SEL3)
- net SEL_CH3: now also U312.1 (SEL1), U312.16 (SEL2)
- net SEL_CH4: now also U312.8 (SEL4), U312.9 (SEL3)
- net SEL_CH5: now also U313.1 (SEL1), U313.16 (SEL2)
- net SEL_CH6: now also U313.8 (SEL4), U313.9 (SEL3)
- net SEL_CH7: now also U314.1 (SEL1), U314.16 (SEL2)
- net SEL_CH8: now also U314.8 (SEL4), U314.9 (SEL3)
- net SEL_CH9: now also U315.1 (SEL1), U315.16 (SEL2)
- new net CH10_OUT_L: U315.11 (S3)
- new net CH10_OUT_R: U315.6 (S4)
- new net CH1_OUT_L: U311.3 (S1)
- new net CH1_OUT_R: U311.14 (S2)
- new net CH2_OUT_L: U311.11 (S3)
- new net CH2_OUT_R: U311.6 (S4)
- new net CH3_OUT_L: U312.3 (S1)
- new net CH3_OUT_R: U312.14 (S2)
- new net CH4_OUT_L: U312.11 (S3)
- new net CH4_OUT_R: U312.6 (S4)
- new net CH5_OUT_L: U313.3 (S1)
- new net CH5_OUT_R: U313.14 (S2)
- new net CH6_OUT_L: U313.11 (S3)
- new net CH6_OUT_R: U313.6 (S4)
- new net CH7_OUT_L: U314.3 (S1)
- new net CH7_OUT_R: U314.14 (S2)
- new net CH8_OUT_L: U314.11 (S3)
- new net CH8_OUT_R: U314.6 (S4)
- new net CH9_OUT_L: U315.3 (S1)
- new net CH9_OUT_R: U315.14 (S2)
- no-connect marks 10 -> 15
Other:
- sheet AmpCh1 ports: added OUT_L, OUT_R; removed AMP_SEL_L, AMP_SEL_R, SEL
- sheet AmpCh10 ports: added OUT_L, OUT_R; removed AMP_SEL_L, AMP_SEL_R, SEL
- sheet AmpCh2 ports: added OUT_L, OUT_R; removed AMP_SEL_L, AMP_SEL_R, SEL
- sheet AmpCh3 ports: added OUT_L, OUT_R; removed AMP_SEL_L, AMP_SEL_R, SEL
- sheet AmpCh4 ports: added OUT_L, OUT_R; removed AMP_SEL_L, AMP_SEL_R, SEL
- sheet AmpCh5 ports: added OUT_L, OUT_R; removed AMP_SEL_L, AMP_SEL_R, SEL
- sheet AmpCh6 ports: added OUT_L, OUT_R; removed AMP_SEL_L, AMP_SEL_R, SEL
- sheet AmpCh7 ports: added OUT_L, OUT_R; removed AMP_SEL_L, AMP_SEL_R, SEL
- sheet AmpCh8 ports: added OUT_L, OUT_R; removed AMP_SEL_L, AMP_SEL_R, SEL
- sheet AmpCh9 ports: added OUT_L, OUT_R; removed AMP_SEL_L, AMP_SEL_R, SEL
