File: AudioV2/AmpChannel.kicad_sch (KiCad schematic)
At the start: 24 parts, among them U601 TMUX7612

Commit message: AudioV2: 再アノテーション（PowerModule の DC-DC を U201 へ戻す）
ユーザーが KiCad で再アノテーション。DC-DC 差し替えの際に U203 へ動いていた
参照を U201 に戻した。副次的に AmpChannel 内の参照割り当ても入れ替わった
（集合は同じで 320 箇所の再割り当て。例: 220k は R603/R608/R611/R612 ->
R603/R605/R609/R611）。

Description はシンボルのプロパティなので部品に付いたまま動いており、
入出力プルダウンの L/R 対応は保たれている（BOM の 220k 行で確認）。
文書側はネット名・機能名で書いてあるため影響を受けない
（SOURCE_OF_TRUTH.md 3 の方針どおり）。

検証:
- check_sexpr 9ファイル / 問題0
- ネットリストで DC-DC 全6ピンが機能どおり:
  1=+Vin -> Net-(U201-+Vin)、2=-Vin -> /PD_GND、3=CTRL -> 未接続、
  4=-Vout -> /-15V、5=COM -> /A_GND、6=+Vout -> /+15V（不一致 0 件）
- AmpChannel の出力プルダウン 20/20 が OUT_L/OUT_R -> A_GND
- ERC 60件で変化なし
- drift 生成コード所有 2/2 一致
- PARTS.md の BOM を再生成（--check rc=0）

Co-Authored-By: Claude Opus 5 <noreply@anthropic.com>
Parts:
- renumbered C602 to C601, C601 to C602, C605 to C604, C604 to C605, C608 to C607, C607 to C608, R604 to R601, R611 to R603, R605 to R604, R603 to R605, R601 to R606, R609 to R607, R607 to R608, R612 to R609, R608 to R611, R606 to R612

Commit message: AudioV2: D22/D23 を回路図へ実装（出力のみ MUX ＋ 入力 A案）
AmpChannel（1ch、これで両版共通になった）:
- TMUX7612 を外した。1 IC = 2ch なので per-channel シートには置けない
- 入力の 10µF 電解 ×2 と 220k プルダウン ×2 を撤去
- 結合C 100nF film -> 1uF film（P5.00 には入らないので 10mm ピッチの MKT へ）
- バイアス 1k -> 100k
- 階層ピン: SEL を削除、AMP_SEL_L/R -> OUT_L/OUT_R（ch ごとに独立）
- 部品 24 -> 19

AmpBank（切替段を引き受ける）:
- TMUX7612 ×5（U311-U315）と 100nF ×10（C311-C320）を追加
- 各 IC が 2ch を担当。S 側が ch ごと、D 側が共通バス
- 10 インスタンスのシートピンを新しい AmpChannel へ追随
- 出力ラベルを AMP_SEL_L/R -> CHn_OUT_L/R に改名（20件）

**書き起こし直さず、残す部分の手描き配線をそのまま置いた。** アンプ本体（AMP601 と
帰還・出力段）は座標も配線も無傷。sch_edit.py（新規）で部品単位の編集をする。

検証（ネットリスト）:
- /TONE_L に 10ch 分の結合Cが直付け（C602/C702/.../C1502）＝ブロードキャスト成立
- ch1 の + 入力 = {AMP601.3, C602.2, R601.2} ＝ A案そのもの
- /AMP_SEL_L に 5個の TMUX の D1/D3 が全部乗った（18 nodes）
- CHn_OUT_L = {結合C, 220k プルダウン, TMUX の S ピン}
- SEL_CHn = {TMUX の SEL 2本, MCP23017}
- 100k ×20 / 1uF film ×20 / 10µF は 3 個まで減（残りは別シート）
- 部品 362 個すべてユニーク（重複0）

ERC 56 -> 51。**AmpCh1〜10 は違反ゼロ**になった（各 ch にあった TMUX の
ground_pin_not_ground が、AmpBank の 5 個ぶんに集約されたため）。

途中で1件やらかして直した: TMUX7612 は元々 AmpChannel 側にいたので AmpBank の
lib_symbols に無く、入れ忘れたら **5個の TMUX がネットリストから丸ごと消えた**。
母板で娘基板コネクタを足したときと同じ罠。今回はネットリストの中身を見て気付いた。

⚠ build_ampchannel.py / build_ampbank.py は一度きりの移行スクリプトで冪等ではない。
変換済みのシートを食わせると書き込む前に落ちる（そう作ってある）。

⚠ 娘基板は 5ch×2枚（D19）なので、いまの「10ch 1枚・TMUX 5個」は最終形ではない。
1枚 5ch＝TMUX 3個 ×2枚への分割は別ステップ。

Co-Authored-By: Claude Opus 5 <noreply@anthropic.com>
Parts:
- removed C603, C606: 10uF, Capacitor_THT:CP_Radial_D5.0mm_P2.00mm, symbol Device:C_Polarized
- removed R605, R611: 220k, Resistor_SMD:R_1206_3216Metric_Pad1.30x1.75mm_HandSolder, symbol Device:R
- removed U601: TMUX7612, Package_SO:TSSOP-16_4.4x5mm_P0.65mm, symbol AudioV2:TMUX7612
- C602, C605: value 100nF film -> 1uF film; footprint Capacitor_THT:C_Rect_L7.2mm_W2.5mm_P5.00mm_FKS2_FKP2_MKS2_MKP2 -> Capacitor_THT:C_Rect_L11.0mm_W4.2mm_P10.00mm_MKT
- R601, R607: value 1k -> 100k
Connections:
- net IN_L is gone; now on net TONE_L: C602.1
- net IN_R is gone; now on net TONE_R: C605.1
- no-connect marks 1 -> 0
