File: AudioV2/AmpChannel.kicad_sch (KiCad schematic)
At the start: 19 parts

Commit message: AudioV2: TMUX を 270°（ピン1側=CH1）にし、AmpChannel のスイッチ用デカップを外す
S=各ch出力・D=AMP_SEL に戻し、CH1 配線途中の PCB も取り込む。C607/C610 は D22 の残りなのでシートから削除した。

Co-authored-by: Cursor <cursoragent@cursor.com>
Parts:
- removed C607, C610: 100nF, Capacitor_SMD:C_1206_3216Metric_Pad1.33x1.80mm_HandSolder, symbol Device:C

Commit message: AudioV2: Amp カップリングフィルムを TDK B32529 系統の FP に揃えた
入力1µFは P5/W4.5、出力2.2µFは P5/W7.2。旧 P10 / W2.5 の誤りを直し、PCB も同期。

Co-authored-by: Cursor <cursoragent@cursor.com>
Parts:
- C601, C604: footprint Capacitor_THT:C_Rect_L7.2mm_W2.5mm_P5.00mm_FKS2_FKP2_MKS2_MKP2 -> Capacitor_THT:C_Rect_L7.2mm_W7.2mm_P5.00mm_FKS2_FKP2_MKS2_MKP2
- C602, C605: footprint Capacitor_THT:C_Rect_L11.0mm_W4.2mm_P10.00mm_MKT -> Capacitor_THT:C_Rect_L7.2mm_W4.5mm_P5.00mm_FKS2_FKP2_MKS2_MKP2
Changed lines of the file:
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@@
 			)
 		)
-		(property "Footprint" "Capacitor_THT:C_Rect_L11.0mm_W4.2mm_P10.00mm_MKT"
+		(property "Footprint" "Capacitor_THT:C_Rect_L7.2mm_W4.5mm_P5.00mm_FKS2_FKP2_MKS2_MKP2"
 			(at -52.07 140.97 0)
 			(hide yes)
@@
 			)
 		)
-		(property "Footprint" "Capacitor_THT:C_Rect_L7.2mm_W2.5mm_P5.00mm_FKS2_FKP2_MKS2_MKP2"
+		(property "Footprint" "Capacitor_THT:C_Rect_L7.2mm_W7.2mm_P5.00mm_FKS2_FKP2_MKS2_MKP2"
 			(at -25.4 1.27 0)
 			(hide yes)
@@
 			)
 		)
-		(property "Footprint" "Capacitor_THT:C_Rect_L11.0mm_W4.2mm_P10.00mm_MKT"
+		(property "Footprint" "Capacitor_THT:C_Rect_L7.2mm_W4.5mm_P5.00mm_FKS2_FKP2_MKS2_MKP2"
 			(at 11.43 104.14 0)
 			(hide yes)
@@
 			)
 		)
-		(property "Footprint" "Capacitor_THT:C_Rect_L7.2mm_W2.5mm_P5.00mm_FKS2_FKP2_MKS2_MKP2"
+		(property "Footprint" "Capacitor_THT:C_Rect_L7.2mm_W7.2mm_P5.00mm_FKS2_FKP2_MKS2_MKP2"
 			(at 254 177.8 0)
 			(hide yes)

Commit message: AudioV2: 娘を縮小し AMP_SEL を裏へ、A_GND ステッチと Rf/Rg を 0805 に
表の AMP_SEL 幹線を裏本線にし、TMUX デカップと電源幅をピン周りで寄せた。A_GND ビアを TMUX / SEL 脇に足す。比較用 20k は 0805。

Co-authored-by: Cursor <cursoragent@cursor.com>
Parts:
- R604, R606, R610, R612: footprint Resistor_SMD:R_1206_3216Metric_Pad1.30x1.75mm_HandSolder -> Resistor_SMD:R_0805_2012Metric_Pad1.20x1.40mm_HandSolder
Changed lines of the file:
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@@
 			)
 		)
-		(property "Footprint" "Resistor_SMD:R_1206_3216Metric_Pad1.30x1.75mm_HandSolder"
+		(property "Footprint" "Resistor_SMD:R_0805_2012Metric_Pad1.20x1.40mm_HandSolder"
 			(at -27.94 -26.67 0)
 			(hide yes)
@@
 			)
 		)
-		(property "Footprint" "Resistor_SMD:R_1206_3216Metric_Pad1.30x1.75mm_HandSolder"
+		(property "Footprint" "Resistor_SMD:R_0805_2012Metric_Pad1.20x1.40mm_HandSolder"
 			(at 200.66 82.55 0)
 			(hide yes)
@@
 			)
 		)
-		(property "Footprint" "Resistor_SMD:R_1206_3216Metric_Pad1.30x1.75mm_HandSolder"
+		(property "Footprint" "Resistor_SMD:R_0805_2012Metric_Pad1.20x1.40mm_HandSolder"
 			(at -26.67 1.27 0)
 			(hide yes)
@@
 			)
 		)
-		(property "Footprint" "Resistor_SMD:R_1206_3216Metric_Pad1.30x1.75mm_HandSolder"
+		(property "Footprint" "Resistor_SMD:R_0805_2012Metric_Pad1.20x1.40mm_HandSolder"
 			(at -22.86 -10.16 0)
 			(hide yes)
