File: AudioV2/AmpChannel.kicad_sch (KiCad schematic)
At the start: 17 parts

Commit message: AmpChannel Rf/Rg を 0.1% に確定し、PARTS に調達クラスを書く
issue #38: PRECISION/MATCH/SPEC 方針を PARTS.md §0c に反映。
ゲイン抵抗は図上 Value を 20k 0.1% にし D-i を閉じる。
フィルムは既存 B32529/P5 のまま MATCH（LCR 選別）。BOM を再生成。

Co-authored-by: m_arino <indare@users.noreply.github.com>
Parts:
- R604, R606, R610, R612: value 20k -> 20k 0.1%
Changed lines of the file:
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@@
 			)
 		)
-		(property "Value" "20k"
+		(property "Value" "20k 0.1%"
 			(at 74.93 83.82 0)
 			(show_name no)
@@
 			)
 		)
-		(property "Value" "20k"
+		(property "Value" "20k 0.1%"
 			(at 88.9 52.07 90)
 			(show_name no)
@@
 			)
 		)
-		(property "Description" "L feedback Rf; default 20k = GAIN 2"
+		(property "Description" "L feedback Rf; default 20k 0.1% = GAIN 2"
 			(at 200.66 82.55 0)
 			(hide yes)
@@
 			)
 		)
-		(property "Value" "20k"
+		(property "Value" "20k 0.1%"
 			(at 76.2 48.26 0)
 			(show_name no)
@@
 			)
 		)
-		(property "Value" "20k"
+		(property "Value" "20k 0.1%"
 			(at 88.9 88.9 90)
 			(show_name no)
@@
 			)
 		)
-		(property "Description" "R feedback Rf; default 20k = GAIN 2"
+		(property "Description" "R feedback Rf; default 20k 0.1% = GAIN 2"
 			(at -22.86 -10.16 0)
 			(hide yes)
