File: AudioV2/MotherBoard.kicad_sch (KiCad schematic)
At the start: 46 parts, among them J201 +15/-15/A_GND out, J202 PD module in (1=GND 2=+12V), SW402 PWR SW, SW501 DEST L (PHONE/MUTE/LINE), SW502 DEST R (PHONE/MUTE/LINE), U201 REC10K-2415DAW/H2, U202 L7809CV +9V, U402 PT2314E, U403 BP5293-50 +5V

Commit message: AudioV2: 外部入力端子台を入れ、ENC の名前と UI の割り込みを直した（ERC 17 -> 11）
査読の確認で出た3件。ERC は 17 -> 11 件になり、残る11件は全部「宣言済みの型」に
収まった（内訳は CLAUDE.md の表）。

1. 外部入力 L/R の端子台 J_IN401 を追加

   DECISIONS §11.3（基板間リンク）は「外部入力 L/R｜端子台 2〜3P」で確定と
   書いてあるのに symbol が無く、COMMON_L / COMMON_R が1ピン（結合Cの片足だけ）
   だった。出力側は J_HP501 / J_LINE501 が実在するのに入力だけ抜けていた。
   このまま PCB を起こすと入力パッドが空かない。

       J_IN401 → COMMON_L →C406→ PT_LIN → PT2314E → PT_OUT_L →C405→ TONE_L → …

   1=L / 2=A_GND / 3=R。L と R の間に必ず GND が挟まる並び。フットプリントは
   J_RAIL501 と同じ Phoenix MKDS-1,5 3P（横）。
   これで isolated_pin_label が 9 -> 1 件になった（残る1件は DEST_SENSE_MUTE_NC で、
   ミュート位置なので意図的に開放）。

2. ENC1602 の Value を ENC_VOL -> ENC_BASS

   確定は CH / BASS / TREBLE（DECISIONS §2「ENC 割当（確定）」・§10 の表・
   CIRCUIT_DESIGN.md）。「音量をエンコーダー化」は 2026-08-30 に撤回済み。
   そもそも PT2314E のボリューム段は LOUT/ROUT -> LIN/RIN のインサートで
   飛ばしているので、VOL のエンコーダには制御対象が無い。

3. U1610（UI 0x22）の INTA(20) / INTB(19) を Pico の GP16 / GP17 へ

   エンコーダ3個が MCP23017 経由なので、割り込みが無いとポーリングしかない。
   I²C は PT2314E の VDD 9V（L7809CV）× MCU 3.3V により Standard 100 kbit/s 止まり
   （DS p.7 の DATA RATE 表）で、2.42″ OLED が 128x64 なら1フレーム 1024 バイト
   ≈ 92 ms。取りこぼさない周期でエンコーダを叩くとバス占有が単独で 45% になり
   同居できない。

   ⚠ 2本引いたのは MIRROR ビット頼みにしないため。ENC1/2 の A/B/SW と ENC3 の A/B は
     PortA(21-28) だが ENC3_SW だけ PortB(pin1) にいるので、INTA だけだと
     IOCON.MIRROR=1 が前提になる。ADC 兼用の GP26-28 は空けたまま。

Pico の AGND(33) は開放のまま戻した（いったん D_GND へ結んだが撤回）

   lib シンボル MCU_Module:RaspberryPi_Pico は pin3 GND と pin33 AGND を
   どちらも power_out と型付けしている（他の GND 6本は passive）。モジュール側が
   それぞれをグランド源として出しているという宣言なので、外で結ぶと power_out
   同士の衝突になり、実際 pin_to_pin エラーが出た。AGND は Pico 基板上で
   グランドに繋がっている前提でよい。

PARTS.md は再生成した（gen_parts_bom.py）

   生成ブロックが 部品総数 368 / Footprint 未設定 44 の時代のまま止まっていたので、
   このセッションで埋めた footprint 全部と R401 / C1645 / F1603 / J_IN401、
   削除した R407・R412-415 が一気に反映された。
   ⚠ U402 の Role にあった「SOP-28 300 mil。LCSC C90034」は 2fbad17 で
     生成ブロックの中を手編集していたもので、再生成で消えた（マーカー内は毎回
     まるごと差し替わるので当然）。回路図側の Description プロパティに入れ直した。
   §5 の「Footprint 未設定の部品」は 0 個になったので残件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
Parts:
- added J_IN401: AUDIO IN L/R, TerminalBlock_Phoenix:TerminalBlock_Phoenix_MKDS-1,5-3-5.08_1x03_P5.08mm_Horizontal, symbol Connector:Screw_Terminal_01x03
Connections:
- net A_GND: now also J_IN401.2 (Pin_2)
- net COMMON_L: now also J_IN401.1 (Pin_1)
- net COMMON_R: now also J_IN401.3 (Pin_3)
Changed lines of the file:
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@@
+	)
+	(symbol
+		(lib_id "Connector:Screw_Terminal_01x03")
+		(at 431.8 118.11 0)
+		(unit 1)
+		(body_style 1)
+		(exclude_from_sim no)
+		(in_bom yes)
+		(on_board yes)
+		(in_pos_files yes)
+		(dnp no)
+		(property "Reference" "J_IN401"
+			(at 431.8 109.22 0)
+			(show_name no)
+			(do_not_autoplace no)
+			(effects
+				(font
+					(size 1.27 1.27)
+				)
+			)
+		)
+		(property "Value" "AUDIO IN L/R"
+			(at 431.8 111.76 0)
+			(show_name no)
+			(do_not_autoplace no)
+			(effects
+				(font
+					(size 1.27 1.27)
+				)
+			)
+		)
+		(property "Footprint" "TerminalBlock_Phoenix:TerminalBlock_Phoenix_MKDS-1,5-3-5.08_1x03_P5.08mm_Horizontal"
+			(at 431.8 118.11 0)
+			(hide yes)
+			(show_name no)
+			(do_not_autoplace no)
+			(effects
+				(font
+					(size 1.27 1.27)
+				)
+			)
+		)
+		(property "Datasheet" ""
+			(at 431.8 118.11 0)
+			(hide yes)
+			(show_name no)
+			(do_not_autoplace no)
+			(effects
+				(font
+					(size 1.27 1.27)
+				)
+			)
+		)
+		(property "Description" "箱の外部音声入力。1=L / 2=A_GND / 3=R。ここから結合C経由で PT2314E の LIN/RIN へ入る（セレクタとボリューム段は LOUT/ROUT->LIN/RIN のインサートで飛ばしている）。L と R の間に GND を挟むため 3P にした。"
+			(at 431.8 118.11 0)
+			(hide yes)
+			(show_name no)
+			(do_not_autoplace no)
+			(effects
+				(font
+					(size 1.27 1.27)
+				)
+			)
+		)
+		(pin "1"
+		)
+		(pin "2"
+		)
+		(pin "3"
+		)
+		(instances
+			(project "AudioV2Case"
+				(path "/a1000001-0001-4001-8001-000000000001/a1000012-0012-4012-8012-000000000012"
+					(reference "J_IN401")
+					(unit 1)
+				)
+			)
+		)
+	)
+	(label "COMMON_L"
+		(at 426.72 115.57 180)
+		(effects
+			(font
+				(size 1.27 1.27)
+			)
+			(justify right bottom)
+		)
+	)
+	(label "A_GND"
+		(at 426.72 118.11 180)
+		(effects
+			(font
+				(size 1.27 1.27)
+			)
+			(justify right bottom)
+		)
+	)
+	(label "COMMON_R"
+		(at 426.72 120.65 180)
+		(effects
+			(font
+				(size 1.27 1.27)
+			)
+			(justify right bottom)
+		)
 	)
 	(symbol
@@
 			)
 		)
-		(property "Description" ""
-			(at 355.6 0 0)
-			(hide yes)
+		(property "Description" "SOP-28 300 mil（表面実装。無印 PT2314 の DIP 版は入手不可）。LCSC C90034。トーン段だけ使う — 入力セレクタとボリューム段は LOUT/ROUT -> LIN/RIN の インサート点で飛ばしていて、未使用12ピンには no_connect を立ててある。"
+			(at 355.6 0 0)
+			(hide yes)
