File: AudioV2/MeasureControl.kicad_sch (KiCad schematic)
At the start: 105 parts, among them J1601 AUDIO, J1602 V_IN, J1603 15_V_IN, SW1601 DEST sense (3PDT 3rd pole, sa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, U1601 OPA1656, U1602 OPA1656, U1603 LT1763-3.3, U1604 MBC2596-01, U1605 TPS3307-33, U1606 LT1763-5, U1607 BP5293-50, U1608 OPA1656, U1609 XC8107AC20MR-G, U1610 MCP23017 (UI 0x22), Y1601 ASFL1-12.288MHZ-EC-T

Commit message: AudioV2: U1604（MBC2596 非絶縁バック）を削除。ADC の LDO を +15V 直結にした
## なぜ消したか（電源が足りない話とは無関係）

1. 1.2 kHz スパーの最有力容疑者（軽負荷パルススキップ）。
   Audio/MeasurementADC_BRINGUP.md が「未検証・出力に数百Ω足すだけで切り分けできる」と
   書いていた当のもの。部品ごと消えるので切り分け自体が要らなくなった
2. ADC_GND を PD_GND に溶接している唯一の部品だった。DECISIONS 自身が
   「リレーのパルス電流が結合チェーン全体、つまり ADC のアナログ星点を通っていた」と
   名指ししていたチェーン
     A_GND ─NT1601─ ADC_GND ─**U1604 の内部**─ PD_GND ─NT1602─ D_GND
   の中央がこれ

## 変更

  ADC の LDO 入力  PD_12V_SW →F1603→ U1604(バック) → 中間レール 約6.8V
                   ↓
                   +15V 直結

  消した   U1604 / C1644(47uF) / F1603(PPTC 0.15A) / #FLG1603
  足した   NT1603（A_GND <-> D_GND）/ #FLG1604（ADC_GND の PWR_FLAG）
  変えた   C1606・C1619  10uF 16V X7R/1206 -> 10uF 50V X7R/1210
           （15V レールに 16V 品は使えない）
  部品数   372 -> 370

LT1763 は規定入力 1.8-20V、IN/SHDN 絶対最大 ±20V、入出力差 ±20V（ADI_LT1763.pdf）。
15V 入力は規定内。リニア損失は U1603 0.41W / U1606 0.45W、SO-8 の θJA 70°C/W で
温度上昇 29 / 31 °C。

## NT1603 は A6/D28 に反しない

A6/D28 の「足す NetTie は無い」は、A_GND↔D_GND の結合が U1604 の内部を通っている
前提で書かれている。U1604 を消すとグランドが2島に割れる:

    A_GND + ADC_GND   /   PD_GND + D_GND + GND_COIL

TMUX7612 の SEL しきい値は自分の GND ピン(= A_GND)基準（VIH 1.3V / VIL 0.8V、
絶対最大 VSEL -0.5V、TI_TMUX7612.pdf）なのに、駆動は D_GND 基準の MCP23017。
橋が無いと ESD クランプが事実上の結合点になる。

**A_GND↔D_GND の結合点の数は 1 のまま。** 場所が「スイッチングレギュレータの内部
（選べない）」から「置き場所を選べる NetTie」に変わっただけで、趣旨は保たれている。

木は 5 ノード・4 辺のまま（閉路なし）:
    GND_COIL ─NT101─ D_GND ─NT1602─ PD_GND
                       └───NT1603─── A_GND ─NT1601─ ADC_GND

⚠ PCB では NT1601 と NT1603 を隣に置くこと。I2S の帰り（D_GND → A_GND → ADC_GND）が
  3ホップ -> 2ホップに減ったが、2つの NetTie が離れるとその間の A_GND 銅箔が
  そのままループ面積になる。

## 途中で踏んだもの

- 中間レールに +15V というラベルを置いたが、MeasureControl 側のこのレールの名前は
  +15V_A。別ネットになり power_pin_not_driven が2件出て気づいた
- U1604.4(OUT-) が ADC_GND を駆動する唯一の power_output だったので、消すと
  A1601.14(GND, Power input) に power_pin_not_driven が出る。ADC_GND は NT1601 で
  A_GND に結合しているが KiCad の NetTie は passive なので ERC に駆動が伝わらない。
  設計内の #FLG1602 と同じ形で PWR_FLAG を置いた

## ⚠ 未決: ADC 枝の保護が無くなった

F1603（PPTC 0.15A）は U1604 専用だったので一緒に消えた。いま ADC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
Parts:
- removed C1644: 47uF 35V, Capacitor_THT:CP_Radial_D8.0mm_P3.50mm, symbol Device:C_Polarized
- removed F1603: PPTC 0.15A hold, Resistor_THT:R_Axial_DIN0411_L9.9mm_D3.6mm_P12.70mm_Horizontal, symbol Device:Fuse
- removed U1604: MBC2596-01, Library:MBC2596-01_TAEJIN_43x21mm, symbol MeasurementADC_Extras:MBC2596-01
- added NT1603: A_GND-D_GND, NetTie:NetTie-2_SMD_Pad0.5mm, symbol Device:NetTie_2
- C1606, C1619: value 10uF 16V X7R -> 10uF 50V X7R; footprint Capacitor_SMD:C_1206_3216Metric_Pad1.33x1.80mm_HandSolder -> Capacitor_SMD:C_1210_3225Metric_Pad1.33x2.70mm_HandSolder
Connections:
- net +15V_A: now also C1605.1, C1606.1, C1618.1, C1619.1, U1603.5 (SHDN), U1603.8 (IN), U1606.8 (IN)
- net A_GND: now also NT1603.1
- net D_GND: now also NT1603.2

Commit message: AudioV2: レビュー指摘 3・4 を反映（OCP/容量の訂正、旧注釈10個の掃除、J_RAIL501 の Value）
レビューコメント（電源差し替えと U1604 削除の主経路は成立、残る4点は方針/文書/配線手順）
のうち、判断を要しない 3 と 4 を直した。1 と 2 は NOW.md に未判断として置いた。

## 3. DECISIONS の記述訂正（自分の誤り2件）

- U201 の OCP を「150% Io」と書いていたが、それは REC10K の値。
  REC20K-2415DZ は **225% of rated IOUT**（nom. VIN=48VDC、Recom_REC20K-Z_Rev3-2025.pdf）
- 「+15V/-15V とも 259.8µF」は差し替え時点の値。同日の U1604 削除で C1606/C1619
  （計 20.2µF）が中間レールから +15V に載り、いまは **+15V 280.0µF / -15V 259.8µF**。
  REC10K の Cout ±270µF に対して 96% → **103.7% で上限超え**。REC20K の理由②は
  差し替え後にさらに強まった

## 4. MeasureControl の旧注釈を掃除

26 個の text のうち 10 個が 2026-09-01 の再アノテーション前の designator のままだった。
うち3つは内容が現物と食い違っていた:

- [3][4] 電源系の注釈が **削除済みの U1604(MBC2596) の構成を今も説明**していた
  → ⑥-A 後の実配線（ADC の LDO は +15V 直結）に書き直し
- [11] GND の注釈が **NetTie の対応を現物と逆に**書いていた
  （旧「NT702=A_GND─ADC_GND / NT701=ADC_GND_IN─D_GND」→ 現物は NT1601 / NT1602）
  → NT1603 の新設と「3つを近接させる」も足した

残り7個は designator の置換のみ（回路図で1個ずつ対応を確定してから）:
  U704→U1607 U706→U1603 U707→U1606 U708→U1609 U709→U1605
  Y701→Y1601 D701→D1601 A701→A1601
  R717→R1620 R718→R1604 R719→R1611 R720→R1605
  C745→C1614（TPS3307 VDD） C740→C1633（XC8107 CIN） C739→C1631（XC8107 CL）
  NT701→NT1602 NT702→NT1601

同座標・同文の重複 2 組（[13][14] / [15][16]）を1つずつに。残る旧 designator は 0。

## J_RAIL501 の Value

「RAIL IN」→「AMP_SEL OUT」。実ネットは AMP_SEL_L / A_GND / AMP_SEL_R で、
娘基板がスロット直結になる前の名残だった。Description は前回直してある。
Value 変更なので PARTS.md を再生成した（BOM の行が変わる。netlist は変わらない）。

## 1・2 は NOW.md に未判断として置いた

1. ADC 枝の PPTC（旧 F1603）を戻すか — 既に記載あり
2. 計測側の電源端子 J1602/J1603 を残すか — **基板を分けるかの判断の下流**。
   分けないなら J1601 も含めて3個とも不要。分けるなら **J1603 のピン並びが J201 と逆**
   （J201=+15/GND/−15、J1603=−15/GND/+15。ピン番号どおりに繋ぐとレールが入れ替わる）。
   J1602 は F1601 が端子の外側に付いた行き止まりで、⑥-A 後は U1607 1個の 12V 入口

## 検証

  check_sexpr.py -q AudioV2   13 ファイル / 問題 0
  kicad-run.sh erc            11 件（変化なし）
  kicad-run.sh netlist        部品 370 個・重複 0・footprint 未設定 0（変化なし）
  sch_import --roundtrip      6/6 OK
  再生成の冪等性               バイト一致
  gen_parts_bom.py --check    OK

Co-Authored-By: Claude Fabl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
Other:
- note added: "A3 Pico2 横置き: 南列 1-20 西→東 / 北列 21-40 東→西。VSYS=+5V_D via D1601 ショットキ, GND=D_GND | GP0=ADC_DATA GP1=ADC_BCK GP2=ADC_LRCK | GP3/GP4=NC(旧 LCD SPI) | GP5=LCD_CS GP6=LCD_DC GP7=LCD_RST GP8=LCD_EN | GP9=MCLK_SENSE (R1605 1k, 入力専用) | GP10=TP_SDA GP11=TP_SCL GP12=TP_INT GP13=TP_RST | GP15=ADC_nMR (TPS3307 ~MR, OD, H は駆動しない) | GP18=LCD_SCK GP19=LCD_MOSI (SPI0)"
- note added: "GND: NT1601=A_GND─ADC_GND（A1601 近傍・アナログ星点）。NT1602=PD_GND─D_GND（PD 入口）。NT1603=A_GND─D_GND（2026-09-07 新設。U1604 削除で失われた A_GND↔D_GND の橋を明示化）。⚠ NT1601 / NT1602 / NT1603 は PCB で近接させる（1点アース。I2S の帰り・U403 の帰路・U201 の Ciso 経由 CM が全部ここを通る）。Pico/LCD は D_GND のみ。D_GND は太く短く、アナログ入力から離す。"
- note added: "GP9=MCLK_SENSE は R1605 1k 経由の入力専用。出力にすると Y1601 と衝突して SCKI が化ける。"
- note added: "POWER/DIGITAL（2026-09-07）: +15V → U1603(+3V3_A) と U1606(+5V_A, SHDN=+3V3_A)。旧 U1604(MBC2596) は削除。U1607=+5V_D（PD_12V_MEAS から）。D1601 ショットキ: +5V_D → Pico VSYS（USB 逆流止め）。Y1601 12.288MHz → R1604 33Ω → SCKI。R1605 1k → MCLK_SENSE(GP9、監視のみ。⚠ ファームは未使用)。U1609 XC8107 → LCD_VCC。U1605 TPS3307 監視。"
- note added: "U1603 LT1763-3.3 (+3V3_A). Fixed LDO; SHDN tied for always-on or as designed. Local CIN/COUT."
- note added: "U1605=TPS3307-33D SO-8: SENSE1=+5V_A (4.55V) SENSE2=+3V3_A (2.93V) SENSE3=VDD; VDD=+3V3_A C1614 100nF; ~RESET PP -> ADC_nRST + R1611; GP15 OD -> ~MR (do not drive H); RESET pin NC; 200ms delay. Replaces TPS3808G33/G50 SOT-23-6."
- note added: "U1606 EN=+3V3_A (3V3-first). AbsMax VCC-VDD protection."
- note added: "U1609 XC8107AC20MR-G ロードスイッチ: LCD_EN High=ON / Low・Hi-Z=OFF（Active High, VCEH 1.5V min → Pico 3.3V で直接駆動可）。R1620 100k=CE プルダウンで起動時 OFF。初号は常時 ON 可。OFF 運用時は SPI/タッチを Low/Hi-Z に。ソフトスタート 0.6ms typ・短絡/逆流/過熱/UVLO 保護内蔵。C1633=CIN, C1631=CL は各 10uF/3216 を IC 直近へ。FLG は未使用（NC）。"
- note added: "電源: USB VBUS → Pico 内部ショットキ → VSYS。D1601 が +5V_D への逆流を止めるので、USB だけ挿すと Pico は動き LCD は消える。VBUS(pin40) は NC。"
- note added: "電源系（2026-09-07 U1604 削除後） PD_12V_SW ─F1602─ PD_12V_MEAS ─ U1607 BP5293-50 → +5V_D（Pico/LCD。GND=D_GND、CIN=C1645） +15V ─────────────────────── U1603 LT1763-3.3 → +3V3_A（ADC。GND=ADC_GND） +15V ─────────────────────── U1606 LT1763-5 → +5V_A （ADC。SHDN=+3V3_A で 3V3 先行） 旧 U1604（MBC2596 12V→6.6V 非絶縁バック）と F1603/C1644 は削除。ADC の LDO は +15V 直結。"
- note removed: "A3 Pico2 横置き: 南列 1-20 西→東 / 北列 21-40 東→西。VSYS=+5V_D via D701 ショットキ, GND=D_GND | GP0=ADC_DATA GP1=ADC_BCK GP2=ADC_LRCK | GP3/GP4=NC(旧 LCD SPI) | GP5=LCD_CS GP6=LCD_DC GP7=LCD_RST GP8=LCD_EN | GP9=MCLK_SENSE (R720 1k, 入力専用) | GP10=TP_SDA GP11=TP_SCL GP12=TP_INT GP13=TP_RST | GP15=ADC_nMR (TPS3307 ~MR, OD, H は駆動しない) | GP18=LCD_SCK GP19=LCD_MOSI (SPI0)"
- note removed: "ADC_V_IN ├─ BP5293-50 → +5V_D（Pico/LCD） └─ MBC2596 → ~6.6V ├─ LT1763-5 → +5V_A （ADC） └─ LT1763-3.3 → +3V3_A （ADC）"
- note removed: "GND: NT702=A_GND─ADC_GND（A701近傍・アナログ星点）。NT701=ADC_GND_IN─D_GND（PD入口）。Pico/LCD は D_GND のみ。D_GND は太く短く、アナログ入力から離す。計測経路は PD 基準（非絶縁完成）。"
- note removed: "GP9=MCLK_SENSE は R720 1k 経由の入力専用。出力にすると Y701 と衝突して SCKI が化ける。"
- note removed: "POWER/DIGITAL: ADC_VIN->U705(MBC2596 6.6-6.8V)->U706(+3V3_A) then U707(+5V_A EN=+3V3_A). U704=+5V_D; D701 Schottky +5V_D->VSYS so USB cannot backfeed +5V_D. Y701 ASFL1->R718->ADC_MCLK (TP701; R720 1k to GP9 sense). U709 TPS3307-33D SO-8 watches +5V_A/+3V3_A, ~RESET->ADC_nRST (PP, 200ms), GP15 OD -> ~MR. U708 XC8107 LCD load-SW (LCD_EN High=ON)."
- note removed: "U706 LT1763-3.3 (+3V3_A). Fixed LDO; SHDN tied for always-on or as designed. Local CIN/COUT."
- note removed: "U707 EN=+3V3_A (3V3-first). AbsMax VCC-VDD protection."
- note removed: "U708 XC8107AC20MR-G ロードスイッチ: LCD_EN High=ON / Low・Hi-Z=OFF（Active High, VCEH 1.5V min → Pico 3.3V で直接駆動可）。R717 100k=CE プルダウンで起動時 OFF。初号は常時 ON 可。OFF 運用時は SPI/タッチを Low/Hi-Z に。ソフトスタート 0.6ms typ・短絡/逆流/過熱/UVLO 保護内蔵。C740=CIN, C739=CL は各 10uF/3216 を IC 直近へ。FLG は未使用（NC）。"
- note removed: "U709=TPS3307-33D SO-8: SENSE1=+5V_A (4.55V) SENSE2=+3V3_A (2.93V) SENSE3=VDD; VDD=+3V3_A C745 100nF; ~RESET PP -> ADC_nRST + R719; GP15 OD -> ~MR (do not drive H); RESET pin NC; 200ms delay. Replaces TPS3808G33/G50 SOT-23-6."
- note removed: "電源: USB VBUS → Pico 内部ショットキ → VSYS。D701 が +5V_D への逆流を止めるので、USB だけ挿すと Pico は動き LCD は消える。VBUS(pin40) は NC。"
Changed lines of the file:
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@@
 		)
 	)
-	(text "ADC_V_IN\n  ├─ BP5293-50 → +5V_D（Pico/LCD）\n  └─ MBC2596 → ~6.6V\n         ├─ LT1763-5   → +5V_A  （ADC）\n         └─ LT1763-3.3 → +3V3_A （ADC）"
+	(text "電源系（2026-09-07 U1604 削除後）\nPD_12V_SW ─F1602─ PD_12V_MEAS ─ U1607 BP5293-50 → +5V_D（Pico/LCD。GND=D_GND、CIN=C1645）\n+15V ─────────────────────── U1603 LT1763-3.3 → +3V3_A（ADC。GND=ADC_GND）\n+15V ─────────────────────── U1606 LT1763-5   → +5V_A （ADC。SHDN=+3V3_A で 3V3 先行）\n旧 U1604（MBC2596 12V→6.6V 非絶縁バック）と F1603/C1644 は削除。ADC の LDO は +15V 直結。"
 		(exclude_from_sim no)
 		(at 257.81 27.94 0)
@@
 		)
 	)
-	(text "POWER/DIGITAL: ADC_VIN->U705(MBC2596 6.6-6.8V)->U706(+3V3_A) then U707(+5V_A EN=+3V3_A). U704=+5V_D; D701 Schottky +5V_D->VSYS so USB cannot backfeed +5V_D. Y701 ASFL1->R718->ADC_MCLK (TP701; R720 1k to GP9 sense). U709 TPS3307-33D SO-8 watches +5V_A/+3V3_A, ~RESET->ADC_nRST (PP, 200ms), GP15 OD -> ~MR. U708 XC8107 LCD load-SW (LCD_EN High=ON)."
+	(text "POWER/DIGITAL（2026-09-07）: +15V → U1603(+3V3_A) と U1606(+5V_A, SHDN=+3V3_A)。旧 U1604(MBC2596) は削除。U1607=+5V_D（PD_12V_MEAS から）。D1601 ショットキ: +5V_D → Pico VSYS（USB 逆流止め）。Y1601 12.288MHz → R1604 33Ω → SCKI。R1605 1k → MCLK_SENSE(GP9、監視のみ。⚠ ファームは未使用)。U1609 XC8107 → LCD_VCC。U1605 TPS3307 監視。"
 		(exclude_from_sim no)
 		(at 325.12 17.78 0)
@@
 		)
 	)
-	(text "GP9=MCLK_SENSE は R720 1k 経由の入力専用。出力にすると Y701 と衝突して SCKI が化ける。"
+	(text "GP9=MCLK_SENSE は R1605 1k 経由の入力専用。出力にすると Y1601 と衝突して SCKI が化ける。"
 		(exclude_from_sim no)
 		(at 171.45 223.52 0)
@@
 		)
 	)
-	(text "A3 Pico2 横置き: 南列 1-20 西→東 / 北列 21-40 東→西。VSYS=+5V_D via D701 ショットキ, GND=D_GND | GP0=ADC_DATA GP1=ADC_BCK GP2=ADC_LRCK | GP3/GP4=NC(旧 LCD SPI) | GP5=LCD_CS GP6=LCD_DC GP7=LCD_RST GP8=LCD_EN | GP9=MCLK_SENSE (R720 1k, 入力専用) | GP10=TP_SDA GP11=TP_SCL GP12=TP_INT GP13=TP_RST | GP15=ADC_nMR (TPS3307 ~MR, OD, H は駆動しない) | GP18=LCD_SCK GP19=LCD_MOSI (SPI0)"
+	(text "A3 Pico2 横置き: 南列 1-20 西→東 / 北列 21-40 東→西。VSYS=+5V_D via D1601 ショットキ, GND=D_GND | GP0=ADC_DATA GP1=ADC_BCK GP2=ADC_LRCK | GP3/GP4=NC(旧 LCD SPI) | GP5=LCD_CS GP6=LCD_DC GP7=LCD_RST GP8=LCD_EN | GP9=MCLK_SENSE (R1605 1k, 入力専用) | GP10=TP_SDA GP11=TP_SCL GP12=TP_INT GP13=TP_RST | GP15=ADC_nMR (TPS3307 ~MR, OD, H は駆動しない) | GP18=LCD_SCK GP19=LCD_MOSI (SPI0)"
 		(exclude_from_sim no)
 		(at 171.45 213.36 0)
@@
 		)
 	)
-	(text "U707 EN=+3V3_A (3V3-first). AbsMax VCC-VDD protection."
+	(text "U1606 EN=+3V3_A (3V3-first). AbsMax VCC-VDD protection."
 		(exclude_from_sim no)
 		(at 325.628 20.828 0)
@@
 		)
 	)
-	(text "GND: NT702=A_GND─ADC_GND（A701近傍・アナログ星点）。NT701=ADC_GND_IN─D_GND（PD入口）。Pico/LCD は D_GND のみ。D_GND は太く短く、アナログ入力から離す。計測経路は PD 基準（非絶縁完成）。"
+	(text "GND: NT1601=A_GND─ADC_GND（A1601 近傍・アナログ星点）。NT1602=PD_GND─D_GND（PD 入口）。NT1603=A_GND─D_GND（2026-09-07 新設。U1604 削除で失われた A_GND↔D_GND の橋を明示化）。⚠ NT1601 / NT1602 / NT1603 は PCB で近接させる（1点アース。I2S の帰り・U403 の帰路・U201 の Ciso 経由 CM が全部ここを通る）。Pico/LCD は D_GND のみ。D_GND は太く短く、アナログ入力から離す。"
 		(exclude_from_sim no)
 		(at 63.246 14.478 0)
@@
 		)
 	)
-	(text "U709=TPS3307-33D SO-8: SENSE1=+5V_A (4.55V) SENSE2=+3V3_A (2.93V) SENSE3=VDD; VDD=+3V3_A C745 100nF; ~RESET PP -> ADC_nRST + R719; GP15 OD -> ~MR (do not drive H); RESET pin NC; 200ms delay. Replaces TPS3808G33/G50 SOT-23-6."
+	(text "U1605=TPS3307-33D SO-8: SENSE1=+5V_A (4.55V) SENSE2=+3V3_A (2.93V) SENSE3=VDD; VDD=+3V3_A C1614 100nF; ~RESET PP -> ADC_nRST + R1611; GP15 OD -> ~MR (do not drive H); RESET pin NC; 200ms delay. Replaces TPS3808G33/G50 SOT-23-6."
 		(exclude_from_sim no)
 		(at 406.654 16.002 0)
@@
 		(exclude_from_sim no)
 		(at 20.32 78.74 0)
-		(effects
-			(font
-				(size 1.397 1.397)
-			)
-			(justify left bottom)
-		)
-	)
-	(text "チャンネルあたりの公式リファレンス構成: 入力インバータ + ADC VCOM 基準の反転 LPF ドライバ×2。"
-		(exclude_from_sim no)
-		(at 20.32 78.74 0)
-		(effects
-			(font
-				(size 1.397 1.397)
-			)
-			(justify left bottom)
-		)
-	)
-	(text "OPA2134 からの OPA1656 置き換え。3.3k/4.7k 網では FET 入力が有利。試作で安定性とフルスケール・レベルを確認すること。"
-		(exclude_from_sim no)
-		(at 20.32 81.28 0)
 		(effects
 			(font
@@
 		)
 	)
-	(text "U706 LT1763-3.3 (+3V3_A). Fixed LDO; SHDN tied for always-on or as designed. Local CIN/COUT."
+	(text "U1603 LT1763-3.3 (+3V3_A). Fixed LDO; SHDN tied for always-on or as designed. Local CIN/COUT."
 		(exclude_from_sim no)
 		(at 407.416 13.97 0)
@@
 		)
 	)
-	(text "電源: USB VBUS → Pico 内部ショットキ → VSYS。D701 が +5V_D への逆流を止めるので、USB だけ挿すと Pico は動き LCD は消える。VBUS(pin40) は NC。"
+	(text "電源: USB VBUS → Pico 内部ショットキ → VSYS。D1601 が +5V_D への逆流を止めるので、USB だけ挿すと Pico は動き LCD は消える。VBUS(pin40) は NC。"
 		(exclude_from_sim no)
 		(at 171.45 219.71 0)
@@
 		)
 	)
-	(text "U708 XC8107AC20MR-G ロードスイッチ: LCD_EN High=ON / Low・Hi-Z=OFF（Active High, VCEH 1.5V min → Pico 3.3V で直接駆動可）。R717 100k=CE プルダウンで起動時 OFF。初号は常時 ON 可。OFF 運用時は SPI/タッチを Low/Hi-Z に。ソフトスタート 0.6ms typ・短絡/逆流/過熱/UVLO 保護内蔵。C740=CIN, C739=CL は各 10uF/3216 を IC 直近へ。FLG は未使用（NC）。"
+	(text "U1609 XC8107AC20MR-G ロードスイッチ: LCD_EN High=ON / Low・Hi-Z=OFF（Active High, VCEH 1.5V min → Pico 3.3V で直接駆動可）。R1620 100k=CE プルダウンで起動時 OFF。初号は常時 ON 可。OFF 運用時は SPI/タッチを Low/Hi-Z に。ソフトスタート 0.6ms typ・短絡/逆流/過熱/UVLO 保護内蔵。C1633=CIN, C1631=CL は各 10uF/3216 を IC 直近へ。FLG は未使用（NC）。"
 		(exclude_from_sim no)
 		(at 312.42 163.83 0)

Commit message: AudioV2: 計測タップにバッファを戻し、ADC のヘッドルームを直し、MCLK_SENSE を落とした
NOW.md の「次に手を動かすなら」1・2 と安い2件を実装した。すべて MeasureControl（手編集所有）。
部品 370 → 374。ERC 11 件は不変。

## 1. 計測タップの「+」側バッファ（v1 の AdcBuffer を OPA1656 で復元）

U1611 OPA1656 dual をユニティフォロワで AMP_SEL_L/R と前段の間に入れた。
挿入は AUDIO_L_IN / AUDIO_R_IN のラベル1枚ずつを新ネット ADC_BUF_L/R に改名するだけ
（下流の R1612/C1628・R1601/C1613 が丸ごと移り、バスには J1601・階層ピン・バッファ入力だけが残る）。
  入力バイアス   R1659/R1660 100k → A_GND（v1 の R805/R810 相当）
  デカップリング C1646/C1647 100nF
  出力 47Ω       付けない。「−」枝は U1602 出力(0Ω)から 10µF を見るので「+」枝も 0Ω で揃える

switch_thd.py を新負荷 30.4kΩ（RV501 50k ∥ R603 220k ∥ R1659 100k）で実行:
  TMUX7612 H3   −94.9 dB（1.87k） → −115.5 dB（30.4k）  +20.6 dB
H3 は実用律速 −106 dBc の下に戻った。

## 2. ADC のヘッドルーム — 前段入力抵抗 3.3k → 6.19k（0.1% E96）×4

R1614/R1618/R1603/R1609。帰還 1k と 1.8nF は触らないので LPF の極 88.4kHz は不変。
  差動ゲイン      0.606 → 0.323
  ADC FS バス換算  2.92 → 5.47 Vrms
  PT2314E typ 2.6 Vrms × AmpChannel ゲイン2 = 5.2 Vrms に対して +5.0 dBFS（超過）→ −0.4 dBFS
v1 で「+5.4 dBFS … ADC FS 超え。不可」と測定が止まった不具合の是正。

## 3. MCLK_SENSE を削除

R1605(1k)・ラベル2枚・スタブ3本を外し、A1602.12(GP9) を no_connect。
measurement_fw の全 .py で GP9 を読むコードは無かった。SCKI の生死は BCK(=SCKI/4) で分かる。
ADC_MCLK は A1601.7 / R1604.2 / TP1601.1 の3ピンに閉じた。12.288MHz が境界を渡る経路が消えた。

## 4. dcdc_survey.py: collect() が DigiKey の Offset+Limit<=300 を見ていなかった

1〜3W のビンで HTTP 400 で落ちていた（10〜20W では母集団が 300 未満で露出しなかった）。
300 で打ち切り、溢れたビンは軸を分けて引き直すよう警告する。

## 検証

  check_sexpr.py -q AudioV2   13 ファイル / 問題 0
  kicad-run.sh erc            11 件（変化なし。pin_not_connected も power_pin_not_driven も無し）
  kicad-run.sh netlist        部品 374 個・重複 0・footprint 未設定 0
  sch_import --roundtrip      6/6 OK
  sch_facts dangling / iface  0 本 / 0 件
  受け入れ条件  ADC_BUF_L = {C1628.2, R1612.2, U1611.1, U1611.2} / ADC_BUF_R 同形
                U1611.3/.5 → AMP_SEL_L/R、U1611.8/.4 → +15V/-15V
                ADC_MCLK 3 ピン、MCLK_SENSE 消滅
  再生成の冪等性               バイト一致
  gen_parts_bom.py            再生成済み

CLAUDE.md の期待値を 374 に更新。DECISIONS の3節を【確定】に、NOW.md の次の一手を差し替え。

Co-Authored-By: Claude Fable 5.1 <noreply@ant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
Parts:
- removed R1605: 1k, Resistor_SMD:R_1206_3216Metric_Pad1.30x1.75mm_HandSolder, symbol Device:R
- added C1646, C1647: 100nF, Capacitor_SMD:C_1206_3216Metric_Pad1.33x1.80mm_HandSolder, symbol Device:C
- added R1659, R1660: 100k, Resistor_SMD:R_1206_3216Metric_Pad1.30x1.75mm_HandSolder, symbol Device:R
- added U1611: OPA1656, Package_SO:SOIC-8_3.9x4.9mm_P1.27mm, symbol MeasurementADC1804:OPA1656
- R1603, R1609, R1614, R1618: value 3.3k 0.1% -> 6.19k 0.1%
Connections:
- net +15V_A: now also C1646.1, U1611.8 (V+)
- net -15V_A: now also C1647.2, U1611.4 (V-)
- net AUDIO_L_IN: now also R1659.1, U1611.3 (INA+); no longer C1628.2, R1612.2
- net AUDIO_R_IN: now also R1660.1, U1611.5 (INB+); no longer C1613.2, R1601.2
- net A_GND: now also C1646.2, C1647.1, R1659.2, R1660.2
- net MCLK_SENSE: no longer names the net of A1602.12 (GPIO9)
- new net ADC_BUF_L: C1628.2, R1612.2, U1611.1 (OUTA), U1611.2 (INA-)
- new net ADC_BUF_R: C1613.2, R1601.2, U1611.6 (INB-), U1611.7 (OUTB)
- no-connect marks 21 -> 22
Other:
- note added: "GP9: 旧 MCLK_SENSE（R1605 1k 経由）は 2026-09-07 に削除。ファームは GP9 を読んでいなかった。SCKI の生死は BCK（=SCKI/4）で分かる。GP9 は no_connect。"
- note removed: "A3 Pico2 横置き: 南列 1-20 西→東 / 北列 21-40 東→西。VSYS=+5V_D via D1601 ショットキ, GND=D_GND | GP0=ADC_DATA GP1=ADC_BCK GP2=ADC_LRCK | GP3/GP4=NC(旧 LCD SPI) | GP5=LCD_CS GP6=LCD_DC GP7=LCD_RST GP8=LCD_EN | GP9=MCLK_SENSE (R1605 1k, 入力専用) | GP10=TP_SDA GP11=TP_SCL GP12=TP_INT GP13=TP_RST | GP15=ADC_nMR (TPS3307 ~MR, OD, H は駆動しない) | GP18=LCD_SCK GP19=LCD_MOSI (SPI0)"
- note removed: "GP9=MCLK_SENSE は R1605 1k 経由の入力専用。出力にすると Y1601 と衝突して SCKI が化ける。"
