File: AudioV2/MeasureControl.kicad_sch (KiCad schematic)
At the start: 107 parts, among them J1601 AUDIO, J1602 V_IN, J1603 15_V_IN, SW1601 DEST sense (3PDT 3rd pole, sa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, U1601 OPA1656, U1602 OPA1656, U1603 LT1763-3.3, U1605 TPS3307-33, U1606 LT1763-5, U1607 BP5293-50, U1608 OPA1656, U1609 XC8107AC20MR-G, U1610 MCP23017 (UI 0x22), U1611 OPA1656, Y1601 ASFL1-12.288MHZ-EC-T

Commit message: AudioV2: ENC_INT に外付けプルアップ、BP5293 注釈を DS に合わせた
MCP23017 の INTA/INTB は OD なので 10k→3V3 を足した。BP5293 の穴は DS
推奨どおり Ø0.9 のまま（「1.2」は外形注記の誤読）で、等ピッチと推奨ランド
を Description に直した。Pico ピン注記と母板の旧 ENC→GP 文も現状へ。

Co-authored-by: m_arino <indare@users.noreply.github.com>
Parts:
- added R1661, R1662: 10k, Resistor_SMD:R_1206_3216Metric_Pad1.30x1.75mm_HandSolder, symbol Device:R
Connections:
- net 3V3: now also R1661.1, R1662.1
- net ENC_INTA: now also R1661.2
- net ENC_INTB: now also R1662.2
Other:
- note added: "A3 Pico2 横置き: 南列 1-20 西→東 / 北列 21-40 東→西。VSYS=+5V_D via D1601 ショットキ, GND=D_GND | GP0=ADC_DATA GP1=ADC_BCK GP2=ADC_LRCK | GP3/GP4=NC(旧 LCD SPI) | GP5=LCD_CS GP6=LCD_DC GP7=LCD_RST GP8=LCD_EN | GP9=NC（旧 MCLK_SENSE、2026-09-07 削除） | GP10=TP_SDA GP11=TP_SCL GP12=TP_INT GP13=TP_RST | GP15=ADC_nMR (TPS3307 ~MR, OD, H は駆動しない) | GP16=ENC_INTA GP17=ENC_INTB (U1610 MCP23017 割り込み、外付け 10k→3V3) | GP18=LCD_SCK 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"
- note removed: "A3 Pico2 横置き: 南列 1-20 西→東 / 北列 21-40 東→西。VSYS=+5V_D via D1601 ショットキ, GND=D_GND | GP0=ADC_DATA GP1=ADC_BCK GP2=ADC_LRCK | GP3/GP4=NC(旧 LCD SPI) | GP5=LCD_CS GP6=LCD_DC GP7=LCD_RST GP8=LCD_EN | GP9=NC（旧 MCLK_SENSE、2026-09-07 削除） | GP10=TP_SDA GP11=TP_SCL GP12=TP_INT GP13=TP_RST | GP15=ADC_nMR (TPS3307 ~MR, OD, H は駆動しない) | GP16=ENC_INTA GP17=ENC_INTB (U1610 MCP23017 割り込み) | GP18=LCD_SCK GP19=LCD_MOS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"
Changed lines of the file:
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@@
 		(comment 2 "共立 ADC_1804_F マニュアル p.7 の基準インターフェースに基づく")
 		(comment 3 "ASFL1 12.288MHz MCLK。ADCマスタ 48k/256fs。ジャンパ S/M=L, OSR2=L OSR1=H OSR0=H")
-		(comment 4 "電源: ADC_VIN→MBC2596→LT1763×2(+3V3_A先行/+5V_A)。+5V_D=BP5293。D701 SOD-123 ショットキ +5V_D→VSYS。U708=XC8107 LCD、U709=TPS3307-33D（3.3V+5V 監視 SO-8）")
+		(comment 4 "電源: +15V→LT1763×2(+3V3_A先行/+5V_A)。+5V_D=BP5293。D1601 ショットキ +5V_D→VSYS。U1609=XC8107 LCD、U1605=TPS3307-33D（3.3V+5V 監視 SO-8）。旧 U1604(MBC2596) は削除済み")
 	)
 	(text "ADC1804_F には PCM1804 のデカップリングとジャンパが内蔵済み。本シートは外部コネクタのみをモデル化。"
@@
 		)
 	)
-	(text "A3 Pico2 横置き: 南列 1-20 西→東 / 北列 21-40 東→西。VSYS=+5V_D via D1601 ショットキ, GND=D_GND | GP0=ADC_DATA GP1=ADC_BCK GP2=ADC_LRCK | GP3/GP4=NC(旧 LCD SPI) | GP5=LCD_CS GP6=LCD_DC GP7=LCD_RST GP8=LCD_EN | GP9=NC（旧 MCLK_SENSE、2026-09-07 削除） | GP10=TP_SDA GP11=TP_SCL GP12=TP_INT GP13=TP_RST | GP15=ADC_nMR (TPS3307 ~MR, OD, H は駆動しない) | GP16=ENC_INTA GP17=ENC_INTB (U1610 MCP23017 割り込み) | GP18=LCD_SCK GP19=LCD_MOSI (SPI0)"
+	(text "A3 Pico2 横置き: 南列 1-20 西→東 / 北列 21-40 東→西。VSYS=+5V_D via D1601 ショットキ, GND=D_GND | GP0=ADC_DATA GP1=ADC_BCK GP2=ADC_LRCK | GP3/GP4=NC(旧 LCD SPI) | GP5=LCD_CS GP6=LCD_DC GP7=LCD_RST GP8=LCD_EN | GP9=NC（旧 MCLK_SENSE、2026-09-07 削除） | GP10=TP_SDA GP11=TP_SCL GP12=TP_INT GP13=TP_RST | GP15=ADC_nMR (TPS3307 ~MR, OD, H は駆動しない) | GP16=ENC_INTA GP17=ENC_INTB (U1610 MCP23017 割り込み、外付け 10k→3V3) | GP18=LCD_SCK GP19=LCD_MOSI (SPI0) | GP20=I2C_SDA GP21=I2C_SCL | GP26=DEST_ADC"
 		(exclude_from_sim no)
 		(at 171.45 213.36 0)
@@
 			)
 		)
-		(property "Description" "BP5293/MBC2596 input bulk. 15V rail -> 35V rating. Return on ADC_GND_IN."
+		(property "Description" "ADC_V_IN bulk 47uF 35V. Return on ADC_GND_IN."
 			(at 237.49 49.53 0)
 			(hide yes)
@@
 		)
 	)
+	(symbol
+		(lib_id "Device:R")
+		(at 309.88 381.0 0)
+		(unit 1)
+		(body_style 1)
+		(exclude_from_sim no)
+		(in_bom yes)
+		(on_board yes)
+		(in_pos_files yes)
+		(dnp no)
+		(fields_autoplaced yes)
+		(property "Reference" "R1661"
+			(at 309.88 378.46 0)
+			(show_name no)
+			(do_not_autoplace no)
+			(effects
+				(font
+					(size 1.27 1.27)
+				)
+			)
+		)
+		(property "Value" "10k"
+			(at 309.88 383.54 0)
+			(show_name no)
+			(do_not_autoplace no)
+			(effects
+				(font
+					(size 1.27 1.27)
+				)
+			)
+		)
+		(property "Footprint" "Resistor_SMD:R_1206_3216Metric_Pad1.30x1.75mm_HandSolder"
+			(at 0 0 0)
+			(show_name no)
+			(do_not_autoplace no)
+			(hide yes)
+			(effects
+				(font
+					(size 1.27 1.27)
+				)
+			)
+		)
+		(property "Datasheet" ""
+			(at 0 0 0)
+			(show_name no)
+			(do_not_autoplace no)
+			(hide yes)
+			(effects
+				(font
+					(size 1.27 1.27)
+				)
+			)
+		)
+		(property "Description" "U1610 MCP23017 ENC_INTA open-drain pull-up to 3V3"
+			(at 0 0 0)
+			(show_name no)
+			(do_not_autoplace no)
+			(hide yes)
+			(effects
+				(font
+					(size 1.27 1.27)
+				)
+			)
+		)
+		(pin "1"
+		)
+		(pin "2"
+		)
+		(instances
+			(project "AudioV2Case"
+				(path "/a1000001-0001-4001-8001-000000000001/43e41fda-fe26-43e3-950a-c017f3070bbf"
+					(reference "R1661")
+					(unit 1)
+				)
+			)
+		)
+	)
+	(label "3V3"
+		(at 309.88 377.19 0)
+		(effects
+			(font
+				(size 1.27 1.27)
+			)
+			(justify left bottom)
+		)
+	)
+	(label "ENC_INTA"
+		(at 309.88 384.81 0)
+		(effects
+			(font
+				(size 1.27 1.27)
+			)
+			(justify left bottom)
+		)
+	)
+	(symbol
+		(lib_id "Device:R")
+		(at 325.12 381.0 0)
+		(unit 1)
+		(body_style 1)
+		(exclude_from_sim no)
+		(in_bom yes)
+		(on_board yes)
+		(in_pos_files yes)
+		(dnp no)
+		(fields_autoplaced yes)
+		(property "Reference" "R1662"
+			(at 325.12 378.46 0)
+			(show_name no)
+			(do_not_autoplace no)
+			(effects
+				(font
+					(size 1.27 1.27)
+				)
+			)
+		)
+		(property "Value" "10k"
+			(at 325.12 383.54 0)
+			(show_name no)
+			(do_not_autoplace no)
+			(effects
+				(font
+					(size 1.27 1.27)
+				)
+			)
+		)
+		(property "Footprint" "Resistor_SMD:R_1206_3216Metric_Pad1.30x1.75mm_HandSolder"
+			(at 0 0 0)
+			(show_name no)
+			(do_not_autoplace no)
+			(hide yes)
+			(effects
+				(font
+					(size 1.27 1.27)
+				)
+			)
+		)
+		(property "Datasheet" ""
+			(at 0 0 0)
+			(show_name no)
+			(do_not_autoplace no)
+			(hide yes)
+			(effects
+				(font
+					(size 1.27 1.27)
+				)
+			)
+		)
+		(property "Description" "U1610 MCP23017 ENC_INTB open-drain pull-up to 3V3"
+			(at 0 0 0)
+			(show_name no)
+			(do_not_autoplace no)
+			(hide yes)
+			(effects
+				(font
+					(size 1.27 1.27)
+				)
+			)
+		)
+		(pin "1"
+		)
+		(pin "2"
+		)
+		(instances
+			(project "AudioV2Case"
+				(path "/a1000001-0001-4001-8001-000000000001/43e41fda-fe26-43e3-950a-c017f3070bbf"
+					(reference "R1662")
+					(unit 1)
+				)
+			)
+		)
+	)
+	(label "3V3"
+		(at 325.12 377.19 0)
+		(effects
+			(font
+				(size 1.27 1.27)
+			)
+			(justify left bottom)
+		)
+	)
+	(label "ENC_INTB"
+		(at 325.12 384.81 0)
+		(effects
+			(font
+				(size 1.27 1.27)
+			)
+			(justify left bottom)
+		)
+	)
