File: AudioV2/AudioV2Case.kicad_pcb (KiCad board)
At the start: 2 copper layers, 0 parts

Commit message: AudioV2: ENC の MP を D_GND へ、リレー版を BOM/基板除外し PCB を起こした
アナログSW版を優先するため AmpBankRelay シートを on_board/in_bom=no に固定。
EC11 は RotaryEncoder_Switch_MP に差し替え、固定足を D_GND に接続した。

Co-authored-by: Cursor <cursoragent@cursor.com>
Parts:
- added A1601: ADC1804_F_MODULE, ADC1804_F_KYOHRITSU_56x33mm, F.Cu at (40.0, 55.0)
- added A1602: Pico2, RaspberryPi_Pico_Common_THT, F.Cu at (55.0, 55.0)
- added AMP1001: NE5532 / DIP-8 compatible, DIP-8_W7.62mm_Socket, F.Cu at (40.0, 205.0)
- added AMP601: NE5532 / DIP-8 compatible, DIP-8_W7.62mm_Socket, F.Cu at (100.0, 145.0)
- added AMP701: NE5532 / DIP-8 compatible, DIP-8_W7.62mm_Socket, F.Cu at (85.0, 160.0)
- added AMP801: NE5532 / DIP-8 compatible, DIP-8_W7.62mm_Socket, F.Cu at (70.0, 175.0)
- added AMP901: NE5532 / DIP-8 compatible, DIP-8_W7.62mm_Socket, F.Cu at (55.0, 190.0)
- added C1001: 2.2uF film, C_Rect_L7.2mm_W2.5mm_P5.00mm_FKS2_FKP2_MKS2_MKP2, F.Cu at (55.0, 205.0)
- added C1002: 1uF film, C_Rect_L11.0mm_W4.2mm_P10.00mm_MKT, F.Cu at (70.0, 205.0)
- added C1004: 2.2uF film, C_Rect_L7.2mm_W2.5mm_P5.00mm_FKS2_FKP2_MKS2_MKP2, F.Cu at (85.0, 205.0)
- added C1005: 1uF film, C_Rect_L11.0mm_W4.2mm_P10.00mm_MKT, F.Cu at (100.0, 205.0)
- added C1007: 100nF, C_1206_3216Metric_Pad1.33x1.80mm_HandSolder, F.Cu at (115.0, 205.0)
- added C1008: 100nF, C_1206_3216Metric_Pad1.33x1.80mm_HandSolder, F.Cu at (130.0, 205.0)
- added C1009: 100nF, C_1206_3216Metric_Pad1.33x1.80mm_HandSolder, F.Cu at (145.0, 205.0)
- added C1010: 100nF, C_1206_3216Metric_Pad1.33x1.80mm_HandSolder, F.Cu at (160.0, 205.0)
- added C1601: 10nF, C_1206_3216Metric_Pad1.33x1.80mm_HandSolder, F.Cu at (70.0, 55.0)
- added C1602: 10uF 25V NP, C_Radial_D5.0mm_H7.0mm_P2.00mm, F.Cu at (85.0, 55.0)
- added C1603: 10uF 10V X7R, C_1206_3216Metric_Pad1.33x1.80mm_HandSolder, F.Cu at (100.0, 55.0)
- added C1604: 100nF, C_1206_3216Metric_Pad1.33x1.80mm_HandSolder, F.Cu at (115.0, 55.0)
- added C1605: 100nF, C_1206_3216Metric_Pad1.33x1.80mm_HandSolder, F.Cu at (130.0, 55.0)
- added C1606: 10uF 50V X7R, C_1210_3225Metric_Pad1.33x2.70mm_HandSolder, F.Cu at (145.0, 55.0)
- added C1607: 100nF, C_1206_3216Metric_Pad1.33x1.80mm_HandSolder, F.Cu at (160.0, 55.0)
- added C1608: 10nF, C_1206_3216Metric_Pad1.33x1.80mm_HandSolder, F.Cu at (175.0, 55.0)
- added C1609: 1.8nF C0G, C_1206_3216Metric_Pad1.33x1.80mm_HandSolder, F.Cu at (190.0, 55.0)
- added C1610: 47uF 35V, CP_Radial_D8.0mm_P3.50mm, F.Cu at (205.0, 55.0)
- added C1611: 10uF, C_1206_3216Metric_Pad1.33x1.80mm_HandSolder, F.Cu at (220.0, 55.0)
- added C1612: 100nF, C_1206_3216Metric_Pad1.33x1.80mm_HandSolder, F.Cu at (235.0, 55.0)
- added C1613: 10uF 25V NP, C_Radial_D5.0mm_H7.0mm_P2.00mm, F.Cu at (250.0, 55.0)
- added C1614: 100nF, C_1206_3216Metric_Pad1.33x1.80mm_HandSolder, F.Cu at (265.0, 55.0)
- added C1615: 100nF, C_1206_3216Metric_Pad1.33x1.80mm_HandSolder, F.Cu at (280.0, 55.0)
- added C1616: 10uF 16V X7R, C_1206_3216Metric_Pad1.33x1.80mm_HandSolder, F.Cu at (295.0, 55.0)
- added C1617: 100nF, C_1206_3216Metric_Pad1.33x1.80mm_HandSolder, F.Cu at (10.0, 70.0)
- added C1618: 100nF, C_1206_3216Metric_Pad1.33x1.80mm_HandSolder, F.Cu at (25.0, 70.0)
- added C1619: 10uF 50V X7R, C_1210_3225Metric_Pad1.33x2.70mm_HandSolder, F.Cu at (40.0, 70.0)
- added C1620: 1.8nF C0G, C_1206_3216Metric_Pad1.33x1.80mm_HandSolder, F.Cu at (55.0, 70.0)
- added C1621: 47uF, CP_Radial_D8.0mm_P3.50mm, F.Cu at (70.0, 70.0)
- added C1622: 100nF, C_1206_3216Metric_Pad1.33x1.80mm_HandSolder, F.Cu at (85.0, 70.0)
- added C1623: 10nF, C_1206_3216Metric_Pad1.33x1.80mm_HandSolder, F.Cu at (100.0, 70.0)
- added C1624: 100nF, C_1206_3216Metric_Pad1.33x1.80mm_HandSolder, F.Cu at (115.0, 70.0)
- added C1625: 100nF, C_1206_3216Metric_Pad1.33x1.80mm_HandSolder, F.Cu at (130.0, 70.0)
- added C1626: 10uF 25V NP, C_Radial_D5.0mm_H7.0mm_P2.00mm, F.Cu at (145.0, 70.0)
- added C1627: 1.8nF C0G, C_1206_3216Metric_Pad1.33x1.80mm_HandSolder, F.Cu at (160.0, 70.0)
- added C1628: 10uF 25V NP, C_Radial_D5.0mm_H7.0mm_P2.00mm, F.Cu at (175.0, 70.0)
- added C1629: 100nF, C_1206_3216Metric_Pad1.33x1.80mm_HandSolder, F.Cu at (190.0, 70.0)
- added C1630: 22uF, CP_Radial_D6.3mm_P2.50mm, F.Cu at (205.0, 70.0)
- added C1631: 10uF, C_1206_3216Metric_Pad1.33x1.80mm_HandSolder, F.Cu at (220.0, 70.0)
- added C1632: 1.8nF C0G, C_1206_3216Metric_Pad1.33x1.80mm_HandSolder, F.Cu at (235.0, 70.0)
- added C1633: 10uF, C_1206_3216Metric_Pad1.33x1.80mm_HandSolder, F.Cu at (250.0, 70.0)
- added C1634: 100nF, C_1206_3216Metric_Pad1.33x1.80mm_HandSolder, F.Cu at (265.0, 70.0)
- added C1635: 10uF 50V, CP_Radial_D5.0mm_P2.00mm, F.Cu at (280.0, 70.0)
- added C1636: 100nF, C_1206_3216Metric_Pad1.33x1.80mm_HandSolder, F.Cu at (295.0, 70.0)
- added C1637: 100nF, C_1206_3216Metric_Pad1.33x1.80mm_HandSolder, F.Cu at (10.0, 85.0)
- added C1638: 100nF, C_1206_3216Metric_Pad1.33x1.80mm_HandSolder, F.Cu at (25.0, 85.0)
- added C1639: 100nF, C_1206_3216Metric_Pad1.33x1.80mm_HandSolder, F.Cu at (40.0, 85.0)
- added C1640: 10uF 50V, CP_Radial_D5.0mm_P2.00mm, F.Cu at (55.0, 85.0)
- added C1641: 100nF, C_1206_3216Metric_Pad1.33x1.80mm_HandSolder, F.Cu at (70.0, 85.0)
- added C1642: 100nF, C_1206_3216Metric_Pad1.33x1.80mm_HandSolder, F.Cu at (85.0, 85.0)
- added C1643: 100nF, C_1206_3216Metric_Pad1.33x1.80mm_HandSolder, F.Cu at (100.0, 85.0)
- added C1645: 10uF 50V, C_1206_3216Metric_Pad1.33x1.80mm_HandSolder, F.Cu at (115.0, 85.0)
- added C1646: 100nF, C_1206_3216Metric_Pad1.33x1.80mm_HandSolder, F.Cu at (130.0, 85.0)
- added C1647: 100nF, C_1206_3216Metric_Pad1.33x1.80mm_HandSolder, F.Cu at (145.0, 85.0)
- added C1650: 100nF, C_1206_3216Metric_Pad1.33x1.80mm_HandSolder, F.Cu at (160.0, 85.0)
- added C201: 47u, CP_Radial_D8.0mm_P3.50mm, F.Cu at (10.0, 10.0)
- added C202: 0.1u, C_1206_3216Metric_Pad1.33x1.80mm_HandSolder, F.Cu at (25.0, 10.0)
- added C203: 10u, CP_Radial_D5.0mm_P2.00mm, F.Cu at (40.0, 10.0)
- added C204: 0.1u, C_1206_3216Metric_Pad1.33x1.80mm_HandSolder, F.Cu at (55.0, 10.0)
- added C205: 47u, CP_Radial_D8.0mm_P3.50mm, F.Cu at (70.0, 10.0)
- added C206: 0.1u, C_1206_3216Metric_Pad1.33x1.80mm_HandSolder, F.Cu at (85.0, 10.0)
- added C207: 47u, CP_Radial_D8.0mm_P3.50mm, F.Cu at (100.0, 10.0)
- added C208: 0.1u, C_1206_3216Metric_Pad1.33x1.80mm_HandSolder, F.Cu at (115.0, 10.0)
- added C311: 100nF, C_1206_3216Metric_Pad1.33x1.80mm_HandSolder, F.Cu at (175.0, 130.0)
- added C312: 100nF, C_1206_3216Metric_Pad1.33x1.80mm_HandSolder, F.Cu at (190.0, 130.0)
- added C313: 100nF, C_1206_3216Metric_Pad1.33x1.80mm_HandSolder, F.Cu at (205.0, 130.0)
- added C314: 100nF, C_1206_3216Metric_Pad1.33x1.80mm_HandSolder, F.Cu at (220.0, 130.0)
- added C315: 100nF, C_1206_3216Metric_Pad1.33x1.80mm_HandSolder, F.Cu at (235.0, 130.0)
- added C316: 100nF, C_1206_3216Metric_Pad1.33x1.80mm_HandSolder, F.Cu at (250.0, 130.0)
- added C401: 22u, CP_Radial_D6.3mm_P2.50mm, F.Cu at (130.0, 10.0)
- added C402: 0.1u, C_1206_3216Metric_Pad1.33x1.80mm_HandSolder, F.Cu at (145.0, 10.0)
- added C403: 100n, C_1206_3216Metric_Pad1.33x1.80mm_HandSolder, F.Cu at (160.0, 10.0)
- added C404: 100n, C_1206_3216Metric_Pad1.33x1.80mm_HandSolder, F.Cu at (175.0, 10.0)
- added C405: 2.2u, C_Rect_L7.2mm_W2.5mm_P5.00mm_FKS2_FKP2_MKS2_MKP2, F.Cu at (190.0, 10.0)
- added C406: 2.2u, C_Rect_L7.2mm_W2.5mm_P5.00mm_FKS2_FKP2_MKS2_MKP2, F.Cu at (205.0, 10.0)
- added C407: 2.2u, C_Rect_L7.2mm_W2.5mm_P5.00mm_FKS2_FKP2_MKS2_MKP2, F.Cu at (220.0, 10.0)
- added C408: 2.7n, C_1206_3216Metric_Pad1.33x1.80mm_HandSolder, F.Cu at (235.0, 10.0)
- added C409: 2.2u, C_Rect_L7.2mm_W2.5mm_P5.00mm_FKS2_FKP2_MKS2_MKP2, F.Cu at (250.0, 10.0)
- added C410: 100n, C_1206_3216Metric_Pad1.33x1.80mm_HandSolder, F.Cu at (265.0, 10.0)
- added C411: 100n, C_1206_3216Metric_Pad1.33x1.80mm_HandSolder, F.Cu at (280.0, 10.0)
- added C412: 2.7n, C_1206_3216Metric_Pad1.33x1.80mm_HandSolder, F.Cu at (295.0, 10.0)
- added C501: 470uF 25V NP, CP_Radial_D10.0mm_P5.00mm, F.Cu at (10.0, 25.0)
- added C502: 470uF 25V NP, CP_Radial_D10.0mm_P5.00mm, F.Cu at (25.0, 25.0)
- added C503: 10uF 25V X7R, C_1206_3216Metric_Pad1.33x1.80mm_HandSolder, F.Cu at (40.0, 25.0)
- added C504: 10uF 25V X7R, C_1206_3216Metric_Pad1.33x1.80mm_HandSolder, F.Cu at (55.0, 25.0)
- added C505: 100nF, C_1206_3216Metric_Pad1.33x1.80mm_HandSolder, F.Cu at (70.0, 25.0)
- added C506: 100nF, C_1206_3216Metric_Pad1.33x1.80mm_HandSolder, F.Cu at (85.0, 25.0)
- added C601: 2.2uF film, C_Rect_L7.2mm_W2.5mm_P5.00mm_FKS2_FKP2_MKS2_MKP2, F.Cu at (115.0, 145.0)
- added C602: 1uF film, C_Rect_L11.0mm_W4.2mm_P10.00mm_MKT, F.Cu at (130.0, 145.0)
- added C604: 2.2uF film, C_Rect_L7.2mm_W2.5mm_P5.00mm_FKS2_FKP2_MKS2_MKP2, F.Cu at (145.0, 145.0)
- added C605: 1uF film, C_Rect_L11.0mm_W4.2mm_P10.00mm_MKT, F.Cu at (160.0, 145.0)
- added C607: 100nF, C_1206_3216Metric_Pad1.33x1.80mm_HandSolder, F.Cu at (175.0, 145.0)
- added C608: 100nF, C_1206_3216Metric_Pad1.33x1.80mm_HandSolder, F.Cu at (190.0, 145.0)
- added C609: 100nF, C_1206_3216Metric_Pad1.33x1.80mm_HandSolder, F.Cu at (205.0, 145.0)
- added C610: 100nF, C_1206_3216Metric_Pad1.33x1.80mm_HandSolder, F.Cu at (220.0, 145.0)
- added C701: 2.2uF film, C_Rect_L7.2mm_W2.5mm_P5.00mm_FKS2_FKP2_MKS2_MKP2, F.Cu at (100.0, 160.0)
- added C702: 1uF film, C_Rect_L11.0mm_W4.2mm_P10.00mm_MKT, F.Cu at (115.0, 160.0)
- added C704: 2.2uF film, C_Rect_L7.2mm_W2.5mm_P5.00mm_FKS2_FKP2_MKS2_MKP2, F.Cu at (130.0, 160.0)
- added C705: 1uF film, C_Rect_L11.0mm_W4.2mm_P10.00mm_MKT, F.Cu at (145.0, 160.0)
- added C707: 100nF, C_1206_3216Metric_Pad1.33x1.80mm_HandSolder, F.Cu at (160.0, 160.0)
- added C708: 100nF, C_1206_3216Metric_Pad1.33x1.80mm_HandSolder, F.Cu at (175.0, 160.0)
- added C709: 100nF, C_1206_3216Metric_Pad1.33x1.80mm_HandSolder, F.Cu at (190.0, 160.0)
- added C710: 100nF, C_1206_3216Metric_Pad1.33x1.80mm_HandSolder, F.Cu at (205.0, 160.0)
- added C801: 2.2uF film, C_Rect_L7.2mm_W2.5mm_P5.00mm_FKS2_FKP2_MKS2_MKP2, F.Cu at (85.0, 175.0)
- added C802: 1uF film, C_Rect_L11.0mm_W4.2mm_P10.00mm_MKT, F.Cu at (100.0, 175.0)
- added C804: 2.2uF film, C_Rect_L7.2mm_W2.5mm_P5.00mm_FKS2_FKP2_MKS2_MKP2, F.Cu at (115.0, 175.0)
- added C805: 1uF film, C_Rect_L11.0mm_W4.2mm_P10.00mm_MKT, F.Cu at (130.0, 175.0)
- added C807: 100nF, C_1206_3216Metric_Pad1.33x1.80mm_HandSolder, F.Cu at (145.0, 175.0)
- added C808: 100nF, C_1206_3216Metric_Pad1.33x1.80mm_HandSolder, F.Cu at (160.0, 175.0)
- added C809: 100nF, C_1206_3216Metric_Pad1.33x1.80mm_HandSolder, F.Cu at (175.0, 175.0)
- added C810: 100nF, C_1206_3216Metric_Pad1.33x1.80mm_HandSolder, F.Cu at (190.0, 175.0)
- added C901: 2.2uF film, C_Rect_L7.2mm_W2.5mm_P5.00mm_FKS2_FKP2_MKS2_MKP2, F.Cu at (70.0, 190.0)
- added C902: 1uF film, C_Rect_L11.0mm_W4.2mm_P10.00mm_MKT, F.Cu at (85.0, 190.0)
- added C904: 2.2uF film, C_Rect_L7.2mm_W2.5mm_P5.00mm_FKS2_FKP2_MKS2_MKP2, F.Cu at (100.0, 190.0)
- added C905: 1uF film, C_Rect_L11.0mm_W4.2mm_P10.00mm_MKT, F.Cu at (115.0, 190.0)
- added C907: 100nF, C_1206_3216Metric_Pad1.33x1.80mm_HandSolder, F.Cu at (130.0, 190.0)
- added C908: 100nF, C_1206_3216Metric_Pad1.33x1.80mm_HandSolder, F.Cu at (145.0, 190.0)
- added C909: 100nF, C_1206_3216Metric_Pad1.33x1.80mm_HandSolder, F.Cu at (160.0, 190.0)
- added C910: 100nF, C_1206_3216Metric_Pad1.33x1.80mm_HandSolder, F.Cu at (175.0, 190.0)
- added C_BULK_N301: 100uF 35V, CP_Elec_10x12.6, F.Cu at (265.0, 130.0)
- added C_BULK_P301: 100uF 35V, CP_Elec_10x12.6, F.Cu at (280.0, 130.0)
- added C_IO301: 100nF, C_1206_3216Metric_Pad1.33x1.80mm_HandSolder, F.Cu at (295.0, 130.0)
- added D1601: RB160M-30, D_SOD-123, F.Cu at (175.0, 85.0)
- added D1610: DEST 1, LED_D5.0mm, F.Cu at (190.0, 85.0)
- added D1611: DEST 2, LED_D5.0mm, F.Cu at (205.0, 85.0)
- added D403: 12V panel LED, LED_D5.0mm, F.Cu at (100.0, 25.0)
- added ENC1601: ENC_CH, RotaryEncoder_Alps_EC11E-Switch_Vertical_H20mm, F.Cu at (220.0, 85.0)
- added ENC1602: ENC_BASS, RotaryEncoder_Alps_EC11E-Switch_Vertical_H20mm, F.Cu at (235.0, 85.0)
- added ENC1603: ENC_TREBLE, RotaryEncoder_Alps_EC11E-Switch_Vertical_H20mm, F.Cu at (250.0, 85.0)
- added F1601: T1A slow 5x20, Fuseholder_Cylinder-5x20mm_Schurter_0031_8201_Horizontal_Open, F.Cu at (265.0, 85.0)
- added F1602: PPTC 0.5A hold, PPTC_Radial_D7.9mm_T3.1mm_P5.08mm, F.Cu at (280.0, 85.0)
- added F201: T1.6A slow 5x20, Fuseholder_Cylinder-5x20mm_Schurter_0031_8201_Horizontal_Open, F.Cu at (115.0, 25.0)
- added F202: PPTC 0.4A hold, PPTC_Radial_D7.9mm_T3.1mm_P5.08mm, F.Cu at (130.0, 25.0)
- added F203: PPTC 0.1A hold, PPTC_Radial_D7.9mm_T3.1mm_P5.08mm, F.Cu at (145.0, 25.0)
- added J1601: AUDIO, TerminalBlock_Phoenix_MKDS-1,5-2-5.08_1x02_P5.08mm_Horizontal, F.Cu at (295.0, 85.0)
- added J1602: V_IN, TerminalBlock_Phoenix_MKDS-1,5-2-5.08_1x02_P5.08mm_Horizontal, F.Cu at (10.0, 100.0)
- added J1603: 15_V_IN, TerminalBlock_Phoenix_MKDS-1,5-3-5.08_1x03_P5.08mm_Horizontal, F.Cu at (25.0, 100.0)
- added J201: +15/A_GND/-15 out, TerminalBlock_Phoenix_MKDS-1,5-3-5.08_1x03_P5.08mm_Horizontal, F.Cu at (160.0, 25.0)
- added J202: PD module in (1=GND 2=+12V), TerminalBlock_Phoenix_MKDS-1,5-2-5.08_1x02_P5.08mm_Horizontal, F.Cu at (175.0, 25.0)
- added J_ANA101: SLOT1 ANA (D18), PinSocket_2x05_P2.54mm_Vertical, F.Cu at (190.0, 25.0)
- added J_ANA102: SLOT2 ANA (D18), PinSocket_2x05_P2.54mm_Vertical, F.Cu at (205.0, 25.0)
- added J_ANA301: SLOT ANA (D18), PinHeader_2x05_P2.54mm_Vertical, F.Cu at (10.0, 145.0)
- added J_HP501: HP OUT, TerminalBlock_Phoenix_MKDS-1,5-3-5.08_1x03_P5.08mm_Horizontal, F.Cu at (220.0, 25.0)
- added J_IN401: AUDIO IN L/R, TerminalBlock_Phoenix_MKDS-1,5-3-5.08_1x03_P5.08mm_Horizontal, F.Cu at (235.0, 25.0)
- added J_LINE501: LINE OUT, TerminalBlock_Phoenix_MKDS-1,5-3-5.08_1x03_P5.08mm_Horizontal, F.Cu at (250.0, 25.0)
- added J_OLED1601: 2.42 OLED I2C GND/3V3/SCL/SDA, PinHeader_1x04_P2.54mm_Vertical, F.Cu at (40.0, 100.0)
- added J_PWR101: SLOT1 PWR/CTRL (D18), PinSocket_2x06_P2.54mm_Vertical, F.Cu at (265.0, 25.0)
- added J_PWR102: SLOT2 PWR/CTRL (D18), PinSocket_2x06_P2.54mm_Vertical, F.Cu at (280.0, 25.0)
- added J_PWR301: SLOT PWR/CTRL (D18), PinHeader_2x06_P2.54mm_Vertical, F.Cu at (25.0, 145.0)
- added J_RAIL501: AMP_SEL OUT, TerminalBlock_Phoenix_MKDS-1,5-3-5.08_1x03_P5.08mm_Horizontal, F.Cu at (295.0, 25.0)
- added LCDDisplay1601: WAVESHARE-29318, PinHeader_1x15_P2.54mm_Vertical, F.Cu at (55.0, 100.0)
- added NT101: GND_COIL-D_GND, NetTie-2_SMD_Pad2.0mm, F.Cu at (10.0, 40.0)
- added NT1601: A_GND-ADC_GND, NetTie-2_SMD_Pad2.0mm, F.Cu at (70.0, 100.0)
- added NT1602: ADC_GND_IN-D_GND, NetTie-2_SMD_Pad2.0mm, F.Cu at (85.0, 100.0)
- added NT1603: A_GND-D_GND, NetTie-2_SMD_Pad0.5mm, F.Cu at (100.0, 100.0)
- added Q401: BSS138, SOT-23, F.Cu at (25.0, 40.0)
- added Q402: BSS138, SOT-23, F.Cu at (40.0, 40.0)
- added R1001: 100k, R_1206_3216Metric_Pad1.30x1.75mm_HandSolder, F.Cu at (175.0, 205.0)
- added R1002: 47R, R_1206_3216Metric_Pad1.30x1.75mm_HandSolder, F.Cu at (190.0, 205.0)
- added R1003: 220k, R_1206_3216Metric_Pad1.30x1.75mm_HandSolder, F.Cu at (205.0, 205.0)
- added R1004: 20k, R_1206_3216Metric_Pad1.30x1.75mm_HandSolder, F.Cu at (220.0, 205.0)
- added R1006: 20k, R_1206_3216Metric_Pad1.30x1.75mm_HandSolder, F.Cu at (235.0, 205.0)
- added R1007: 100k, R_1206_3216Metric_Pad1.30x1.75mm_HandSolder, F.Cu at (250.0, 205.0)
- added R1008: 47R, R_1206_3216Metric_Pad1.30x1.75mm_HandSolder, F.Cu at (265.0, 205.0)
- added R1009: 220k, R_1206_3216Metric_Pad1.30x1.75mm_HandSolder, F.Cu at (280.0, 205.0)
- added R1010: 20k, R_1206_3216Metric_Pad1.30x1.75mm_HandSolder, F.Cu at (295.0, 205.0)
- added R1012: 20k, R_1206_3216Metric_Pad1.30x1.75mm_HandSolder, F.Cu at (10.0, 220.0)
- added R1601: 4.7k 0.1%, R_1206_3216Metric_Pad1.30x1.75mm_HandSolder, F.Cu at (115.0, 100.0)
- added R1602: 47, R_1206_3216Metric_Pad1.30x1.75mm_HandSolder, F.Cu at (130.0, 100.0)
- added R1603: 6.19k 0.1%, R_1206_3216Metric_Pad1.30x1.75mm_HandSolder, F.Cu at (145.0, 100.0)
- added R1604: 33, R_1206_3216Metric_Pad1.30x1.75mm_HandSolder, F.Cu at (160.0, 100.0)
- added R1606: 4.7k 0.1%, R_1206_3216Metric_Pad1.30x1.75mm_HandSolder, F.Cu at (175.0, 100.0)
- added R1607: 1k 0.1%, R_1206_3216Metric_Pad1.30x1.75mm_HandSolder, F.Cu at (190.0, 100.0)
- added R1608: 47, R_1206_3216Metric_Pad1.30x1.75mm_HandSolder, F.Cu at (205.0, 100.0)
- added R1609: 6.19k 0.1%, R_1206_3216Metric_Pad1.30x1.75mm_HandSolder, F.Cu at (220.0, 100.0)
- added R1610: 1k 0.1%, R_1206_3216Metric_Pad1.30x1.75mm_HandSolder, F.Cu at (235.0, 100.0)
- added R1611: 10k, R_1206_3216Metric_Pad1.30x1.75mm_HandSolder, F.Cu at (250.0, 100.0)
- added R1612: 4.7k 0.1%, R_1206_3216Metric_Pad1.30x1.75mm_HandSolder, F.Cu at (265.0, 100.0)
- added R1613: 47, R_1206_3216Metric_Pad1.30x1.75mm_HandSolder, F.Cu at (280.0, 100.0)
- added R1614: 6.19k 0.1%, R_1206_3216Metric_Pad1.30x1.75mm_HandSolder, F.Cu at (295.0, 100.0)
- added R1615: 4.7k 0.1%, R_1206_3216Metric_Pad1.30x1.75mm_HandSolder, F.Cu at (10.0, 115.0)
- added R1616: 1k 0.1%, R_1206_3216Metric_Pad1.30x1.75mm_HandSolder, F.Cu at (25.0, 115.0)
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
Commit message: AudioV2: ネットクラス（電源幹線1mm / 局所・音声0.5mm / デジタル0.3mm）を設定
KiCad 終了時の PCB・親回路図の保存も取り込み。生成娘シートの書き換えは捨てた。

Co-authored-by: Cursor <cursoragent@cursor.com>
Parts:
- A1601: footprint ADC1804_F_KYOHRITSU_56x33mm -> Library:ADC1804_F_KYOHRITSU_56x33mm
- A1602: footprint RaspberryPi_Pico_Common_THT -> Module:RaspberryPi_Pico_Common_THT
- AMP1001, AMP601, AMP701, AMP801, AMP901, U501: footprint DIP-8_W7.62mm_Socket -> Package_DIP:DIP-8_W7.62mm_Socket
- C1001, C1004, C405, C406, C407, C409, C601, C604, C701, C704, C801, C804, C901, C904: footprint C_Rect_L7.2mm_W2.5mm_P5.00mm_FKS2_FKP2_MKS2_MKP2 -> Capacitor_THT:C_Rect_L7.2mm_W2.5mm_P5.00mm_FKS2_FKP2_MKS2_MKP2
- C1002, C1005, C602, C605, C702, C705, C802, C805, C902, C905: footprint C_Rect_L11.0mm_W4.2mm_P10.00mm_MKT -> Capacitor_THT:C_Rect_L11.0mm_W4.2mm_P10.00mm_MKT
- C1007, C1008, C1009, C1010, C1601, C1603, C1604, C1605, C1607, C1608, C1609, C1611, C1612, C1614, C1615, C1616, C1617, C1618, C1620, C1622, C1623, C1624, C1625, C1627, C1629, C1631, C1632, C1633, C1634, C1636, C1637, C1638, C1639, C1641, C1642, C1643, C1645, C1646, C1647, C1650, C202, C204, C206, C208, C311, C312, C313, C314, C315, C316, C402, C403, C404, C408, C410, C411, C412, C503, C504, C505, C506, C607, C608, C609, C610, C707, C708, C709, C710, C807, C808, C809, C810, C907, C908, C909, C910, C_IO301: footprint C_1206_3216Metric_Pad1.33x1.80mm_HandSolder -> Capacitor_SMD:C_1206_3216Metric_Pad1.33x1.80mm_HandSolder
- C1602, C1613, C1626, C1628: footprint C_Radial_D5.0mm_H7.0mm_P2.00mm -> Capacitor_THT:C_Radial_D5.0mm_H7.0mm_P2.00mm
- C1606, C1619: footprint C_1210_3225Metric_Pad1.33x2.70mm_HandSolder -> Capacitor_SMD:C_1210_3225Metric_Pad1.33x2.70mm_HandSolder
- C1610, C1621, C201, C205, C207: footprint CP_Radial_D8.0mm_P3.50mm -> Capacitor_THT:CP_Radial_D8.0mm_P3.50mm
- C1630, C401: footprint CP_Radial_D6.3mm_P2.50mm -> Capacitor_THT:CP_Radial_D6.3mm_P2.50mm
- C1635, C1640, C203: footprint CP_Radial_D5.0mm_P2.00mm -> Capacitor_THT:CP_Radial_D5.0mm_P2.00mm
- C501, C502: footprint CP_Radial_D10.0mm_P5.00mm -> Capacitor_THT:CP_Radial_D10.0mm_P5.00mm
- C_BULK_N301, C_BULK_P301: footprint CP_Elec_10x12.6 -> Capacitor_SMD:CP_Elec_10x12.6
- D1601: footprint D_SOD-123 -> Diode_SMD:D_SOD-123
- D1610, D1611, D403: footprint LED_D5.0mm -> LED_THT:LED_D5.0mm
- ENC1601, ENC1602, ENC1603: footprint RotaryEncoder_Alps_EC11E-Switch_Vertical_H20mm -> Rotary_Encoder:RotaryEncoder_Alps_EC11E-Switch_Vertical_H20mm
- F1601, F201: footprint Fuseholder_Cylinder-5x20mm_Schurter_0031_8201_Horizontal_Open -> Fuse:Fuseholder_Cylinder-5x20mm_Schurter_0031_8201_Horizontal_Open
- F1602, F202, F203: footprint PPTC_Radial_D7.9mm_T3.1mm_P5.08mm -> Library:PPTC_Radial_D7.9mm_T3.1mm_P5.08mm
- J1601, J1602, J202: footprint TerminalBlock_Phoenix_MKDS-1,5-2-5.08_1x02_P5.08mm_Horizontal -> TerminalBlock_Phoenix:TerminalBlock_Phoenix_MKDS-1,5-2-5.08_1x02_P5.08mm_Horizontal
- J1603, J201, J_HP501, J_IN401, J_LINE501, J_RAIL501: footprint TerminalBlock_Phoenix_MKDS-1,5-3-5.08_1x03_P5.08mm_Horizontal -> TerminalBlock_Phoenix:TerminalBlock_Phoenix_MKDS-1,5-3-5.08_1x03_P5.08mm_Horizontal
- J_ANA101, J_ANA102: footprint PinSocket_2x05_P2.54mm_Vertical -> Connector_PinSocket_2.54mm:PinSocket_2x05_P2.54mm_Vertical
- J_ANA301: footprint PinHeader_2x05_P2.54mm_Vertical -> Connector_PinHeader_2.54mm:PinHeader_2x05_P2.54mm_Vertical
- J_OLED1601, SW1601, SW501, SW502: footprint PinHeader_1x04_P2.54mm_Vertical -> Connector_PinHeader_2.54mm:PinHeader_1x04_P2.54mm_Vertical
- J_PWR101, J_PWR102: footprint PinSocket_2x06_P2.54mm_Vertical -> Connector_PinSocket_2.54mm:PinSocket_2x06_P2.54mm_Vertical
- J_PWR301: footprint PinHeader_2x06_P2.54mm_Vertical -> Connector_PinHeader_2.54mm:PinHeader_2x06_P2.54mm_Vertical
- LCDDisplay1601: footprint PinHeader_1x15_P2.54mm_Vertical -> Connector_PinHeader_2.54mm:PinHeader_1x15_P2.54mm_Vertical
- NT101, NT1601, NT1602: footprint NetTie-2_SMD_Pad2.0mm -> NetTie:NetTie-2_SMD_Pad2.0mm
- NT1603: footprint NetTie-2_SMD_Pad0.5mm -> NetTie:NetTie-2_SMD_Pad0.5mm
- Q401, Q402: footprint SOT-23 -> Package_TO_SOT_SMD:SOT-23
- R1001, R1002, R1003, R1004, R1006, R1007, R1008, R1009, R1010, R1012, R1601, R1602, R1603, R1604, R1606, R1607, R1608, R1609, R1610, R1611, R1612, R1613, R1614, R1615, R1616, R1617, R1618, R1619, R1620, R1651, R1652, R1653, R1654, R1655, R1656, R1657, R1658, R1659, R1660, R1661, R1662, R401, R410, R411, R412, R413, R501, R502, R503, R504, R601, R602, R603, R604, R606, R607, R608, R609, R610, R612, R701, R702, R703, R704, R706, R707, R708, R709, R710, R712, R801, R802, R803, R804, R806, R807, R808, R809, R810, R812, R901, R902, R903, R904, R906, R907, R908, R909, R910, R912: footprint R_1206_3216Metric_Pad1.30x1.75mm_HandSolder -> Resistor_SMD:R_1206_3216Metric_Pad1.30x1.75mm_HandSolder
- RV501, RV502: footprint PinHeader_1x06_P2.54mm_Vertical -> Connector_PinHeader_2.54mm:PinHeader_1x06_P2.54mm_Vertical
- SW402: footprint PinHeader_1x02_P2.54mm_Vertical -> Connector_PinHeader_2.54mm:PinHeader_1x02_P2.54mm_Vertical
- TP1601: footprint TestPoint_Pad_D1.5mm -> TestPoint:TestPoint_Pad_D1.5mm
- U1601, U1602, U1603, U1605, U1606, U1608, U1611: footprint SOIC-8_3.9x4.9mm_P1.27mm -> Package_SO:SOIC-8_3.9x4.9mm_P1.27mm
- U1607, U403: footprint BP5293-50_ROHM_SIP-3 -> Library:BP5293-50_ROHM_SIP-3
- U1609: footprint SOT-23-5_HandSoldering -> Package_TO_SOT_SMD:SOT-23-5_HandSoldering
- U1610, U_IO301: footprint DIP-28_W7.62mm -> Package_DIP:DIP-28_W7.62mm
- U201: footprint REC20K-Z_1in_THT -> Library:REC20K-Z_1in_THT
- U202: footprint TO-220-3_Vertical -> Package_TO_SOT_THT:TO-220-3_Vertical
- U311, U312, U313: footprint TSSOP-16_4.4x5mm_P0.65mm -> Package_SO:TSSOP-16_4.4x5mm_P0.65mm
- U402: footprint SOIC-28W_7.5x17.9mm_P1.27mm -> Package_SO:SOIC-28W_7.5x17.9mm_P1.27mm
- Y1601: footprint Oscillator_SMD_Abracon_ASFL-4Pin_5.0x3.2mm_HandSoldering -> Library:Oscillator_SMD_Abracon_ASFL-4Pin_5.0x3.2mm_HandSoldering
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Connections:
- A1601 pad 1: (no net) -> /MeasureControl/VINL+
- A1601 pad 10: (no net) -> /MeasureControl/ADC_DATA
- A1601 pad 11: (no net) -> /MeasureControl/ADC_nRST
- A1601 pad 12: (no net) -> /MeasureControl/+5V_A
- A1601 pad 13: (no net) -> /MeasureControl/+3V3_A
- A1601 pad 14: (no net) -> /MeasureControl/ADC_GND
- A1601 pad 2: (no net) -> /MeasureControl/VCOML
- A1601 pad 3: (no net) -> /MeasureControl/VINL-
- A1601 pad 4: (no net) -> /MeasureControl/VINR-
- A1601 pad 5: (no net) -> /MeasureControl/VCOMR
- A1601 pad 6: (no net) -> /MeasureControl/VINR+
- A1601 pad 7: (no net) -> /MeasureControl/ADC_MCLK
- A1601 pad 8: (no net) -> /MeasureControl/ADC_LRCK
- A1601 pad 9: (no net) -> /MeasureControl/ADC_BCK
- A1602 pad 1: (no net) -> /MeasureControl/ADC_DATA
- A1602 pad 10: (no net) -> /MeasureControl/LCD_RST
- A1602 pad 11: (no net) -> /MeasureControl/LCD_EN
- A1602 pad 12: (no net) -> unconnected-(A1602-GPIO9-Pad12)
- A1602 pad 13: (no net) -> /D_GND
- A1602 pad 14: (no net) -> /MeasureControl/TP_SDA
- A1602 pad 15: (no net) -> /MeasureControl/TP_SCL
- A1602 pad 16: (no net) -> /MeasureControl/TP_INT
- A1602 pad 17: (no net) -> /MeasureControl/TP_RST
- A1602 pad 18: (no net) -> /D_GND
- A1602 pad 19: (no net) -> unconnected-(A1602-GPIO14-Pad19)
- A1602 pad 2: (no net) -> /MeasureControl/ADC_BCK
- A1602 pad 20: (no net) -> /MeasureControl/ADC_nMR
- A1602 pad 21: (no net) -> /MeasureControl/ENC_INTA
- A1602 pad 22: (no net) -> /MeasureControl/ENC_INTB
- A1602 pad 23: (no net) -> /D_GND
- A1602 pad 24: (no net) -> /MeasureControl/LCD_SCK
- A1602 pad 25: (no net) -> /MeasureControl/LCD_MOSI
- A1602 pad 26: (no net) -> /I2C_SDA
- A1602 pad 27: (no net) -> /I2C_SCL
- A1602 pad 28: (no net) -> /D_GND
- A1602 pad 29: (no net) -> unconnected-(A1602-GPIO22-Pad29)
- A1602 pad 3: (no net) -> /D_GND
- A1602 pad 30: (no net) -> /3V3
- A1602 pad 31: (no net) -> /MeasureControl/DEST_ADC
- A1602 pad 32: (no net) -> unconnected-(A1602-GPIO27_ADC1-Pad32)
- A1602 pad 33: (no net) -> unconnected-(A1602-AGND-Pad33)
- A1602 pad 34: (no net) -> unconnected-(A1602-GPIO28_ADC2-Pad34)
- A1602 pad 35: (no net) -> /3V3
- A1602 pad 36: (no net) -> /3V3
- A1602 pad 37: (no net) -> unconnected-(A1602-3V3_EN-Pad37)
- A1602 pad 38: (no net) -> /D_GND
- A1602 pad 39: (no net) -> Net-(A1602-VSYS)
- A1602 pad 4: (no net) -> /MeasureControl/ADC_LRCK
- A1602 pad 40: (no net) -> unconnected-(A1602-VBUS-Pad40)
- A1602 pad 5: (no net) -> unconnected-(A1602-GPIO3-Pad5)
- A1602 pad 6: (no net) -> unconnected-(A1602-GPIO4-Pad6)
- A1602 pad 7: (no net) -> /MeasureControl/LCD_CS
- A1602 pad 8: (no net) -> /D_GND
- A1602 pad 9: (no net) -> /MeasureControl/LCD_DC
- AMP1001 pad 1: (no net) -> Net-(AMP1001-Pad1)
- AMP1001 pad 2: (no net) -> Net-(AMP1001A--)
- AMP1001 pad 3: (no net) -> Net-(AMP1001A-+)
- AMP1001 pad 4: (no net) -> /-15V
- AMP1001 pad 5: (no net) -> Net-(AMP1001B-+)
- AMP1001 pad 6: (no net) -> Net-(AMP1001B--)
- AMP1001 pad 7: (no net) -> Net-(AMP1001-Pad7)
- AMP1001 pad 8: (no net) -> /+15V
- AMP601 pad 1: (no net) -> Net-(AMP601-Pad1)
- AMP601 pad 2: (no net) -> Net-(AMP601A--)
- AMP601 pad 3: (no net) -> Net-(AMP601A-+)
- AMP601 pad 4: (no net) -> /-15V
- AMP601 pad 5: (no net) -> Net-(AMP601B-+)
- AMP601 pad 6: (no net) -> Net-(AMP601B--)
- AMP601 pad 7: (no net) -> Net-(AMP601-Pad7)
- AMP601 pad 8: (no net) -> /+15V
- AMP701 pad 1: (no net) -> Net-(AMP701-Pad1)
- AMP701 pad 2: (no net) -> Net-(AMP701A--)
- AMP701 pad 3: (no net) -> Net-(AMP701A-+)
- AMP701 pad 4: (no net) -> /-15V
- AMP701 pad 5: (no net) -> Net-(AMP701B-+)
- AMP701 pad 6: (no net) -> Net-(AMP701B--)
- AMP701 pad 7: (no net) -> Net-(AMP701-Pad7)
- AMP701 pad 8: (no net) -> /+15V
- AMP801 pad 1: (no net) -> Net-(AMP801-Pad1)
- AMP801 pad 2: (no net) -> Net-(AMP801A--)
- AMP801 pad 3: (no net) -> Net-(AMP801A-+)
- AMP801 pad 4: (no net) -> /-15V
- AMP801 pad 5: (no net) -> Net-(AMP801B-+)
- AMP801 pad 6: (no net) -> Net-(AMP801B--)
- AMP801 pad 7: (no net) -> Net-(AMP801-Pad7)
- AMP801 pad 8: (no net) -> /+15V
- AMP901 pad 1: (no net) -> Net-(AMP901-Pad1)
- AMP901 pad 2: (no net) -> Net-(AMP901A--)
- AMP901 pad 3: (no net) -> Net-(AMP901A-+)
- AMP901 pad 4: (no net) -> /-15V
- AMP901 pad 5: (no net) -> Net-(AMP901B-+)
- AMP901 pad 6: (no net) -> Net-(AMP901B--)
- AMP901 pad 7: (no net) -> Net-(AMP901-Pad7)
- AMP901 pad 8: (no net) -> /+15V
- C1001 pad 1: (no net) -> Net-(C1001-Pad1)
- C1001 pad 2: (no net) -> /AmpBankSwitch/CH5_OUT_L
- C1002 pad 1: (no net) -> /TONE_L
- C1002 pad 2: (no net) -> Net-(AMP1001A-+)
- C1004 pad 1: (no net) -> /AmpBankSwitch/CH5_OUT_R
- C1004 pad 2: (no net) -> Net-(C1004-Pad2)
- C1005 pad 1: (no net) -> /TONE_R
- C1005 pad 2: (no net) -> Net-(AMP1001B-+)
- C1007 pad 1: (no net) -> /A_GND
- C1007 pad 2: (no net) -> /+15V
- C1008 pad 1: (no net) -> /+15V
- C1008 pad 2: (no net) -> /A_GND
- C1009 pad 1: (no net) -> /A_GND
- C1009 pad 2: (no net) -> /-15V
- C1010 pad 1: (no net) -> /-15V
- C1010 pad 2: (no net) -> /A_GND
- C1601 pad 1: (no net) -> /MeasureControl/ADC_GND
- C1601 pad 2: (no net) -> /MeasureControl/+3V3_A
- C1602 pad 1: (no net) -> Net-(C1602-Pad1)
- C1602 pad 2: (no net) -> Net-(U1602A-OUTA)
- C1603 pad 1: (no net) -> /MeasureControl/+3V3_A
- C1603 pad 2: (no net) -> /MeasureControl/ADC_GND
- C1604 pad 1: (no net) -> /MeasureControl/+3V3_A
- C1604 pad 2: (no net) -> /MeasureControl/ADC_GND
- C1605 pad 1: (no net) -> /+15V
- C1605 pad 2: (no net) -> /MeasureControl/ADC_GND
- C1606 pad 1: (no net) -> /+15V
- C1606 pad 2: (no net) -> /MeasureControl/ADC_GND
- C1607 pad 1: (no net) -> /MeasureControl/ADC_GND
- C1607 pad 2: (no net) -> /MeasureControl/VCOML
- C1608 pad 1: (no net) -> Net-(U1603-BYP)
- C1608 pad 2: (no net) -> /MeasureControl/ADC_GND
- C1609 pad 1: (no net) -> Net-(U1601A-OUTA)
- C1609 pad 2: (no net) -> Net-(U1601A-INA-)
- C1610 pad 1: (no net) -> /PD_12V_SW
- C1610 pad 2: (no net) -> /PD_GND
- C1611 pad 1: (no net) -> /PD_12V_SW
- C1611 pad 2: (no net) -> /PD_GND
- C1612 pad 1: (no net) -> /PD_12V_SW
- C1612 pad 2: (no net) -> /PD_GND
- C1613 pad 1: (no net) -> Net-(C1613-Pad1)
- C1613 pad 2: (no net) -> /MeasureControl/ADC_BUF_R
- C1614 pad 1: (no net) -> /MeasureControl/+3V3_A
- C1614 pad 2: (no net) -> /MeasureControl/ADC_GND
- C1615 pad 1: (no net) -> /MeasureControl/ADC_GND
- C1615 pad 2: (no net) -> /MeasureControl/VCOMR
- C1616 pad 1: (no net) -> /MeasureControl/+5V_A
- C1616 pad 2: (no net) -> /MeasureControl/ADC_GND
- C1617 pad 1: (no net) -> /MeasureControl/+5V_A
- C1617 pad 2: (no net) -> /MeasureControl/ADC_GND
- C1618 pad 1: (no net) -> /+15V
- C1618 pad 2: (no net) -> /MeasureControl/ADC_GND
- C1619 pad 1: (no net) -> /+15V
- C1619 pad 2: (no net) -> /MeasureControl/ADC_GND
- C1620 pad 1: (no net) -> Net-(U1601B-OUTB)
- C1620 pad 2: (no net) -> Net-(U1601B-INB-)
- C1621 pad 1: (no net) -> /MeasureControl/+5V_D
- C1621 pad 2: (no net) -> /D_GND
- C1622 pad 1: (no net) -> /MeasureControl/+5V_D
- C1622 pad 2: (no net) -> /D_GND
- C1623 pad 1: (no net) -> Net-(U1606-BYP)
- C1623 pad 2: (no net) -> /MeasureControl/ADC_GND
- C1624 pad 1: (no net) -> /MeasureControl/+5V_A
- C1624 pad 2: (no net) -> /MeasureControl/ADC_GND
- C1625 pad 1: (no net) -> /MeasureControl/ADC_GND
- C1625 pad 2: (no net) -> /MeasureControl/+3V3_A
- C1626 pad 1: (no net) -> Net-(C1626-Pad1)
- C1626 pad 2: (no net) -> Net-(U1602B-OUTB)
- C1627 pad 1: (no net) -> Net-(U1608A-OUTA)
- C1627 pad 2: (no net) -> Net-(U1608A-INA-)
- C1628 pad 1: (no net) -> Net-(C1628-Pad1)
- C1628 pad 2: (no net) -> /MeasureControl/ADC_BUF_L
- C1629 pad 1: (no net) -> /D_GND
- C1629 pad 2: (no net) -> /MeasureControl/LCD_VCC
- C1630 pad 1: (no net) -> /MeasureControl/LCD_VCC
- C1630 pad 2: (no net) -> /D_GND
- C1631 pad 1: (no net) -> /MeasureControl/LCD_VCC
- C1631 pad 2: (no net) -> /D_GND
- C1632 pad 1: (no net) -> Net-(U1608B-OUTB)
- C1632 pad 2: (no net) -> Net-(U1608B-INB-)
- C1633 pad 1: (no net) -> /MeasureControl/+5V_D
- C1633 pad 2: (no net) -> /D_GND
- C1634 pad 1: (no net) -> /+15V
- C1634 pad 2: (no net) -> /A_GND
- C1635 pad 1: (no net) -> /+15V
- C1635 pad 2: (no net) -> /A_GND
- C1636 pad 1: (no net) -> /+15V
- C1636 pad 2: (no net) -> /A_GND
- C1637 pad 1: (no net) -> /+15V
- C1637 pad 2: (no net) -> /A_GND
- C1638 pad 1: (no net) -> /+15V
- C1638 pad 2: (no net) -> /A_GND
- C1639 pad 1: (no net) -> /A_GND
- C1639 pad 2: (no net) -> /-15V
- C1640 pad 1: (no net) -> /A_GND
- C1640 pad 2: (no net) -> /-15V
- C1641 pad 1: (no net) -> /A_GND
- C1641 pad 2: (no net) -> /-15V
- C1642 pad 1: (no net) -> /A_GND
- C1642 pad 2: (no net) -> /-15V
- C1643 pad 1: (no net) -> /A_GND
- C1643 pad 2: (no net) -> /-15V
- C1645 pad 1: (no net) -> /MeasureControl/PD_12V_MEAS
- C1645 pad 2: (no net) -> /D_GND
- C1646 pad 1: (no net) -> /+15V
- C1646 pad 2: (no net) -> /A_GND
- C1647 pad 1: (no net) -> /A_GND
- C1647 pad 2: (no net) -> /-15V
- C1650 pad 1: (no net) -> /3V3
- C1650 pad 2: (no net) -> /D_GND
- C201 pad 1: (no net) -> /+15V
- C201 pad 2: (no net) -> /A_GND
- C202 pad 1: (no net) -> /+15V
- C202 pad 2: (no net) -> /A_GND
- C203 pad 1: (no net) -> /VCC_TONE
- C203 pad 2: (no net) -> /A_GND
- C204 pad 1: (no net) -> /VCC_TONE
- C204 pad 2: (no net) -> /A_GND
- C205 pad 1: (no net) -> /PD_GND
- C205 pad 2: (no net) -> Net-(U201-+Vin)
- C206 pad 1: (no net) -> /PD_GND
- C206 pad 2: (no net) -> Net-(U201-+Vin)
- C207 pad 1: (no net) -> /A_GND
- C207 pad 2: (no net) -> /-15V
- C208 pad 1: (no net) -> /A_GND
- C208 pad 2: (no net) -> /-15V
- C311 pad 1: (no net) -> /+15V
- C311 pad 2: (no net) -> /A_GND
- C312 pad 1: (no net) -> /A_GND
- C312 pad 2: (no net) -> /-15V
- C313 pad 1: (no net) -> /+15V
- C313 pad 2: (no net) -> /A_GND
- C314 pad 1: (no net) -> /A_GND
- C314 pad 2: (no net) -> /-15V
- C315 pad 1: (no net) -> /+15V
- C315 pad 2: (no net) -> /A_GND
- C316 pad 1: (no net) -> /A_GND
- C316 pad 2: (no net) -> /-15V
- C401 pad 1: (no net) -> /PT_REF
- C401 pad 2: (no net) -> /A_GND
- C402 pad 1: (no net) -> /VCC_TONE
- C402 pad 2: (no net) -> /A_GND
- C403 pad 1: (no net) -> /PT_BOUT_L
- C403 pad 2: (no net) -> /PT_BASS_L
- C404 pad 1: (no net) -> /PT_BOUT_R
- C404 pad 2: (no net) -> /PT_BASS_R
- C405 pad 1: (no net) -> /PT_OUT_L
- C405 pad 2: (no net) -> /TONE_L
- C406 pad 1: (no net) -> /COMMON_L
- C406 pad 2: (no net) -> /PT_LIN
- C407 pad 1: (no net) -> /COMMON_R
- C407 pad 2: (no net) -> /PT_RIN
- C408 pad 1: (no net) -> /PT_TREB_L
- C408 pad 2: (no net) -> /A_GND
- C409 pad 1: (no net) -> /PT_OUT_R
- C409 pad 2: (no net) -> /TONE_R
- C410 pad 1: (no net) -> /PT_BIN_L
- C410 pad 2: (no net) -> /PT_BASS_L
- C411 pad 1: (no net) -> /PT_BIN_R
- C411 pad 2: (no net) -> /PT_BASS_R
- C412 pad 1: (no net) -> /PT_TREB_R
- C412 pad 2: (no net) -> /A_GND
- C501 pad 1: (no net) -> /HP_RC_L
- C501 pad 2: (no net) -> /PHONE_L
- C502 pad 1: (no net) -> /HP_RC_R
- C502 pad 2: (no net) -> /PHONE_R
- C503 pad 1: (no net) -> /+15V
- C503 pad 2: (no net) -> /A_GND
- C504 pad 1: (no net) -> /A_GND
- C504 pad 2: (no net) -> /-15V
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
Commit message: AudioV2: C501/C502 を Ø16/P7.5 に（Muse ES 470µF が入る）
HP 出力の無極性ブロックを UES1E471MHM クラスの寸法に合わせた。

Co-authored-by: Cursor <cursoragent@cursor.com>
Parts:
- C501, C502: footprint Capacitor_THT:CP_Radial_D10.0mm_P5.00mm -> Capacitor_THT:CP_Radial_D16.0mm_P7.50mm
Changed lines of the file:
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@@
 		)
 	)
-	(footprint "Capacitor_THT:CP_Radial_D10.0mm_P5.00mm"
+	(footprint "Capacitor_THT:CP_Radial_D16.0mm_P7.50mm"
 		(layer "F.Cu")
 		(at 10 25)
-		(descr "CP, Radial series, Radial, pin pitch=5.00mm, diameter=10mm, height=16mm, Electrolytic Capacitor")
-		(tags "CP Radial series Radial pin pitch 5.00mm diameter 10mm height 16mm Electrolytic Capacitor")
+		(descr "CP, Radial series, Radial, pin pitch=7.50mm, diameter=16mm, height=25mm, Electrolytic Capacitor")
+		(tags "CP Radial series Radial pin pitch 7.50mm diameter 16mm height 25mm Electrolytic Capacitor")
 		(property "Reference" "C501"
-			(at 2.5 -6.25 0)
+			(at 3.75 -9.25 0)
 			(layer "F.SilkS")
 			(effects
@@
 		)
 		(property "Value" "470uF 25V NP"
-			(at 2.5 6.25 0)
+			(at 3.75 9.25 0)
 			(layer "F.Fab")
 			(effects
@@
 		)
 		(fp_circle
-			(center 2.5 0)
+			(center 3.75 0)
 			(end 7.62 0)
 			(stroke
@@
 		)
 		(fp_circle
-			(center 2.5 0)
+			(center 3.75 0)
 			(end 7.75 0)
 			(stroke
@@
 		)
 		(fp_circle
-			(center 2.5 0)
+			(center 3.75 0)
 			(end 7.5 0)
 			(stroke
@@
 		(pad "1" thru_hole roundrect
 			(at 0 0)
-			(size 2 2)
-			(drill 1)
+			(size 2.4 2.4)
+			(drill 1.2)
 			(layers "*.Cu" "*.Mask")
 			(remove_unused_layers no)
@@
 		)
 		(pad "2" thru_hole circle
-			(at 5 0)
-			(size 2 2)
-			(drill 1)
+			(at 7.5 0)
+			(size 2.4 2.4)
+			(drill 1.2)
 			(layers "*.Cu" "*.Mask")
 			(remove_unused_layers no)
@@
 		)
 		(embedded_fonts no)
-		(model "${KICAD10_3DMODEL_DIR}/Capacitor_THT.3dshapes/CP_Radial_D10.0mm_P5.00mm.step"
+		(model "${KICAD10_3DMODEL_DIR}/Capacitor_THT.3dshapes/CP_Radial_D16.0mm_P7.50mm.step"
 			(offset
 				(xyz 0 0 0)
@@
 		)
 	)
-	(footprint "Capacitor_THT:CP_Radial_D10.0mm_P5.00mm"
+	(footprint "Capacitor_THT:CP_Radial_D16.0mm_P7.50mm"
 		(layer "F.Cu")
 		(at 25 25)
-		(descr "CP, Radial series, Radial, pin pitch=5.00mm, diameter=10mm, height=16mm, Electrolytic Capacitor")
-		(tags "CP Radial series Radial pin pitch 5.00mm diameter 10mm height 16mm Electrolytic Capacitor")
+		(descr "CP, Radial series, Radial, pin pitch=7.50mm, diameter=16mm, height=25mm, Electrolytic Capacitor")
+		(tags "CP Radial series Radial pin pitch 7.50mm diameter 16mm height 25mm Electrolytic Capacitor")
 		(property "Reference" "C502"
-			(at 2.5 -6.25 0)
+			(at 3.75 -9.25 0)
 			(layer "F.SilkS")
 			(effects
@@
 		)
 		(property "Value" "470uF 25V NP"
-			(at 2.5 6.25 0)
+			(at 3.75 9.25 0)
 			(layer "F.Fab")
 			(effects
@@
 		)
 		(fp_circle
-			(center 2.5 0)
+			(center 3.75 0)
 			(end 7.62 0)
 			(stroke
@@
 		)
 		(fp_circle
-			(center 2.5 0)
+			(center 3.75 0)
 			(end 7.75 0)
 			(stroke
@@
 		)
 		(fp_circle
-			(center 2.5 0)
+			(center 3.75 0)
 			(end 7.5 0)
 			(stroke
@@
 		(pad "1" thru_hole roundrect
 			(at 0 0)
-			(size 2 2)
-			(drill 1)
+			(size 2.4 2.4)
+			(drill 1.2)
 			(layers "*.Cu" "*.Mask")
 			(remove_unused_layers no)
@@
 		)
 		(pad "2" thru_hole circle
-			(at 5 0)
-			(size 2 2)
-			(drill 1)
+			(at 7.5 0)
+			(size 2.4 2.4)
+			(drill 1.2)
 			(layers "*.Cu" "*.Mask")
 			(remove_unused_layers no)
@@
 		)
 		(embedded_fonts no)
-		(model "${KICAD10_3DMODEL_DIR}/Capacitor_THT.3dshapes/CP_Radial_D10.0mm_P5.00mm.step"
+		(model "${KICAD10_3DMODEL_DIR}/Capacitor_THT.3dshapes/CP_Radial_D16.0mm_P7.50mm.step"
 			(offset
 				(xyz 0 0 0)

Commit message: AudioV2: KiCad 保存後の回路図・PCB・pro を取り込み、再生成禁止を NOW に明記
全面 build_*.py は KiCad 保存済みプロジェクトを壊す。以後はピンポイント編集。

Co-authored-by: Cursor <cursoragent@cursor.com>
Parts:
- F201: value T1.6A slow 5x20 -> F2A fast 5x20

Commit message: AudioV2: PCB を sheetpath ゾーン配置し、配線は娘SW→親の順に
アナログスイッチ基板を先に配線する方針を NOW に明記した。

Co-authored-by: Cursor <cursoragent@cursor.com>
Parts:
- moved SW402 463.1 mm to (29.0, 430.0)
- moved SW502 423.5 mm to (85.0, 430.0)
- moved SW501 423.1 mm to (71.0, 430.0)
- moved RV502 417.1 mm to (57.0, 430.0)
- moved RV501 416.8 mm to (43.0, 430.0)
- moved NT1601 394.5 mm to (270.0, 440.0)
- moved NT1602 391.0 mm to (278.0, 440.0)
- moved NT1603 387.6 mm to (286.0, 440.0)
- moved A1602 377.6 mm to (99.0, 430.0)
- moved C1616 369.9 mm to (39.0, 322.0)
- moved J_RAIL501 368.1 mm to (15.0, 264.0)
- moved C1615 367.8 mm to (27.0, 322.0)
- moved C1614 365.8 mm to (15.0, 322.0)
- moved ENC1603 354.4 mm to (169.0, 430.0)
- moved ENC1602 354.2 mm to (155.0, 430.0)
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
Commit message: AudioV2 PCB: AmpCh タイル5枚を TMUX 上下ペアで配置し、娘基板 100x100 の外形を引く
- TMUX7612 は上半分が奇数ch・下半分が偶数ch。DIP-8 は A ユニット(L)が西列で
  固定なので、奇数chはそのまま IC の上、偶数chは 180 度回して下に置くと
  切替出力が交差せず左右対称に着地する（実測 _L 23.75mm / _R 22.44mm、4ch 同値）
- ch1-ch4 を U311/U312 の上下に配置。ch5 は U313 を規定の相対位置へ置いて形を揃えた
- 旧 ch5 の配線 74 本とビア 6 個は U313 移動で無効になるため削除
- Edge.Cuts に娘基板 100x100 を追加（スタック規格 A2 の外形見直し。
  裏面に SMD 82点を回す前提で 80mm から 100mm へ）

Co-authored-by: Cursor <cursoragent@cursor.com>
Parts:
- moved U312 363.7 mm to (413.0, 201.0)
- moved R608 362.1 mm to (376.8, 180.0), turned to 180 degrees
- moved C607 357.9 mm to (371.7, 171.4), turned to 180 degrees
- moved AMP601 347.7 mm to (359.2, 179.4)
- moved C608 346.4 mm to (371.6, 176.9)
- moved R610 338.5 mm to (376.9, 185.5), turned to -90 degrees
- moved R602 336.6 mm to (351.0, 173.9), turned to 180 degrees
- moved C604 336.2 mm to (382.6, 185.1), turned to 90 degrees
- moved U311 327.3 mm to (363.0, 201.0)
- moved R609 322.0 mm to (347.9, 192.2)
- moved C601 321.7 mm to (343.4, 188.2), turned to 90 degrees
- moved R612 320.6 mm to (371.2, 182.2), turned to 90 degrees
- moved C602 320.5 mm to (356.7, 172.0)
- moved C609 319.7 mm to (354.7, 192.3)
- moved R603 318.6 mm to (344.6, 178.4), turned to 180 degrees
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Other:
- board outline added: 100 x 100 mm

Commit message: AudioV2: 娘基板を 4ch 化しスロットを 3 口へ。PCB を回路図に同期
build_daughter.py の AmpCh を 5 -> 4 にし、TMUX7612 を 3 -> 2、リレー版の
ドライバを 2 -> 1 に減らす。母板は SLOT_ADDR に 0x22 を足して 3 口
(J_ANA103 / J_PWR103)。同じスイッチ版を 3 枚まで挿せる。

PCB は全面再生成せず差分だけ合わせた。旧 AmpCh5 一式と U313・そのデカップ
計 22 点を削除し、スロット3のコネクタ 2 点を仮置きで追加。kicad-cli drc の
schematic_parity は 0 件。

Co-authored-by: Cursor <cursoragent@cursor.com>
Parts:
- removed AMP1001: NE5532 / DIP-8 compatible, Package_DIP:DIP-8_W7.62mm_Socket
- removed C1001, C1004: 2.2uF film, Capacitor_THT:C_Rect_L7.2mm_W2.5mm_P5.00mm_FKS2_FKP2_MKS2_MKP2
- removed C1002, C1005: 1uF film, Capacitor_THT:C_Rect_L11.0mm_W4.2mm_P10.00mm_MKT
- removed C1007, C1008, C1009, C1010, C315, C316: 100nF, Capacitor_SMD:C_1206_3216Metric_Pad1.33x1.80mm_HandSolder
- removed R1001, R1007: 100k, Resistor_SMD:R_1206_3216Metric_Pad1.30x1.75mm_HandSolder
- removed R1002, R1008: 47R, Resistor_SMD:R_1206_3216Metric_Pad1.30x1.75mm_HandSolder
- removed R1003, R1009: 220k, Resistor_SMD:R_1206_3216Metric_Pad1.30x1.75mm_HandSolder
- removed R1004, R1006, R1010, R1012: 20k, Resistor_SMD:R_1206_3216Metric_Pad1.30x1.75mm_HandSolder
- removed U313: TMUX7612, Package_SO:TSSOP-16_4.4x5mm_P0.65mm
