File: AudioV2/AudioV2Case.kicad_pcb (KiCad board)
At the start: 2 copper layers, 259 parts, among them J1601 AUDIO, J1602 V_IN, J1603 15_V_IN, J201 +15/A_GND/-15 out, J202 PD module in (1=GND 2=+12V), Q401 BSS138, Q402 BSS138, SW1601 DEST sense (3PDT 3rd pole, sa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, SW402 PWR SW, SW501 DEST L (PHONE/MUTE/LINE), SW502 DEST R (PHONE/MUTE/LINE), U1601 OPA1656, U1602 OPA1656, U1603 LT1763-3.3, U1605 TPS3307-33, U1606 LT1763-5, U1607 BP5293-50, U1608 OPA1656, U1609 XC8107AC20MR-G, U1610 MCP23017 (UI 0x22), U1611 OPA1656, U201 REC20K-2415DZ, U202 L7809CV +9V, U311 TMUX7612, U312 TMUX7612, U402 PT2314E, U403 BP5293-50 +5V, U501 OPA1652, Y1601 ASFL1-12.288MHZ-EC-T

Commit message: AudioV2 PCB: 娘基板の残り10点を配置し AmpBankSwitch 88点を全て盤面へ
上部の空き帯へ U_IO301(MCP23017)・J_PWR301/J_ANA301・±15V バルク2個・
C_IO301 を、TMUX の左に C311-C314 を置いた。部品範囲は 92.3 x 92.2 mm。

コートヤードの重なりは 0。kicad-cli drc で schematic_parity 0、
新規の電気・機械違反なし（増分はリファレンス文字のシルク重なり 9 件のみ）。

配置検証スクリプトの回転規約を修正: KiCad は (x cosθ + y sinθ,
-x sinθ + y cosθ)。符号を逆にしていたため rot90 の部品の bbox が
アンカー基準で反転し、U_IO301 が外形の外に出ていた。

Co-authored-by: Cursor <cursoragent@cursor.com>
Parts:
- moved J_ANA301 390.4 mm to (414.9, 146.3), turned to 90 degrees
- moved C313 375.0 mm to (398.0, 198.5)
- moved C314 364.9 mm to (398.0, 203.0)
- moved J_PWR301 355.4 mm to (391.6, 146.3), turned to 90 degrees
- moved C_IO301 352.6 mm to (364.0, 152.5)
- moved C311 350.2 mm to (348.0, 198.5)
- moved C312 340.3 mm to (348.0, 203.0)
- moved C_BULK_N301 290.0 mm to (368.0, 161.5)
- moved C_BULK_P301 262.9 mm to (352.0, 161.5)
- moved U_IO301 108.6 mm to (347.5, 148.8), turned to 90 degrees
Changed lines of the file:
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@@
 	(footprint "Connector_PinHeader_2.54mm:PinHeader_2x06_P2.54mm_Vertical"
 		(layer "F.Cu")
-		(at 39 102)
+		(at 391.65 146.275 90)
 		(descr "Through hole straight pin header, 2x06, 2.54mm pitch, double rows")
 		(tags "Through hole pin header THT 2x06 2.54mm double row")
@@
 	(footprint "Capacitor_SMD:C_1206_3216Metric_Pad1.33x1.80mm_HandSolder"
 		(layer "F.Cu")
-		(at 15 90)
+		(at 348.0 198.5)
 		(descr "Capacitor SMD 1206 (3216 Metric), square (rectangular) end terminal, IPC-7351 nominal with elongated pad for handsoldering. (Body size source: IPC-SM-782 page 76, https://www.pcb-3d.com/wordpress/wp-content/uploads/ipc-sm-782a_amendment_1_and_2.pdf)")
 		(tags "capacitor handsolder")
@@
 	(footprint "Capacitor_SMD:CP_Elec_10x12.6"
 		(layer "F.Cu")
-		(at 99 90)
+		(at 352.0 161.5)
 		(descr "SMD capacitor, aluminum electrolytic, Panasonic F12, 10.0x12.6mm")
 		(tags "capacitor electrolytic")
@@
 	(footprint "Capacitor_SMD:CP_Elec_10x12.6"
 		(layer "F.Cu")
-		(at 87 90)
+		(at 368.0 161.5)
 		(descr "SMD capacitor, aluminum electrolytic, Panasonic F12, 10.0x12.6mm")
 		(tags "capacitor electrolytic")
@@
 	(footprint "Capacitor_SMD:C_1206_3216Metric_Pad1.33x1.80mm_HandSolder"
 		(layer "F.Cu")
-		(at 51 90)
+		(at 398.0 203.0)
 		(descr "Capacitor SMD 1206 (3216 Metric), square (rectangular) end terminal, IPC-7351 nominal with elongated pad for handsoldering. (Body size source: IPC-SM-782 page 76, https://www.pcb-3d.com/wordpress/wp-content/uploads/ipc-sm-782a_amendment_1_and_2.pdf)")
 		(tags "capacitor handsolder")
@@
 	(footprint "Package_DIP:DIP-28_W7.62mm"
 		(layer "F.Cu")
-		(at 244.98 112.9 -90)
+		(at 347.49 148.805 90)
 		(descr "28-lead though-hole mounted DIP package, row spacing 7.62mm (300 mils)")
 		(tags "THT DIP DIL PDIP 2.54mm 7.62mm 300mil")
@@
 	(footprint "Capacitor_SMD:C_1206_3216Metric_Pad1.33x1.80mm_HandSolder"
 		(layer "F.Cu")
-		(at 39 90)
+		(at 398.0 198.5)
 		(descr "Capacitor SMD 1206 (3216 Metric), square (rectangular) end terminal, IPC-7351 nominal with elongated pad for handsoldering. (Body size source: IPC-SM-782 page 76, https://www.pcb-3d.com/wordpress/wp-content/uploads/ipc-sm-782a_amendment_1_and_2.pdf)")
 		(tags "capacitor handsolder")
@@
 	(footprint "Connector_PinHeader_2.54mm:PinHeader_2x05_P2.54mm_Vertical"
 		(layer "F.Cu")
-		(at 27 102)
+		(at 414.92 146.275 90)
 		(descr "Through hole straight pin header, 2x05, 2.54mm pitch, double rows")
 		(tags "Through hole pin header THT 2x05 2.54mm double row")
@@
 	(footprint "Capacitor_SMD:C_1206_3216Metric_Pad1.33x1.80mm_HandSolder"
 		(layer "F.Cu")
-		(at 15 102)
+		(at 364.0 152.5)
 		(descr "Capacitor SMD 1206 (3216 Metric), square (rectangular) end terminal, IPC-7351 nominal with elongated pad for handsoldering. (Body size source: IPC-SM-782 page 76, https://www.pcb-3d.com/wordpress/wp-content/uploads/ipc-sm-782a_amendment_1_and_2.pdf)")
 		(tags "capacitor handsolder")
@@
 	(footprint "Capacitor_SMD:C_1206_3216Metric_Pad1.33x1.80mm_HandSolder"
 		(layer "F.Cu")
-		(at 27 90)
+		(at 348.0 203.0)
 		(descr "Capacitor SMD 1206 (3216 Metric), square (rectangular) end terminal, IPC-7351 nominal with elongated pad for handsoldering. (Body size source: IPC-SM-782 page 76, https://www.pcb-3d.com/wordpress/wp-content/uploads/ipc-sm-782a_amendment_1_and_2.pdf)")
 		(tags "capacitor handsolder")
