File: AudioV2/AudioV2Case.kicad_pcb (KiCad board)
At the start: 2 copper layers, 259 parts, among them J1601 AUDIO, J1602 V_IN, J1603 15_V_IN, J201 +15/A_GND/-15 out, J202 PD module in (1=GND 2=+12V), Q401 BSS138, Q402 BSS138, SW1601 DEST sense (3PDT 3rd pole, sa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, SW402 PWR SW, SW501 DEST L (PHONE/MUTE/LINE), SW502 DEST R (PHONE/MUTE/LINE), U1601 OPA1656, U1602 OPA1656, U1603 LT1763-3.3, U1605 TPS3307-33, U1606 LT1763-5, U1607 BP5293-50, U1608 OPA1656, U1609 XC8107AC20MR-G, U1610 MCP23017 (UI 0x22), U1611 OPA1656, U201 REC20K-2415DZ, U202 L7809CV +9V, U311 TMUX7612, U312 TMUX7612, U402 PT2314E, U403 BP5293-50 +5V, U501 OPA1652, Y1601 ASFL1-12.288MHZ-EC-T

Commit message: AudioV2 PCB: 娘基板を 110x110 にしコネクタを A2 の勘合座標へ置く
A2 の 100x80 は 4ch では成立しない。タイル4枚だけで 92.3 x 62.7 あり、
M3 を端 5mm に置くと 100mm 幅に収まらない（左右に 3.85mm しか残らない）。
A2 自身が「初版なので PCB 着手時に数値は見直す」と書いている箇所。

A2 の規則は維持した: pin1 の X = 20.00 / 60.00、各コネクタは自分の辺から
10.00mm、両版共通、2x5 と 2x6 のキーイング。高さだけ再計算して
J_PWR_CTRL の pin1 が (60.00, 97.46) になった（80-12.54 -> 110-12.54）。
J_ANA は (20.00, 10.00) のまま。全ピン座標を仕様と照合して一致を確認。

タイル群 82 点を (+7.0, -9.37) 平行移動、上帯を組み直してバルクを
J_PWR301 の真下へ（電源入口から遠い問題を解消）。C_IO301 は U_IO301 の
VDD/VSS の真下。娘領域の重なり 0・外形はみ出し 0・M3 キープアウト干渉 0。
外形拡大で copper_edge_clearance 8 件が解消。schematic_parity は 0 のまま。

⚠ M3 穴はまだ置いていない。⚠ 母板は 3 枚 x 110mm が横に並ばない。

Co-authored-by: Cursor <cursoragent@cursor.com>
Parts:
- moved J_ANA301 100.1 mm to (360.0, 230.0)
- moved C_BULK_P301 50.6 mm to (401.8, 152.6)
- moved C_BULK_N301 49.6 mm to (416.8, 152.6)
- moved AMP701 11.7 mm to (373.8, 213.2)
- moved AMP901 11.7 mm to (423.8, 213.2)
- moved C311 11.7 mm to (355.0, 189.1)
- moved C312 11.7 mm to (355.0, 193.6)
- moved C313 11.7 mm to (405.0, 189.1)
- moved C314 11.7 mm to (405.0, 193.6)
- moved C601 11.7 mm to (350.4, 178.8)
- moved C605 11.7 mm to (366.9, 183.3)
- moved C607 11.7 mm to (378.7, 162.0)
- moved C608 11.7 mm to (378.6, 167.5)
- moved C609 11.7 mm to (361.7, 182.9)
- moved C610 11.7 mm to (361.7, 178.0)
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
Commit message: AudioV2 PCB: 娘基板の電源デカップ 100nF を裏面へ
ソケットは表面のまま、セラミック 21 個だけ B.Cu に回す。DIP の V+/V−
ピン脇と TMUX / MCP の電源ピン直下。DIP ピンは表裏導通済み。
TMUX（TSSOP）だけ配線時にビアが要る。

バルク電解 2 個は高さ 12.6mm のため表面に残す（基板間 15mm に裏面から
出さない）。裏面テキストはミラー DRC を避けるため隠した。
schematic_parity は 0 のまま。

Co-authored-by: Cursor <cursoragent@cursor.com>
Parts:
- C311, C312, C313, C314, C607, C608, C609, C610, C707, C708, C709, C710, C807, C808, C809, C810, C907, C908, C909, C910, C_IO301: moved to B.Cu
- moved C311 17.9 mm to (372.9, 189.7), turned to 90 degrees
- moved C313 17.9 mm to (422.9, 189.7), turned to 90 degrees
- moved C312 12.2 mm to (367.1, 192.9), turned to 90 degrees
- moved C314 12.2 mm to (417.1, 192.9), turned to 90 degrees
- moved C608 8.82 mm to (370.2, 170.1)
- moved C808 8.82 mm to (420.2, 170.1)
- moved C708 8.82 mm to (369.8, 213.2)
- moved C908 8.82 mm to (419.8, 213.2)
- moved C607 8.73 mm to (375.4, 170.1)
- moved C807 8.73 mm to (425.4, 170.1)
- moved C707 8.73 mm to (364.6, 213.2)
- moved C907 8.73 mm to (414.6, 213.2)
- moved C610 8.12 mm to (369.8, 177.7)
- moved C710 8.12 mm to (370.2, 205.6)
- moved C810 8.12 mm to (419.8, 177.7)
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
Commit message: 娘基板に GND ベタを敷き、回路図から来た 6 部品を配置し直す
回路図側で足した M3 取付穴 4 個とスロット 3 のコネクタ 2 個が、KiCad の
「回路図から基板を更新」で自動配置の山として入ってきたので、A2 の座標へ移した。
穴は四隅 5.0 mm、コネクタは既存 2 スロットと同じ並び。

ベタは 4 枚。`A_GND` を 110×110 全面（外形から 0.5 mm 内側）に表裏、`D_GND` を
MCP と `J_PWR301` のデジタル帯だけ表裏で優先度を上げて重ねる。スターグランドの
NetTie を跨がせないため、1 枚のベタで済ませずドメインごとに分けている。

配線は未着手（トラック 0）。フットプリント 265・ゾーン 4。

Co-authored-by: Cursor <cursoragent@cursor.com>
Parts:
- added H301: M3, MountingHole:MountingHole_3.2mm_M3, F.Cu at (345.0, 235.0)
- added H302: M3, MountingHole:MountingHole_3.2mm_M3, F.Cu at (445.0, 235.0)
- added H303: M3, MountingHole:MountingHole_3.2mm_M3, F.Cu at (345.0, 135.0)
- added H304: M3, MountingHole:MountingHole_3.2mm_M3, F.Cu at (445.0, 135.0)
- added J_ANA103: SLOT3 ANA (D18), Connector_PinSocket_2.54mm:PinSocket_2x05_P2.54mm_Vertical, F.Cu at (135.0, 15.0)
- added J_PWR103: SLOT3 PWR/CTRL (D18), Connector_PinSocket_2.54mm:PinSocket_2x06_P2.54mm_Vertical, F.Cu at (147.0, 15.0)
- C311, C312: moved to F.Cu
- R603: moved to B.Cu
- moved U_IO301 41.3 mm to (389.9, 139.1), turned to -90 degrees
- moved C_BULK_N301 41.0 mm to (405.0, 191.9)
- moved C_BULK_P301 40.4 mm to (390.8, 191.4)
- moved R609 24.4 mm to (378.7, 188.2)
- moved C602 23.2 mm to (345.4, 176.8)
- moved R602 17.8 mm to (356.1, 182.2)
- moved R603 14.8 mm to (357.7, 182.5)
- moved C_IO301 11.6 mm to (371.2, 143.1)
- moved C601 8.71 mm to (354.5, 186.5), turned to 0 degrees
- moved C311 6.14 mm to (378.8, 191.3), turned to 0 degrees
- moved C312 6.09 mm to (361.3, 191.3), turned to 0 degrees
- moved R601 3.84 mm to (361.5, 176.5)
- moved R604 3.04 mm to (357.3, 172.2)
- moved C607 2.81 mm to (378.2, 169.9)
- moved C609 2.71 mm to (361.9, 177.7)
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Connections:
- U_IO301 pad 25: /AmpBankSwitch/SEL_CH5 -> unconnected-(U_IO301-GPA4-Pad25)
Routing:
- net /3V3: track 0.00 -> 53.3 mm
- net /I2C_SCL: track 0.00 -> 52.7 mm
- net /I2C_SDA: track 0.00 -> 51.3 mm, vias 0 -> 1
- net /-15V: track 0.00 -> 23.3 mm, vias 0 -> 1
- net Net-(AMP601-Pad1): track 0.00 -> 20.8 mm
- net /A_GND: track 0.00 -> 15.3 mm, vias 0 -> 1
- net /AmpBankSwitch/CH1_OUT_L: track 0.00 -> 13.4 mm
- net Net-(AMP601A--): track 0.00 -> 7.68 mm
- net /AmpBankSwitch/CH1_OUT_R: track 0.00 -> 5.63 mm
- net /+15V: track 0.00 -> 4.38 mm
- net Net-(AMP601A-+): track 0.00 -> 3.67 mm
- added copper zone on B.Cu, net /A_GND
- added copper zone on F.Cu, net /A_GND
- added copper zone on B.Cu, net /D_GND
- added copper zone on F.Cu, net /D_GND

Commit message: AudioV2: TMUX 案C（90°+ピン再割当）と Amp 入力カップリング再配置
PCB 配置に合わせて S↔D・ch 組・SEL 結びを変え、U311 周りを引き出し配線。
C602/C605/C702/C705 はソケット脇へ移し、3層化は保留。

Co-authored-by: Cursor <cursoragent@cursor.com>
Parts:
- C311, C312: moved to B.Cu
- R603: moved to F.Cu
- moved C705 36.0 mm to (342.0, 218.0), turned to 0 degrees
- moved C605 29.3 mm to (396.0, 180.0), turned to 180 degrees
- moved C702 23.0 mm to (395.6, 208.1)
- moved R703 22.0 mm to (374.0, 197.5)
- moved C704 19.5 mm to (368.4, 200.0), turned to 180 degrees
- moved C604 19.4 mm to (371.6, 183.0), turned to 0 degrees
- moved R709 19.3 mm to (366.0, 197.5)
- moved R702 16.6 mm to (381.5, 202.2), turned to 90 degrees
- moved C701 13.7 mm to (376.6, 200.0), turned to 180 degrees
- moved R608 11.1 mm to (381.5, 181.5), turned to 90 degrees
- moved R708 10.8 mm to (358.0, 202.0), turned to -90 degrees
- moved C601 9.54 mm to (363.4, 183.0)
- moved C311 9.47 mm to (369.7, 188.8)
- moved C312 9.00 mm to (369.7, 194.5)
- moved R603 8.84 mm to (366.0, 185.5)
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Connections:
- U311 pad 1: /AmpBankSwitch/SEL_CH1 -> /AmpBankSwitch/SEL_CH2
- U311 pad 10: /AMP_SEL_L -> /AmpBankSwitch/CH1_OUT_R
- U311 pad 11: /AmpBankSwitch/CH2_OUT_L -> /AMP_SEL_R
- U311 pad 14: /AmpBankSwitch/CH1_OUT_R -> /AMP_SEL_L
- U311 pad 15: /AMP_SEL_R -> /AmpBankSwitch/CH1_OUT_L
- U311 pad 2: /AMP_SEL_L -> /AmpBankSwitch/CH2_OUT_R
- U311 pad 3: /AmpBankSwitch/CH1_OUT_L -> /AMP_SEL_R
- U311 pad 6: /AmpBankSwitch/CH2_OUT_R -> /AMP_SEL_L
- U311 pad 7: /AMP_SEL_R -> /AmpBankSwitch/CH2_OUT_L
- U311 pad 9: /AmpBankSwitch/SEL_CH2 -> /AmpBankSwitch/SEL_CH1
- U312 pad 1: /AmpBankSwitch/SEL_CH3 -> /AmpBankSwitch/SEL_CH4
- U312 pad 10: /AMP_SEL_L -> /AmpBankSwitch/CH3_OUT_R
- U312 pad 11: /AmpBankSwitch/CH4_OUT_L -> /AMP_SEL_R
- U312 pad 14: /AmpBankSwitch/CH3_OUT_R -> /AMP_SEL_L
- U312 pad 15: /AMP_SEL_R -> /AmpBankSwitch/CH3_OUT_L
- U312 pad 2: /AMP_SEL_L -> /AmpBankSwitch/CH4_OUT_R
- U312 pad 3: /AmpBankSwitch/CH3_OUT_L -> /AMP_SEL_R
- U312 pad 6: /AmpBankSwitch/CH4_OUT_R -> /AMP_SEL_L
- U312 pad 7: /AMP_SEL_R -> /AmpBankSwitch/CH4_OUT_L
- U312 pad 9: /AmpBankSwitch/SEL_CH4 -> /AmpBankSwitch/SEL_CH3
Routing:
- net Net-(AMP701B-+): track 0.00 -> 26.7 mm
- net /-15V: track 23.3 -> 0.00 mm, vias 1 -> 0
- net Net-(AMP701-Pad1): track 0.00 -> 21.5 mm
- net Net-(AMP701-Pad7): track 0.00 -> 19.8 mm
- net Net-(AMP601-Pad7): track 0.00 -> 19.6 mm
- net Net-(AMP601B-+): track 0.00 -> 14.5 mm
- net /AMP_SEL_R: track 0.00 -> 13.7 mm
- net /AMP_SEL_L: track 0.00 -> 13.7 mm
- net Net-(AMP701A-+): track 0.00 -> 11.7 mm
- net /AmpBankSwitch/CH2_OUT_R: track 0.00 -> 8.14 mm
- net /AmpBankSwitch/CH2_OUT_L: track 0.00 -> 8.14 mm
- net Net-(C704-Pad2): track 0.00 -> 5.83 mm
- net Net-(AMP601A-+): track 3.67 -> 9.44 mm
- net Net-(C701-Pad1): track 0.00 -> 5.52 mm
- net /AmpBankSwitch/CH1_OUT_L: track 13.4 -> 8.40 mm
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