File: AudioV2/AudioV2Case.kicad_pcb (KiCad board)
At the start: 2 copper layers, 110 x 110 mm, 265 parts, among them J1601 AUDIO, J1602 V_IN, J1603 15_V_IN, J201 +15/A_GND/-15 out, J202 PD module in (1=GND 2=+12V), Q401 BSS138, Q402 BSS138, SW1601 DEST sense (3PDT 3rd pole, sa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, SW402 PWR SW, SW501 DEST L (PHONE/MUTE/LINE), SW502 DEST R (PHONE/MUTE/LINE), U1601 OPA1656, U1602 OPA1656, U1603 LT1763-3.3, U1605 TPS3307-33, U1606 LT1763-5, U1607 BP5293-50, U1608 OPA1656, U1609 XC8107AC20MR-G, U1610 MCP23017 (UI 0x22), U1611 OPA1656, U201 REC20K-2415DZ, U202 L7809CV +9V, U311 TMUX7612, U312 TMUX7612, U402 PT2314E, U403 BP5293-50 +5V, U501 OPA1652, Y1601 ASFL1-12.288MHZ-EC-T

Commit message: AudioV2: スロットコネクタを A2 どおり北 ANA / 南 PWR に直した
回路はそのまま。PCB の仮置きで逆になっていた娘 J_ANA/J_PWR と
親スロットの上下を揃え、AMP_SEL 本線は北の J_ANA へ出す。

Co-authored-by: m_arino <indare@users.noreply.github.com>
Parts:
- moved J_PWR103 181.9 mm to (290.0, 127.5)
- moved J_PWR102 163.7 mm to (170.0, 127.5)
- moved J_ANA103 157.0 mm to (290.0, 40.0)
- moved J_ANA102 145.2 mm to (170.0, 40.0)
- moved J_PWR101 113.0 mm to (50.0, 127.5)
- moved J_ANA301 90.0 mm to (360.0, 140.0), turned to 0 degrees
- moved J_PWR301 84.9 mm to (400.0, 227.5), turned to 0 degrees
- moved U_IO301 80.7 mm to (382.0, 219.5)
- moved J_ANA101 43.0 mm to (50.0, 40.0)
Routing:
- net /A_GND: track 15.3 -> 98.4 mm
- net /AMP_SEL_L: track 13.7 -> 67.8 mm
- net /I2C_SCL: track 52.7 -> 0.00 mm
- net /I2C_SDA: track 51.3 -> 0.00 mm, vias 1 -> 0
- net /AMP_SEL_R: track 13.7 -> 64.7 mm
- net /3V3: track 53.3 -> 48.9 mm
