File: AudioV2/AudioV2Case.kicad_pcb (KiCad board)
At the start: 2 copper layers, 110 x 110 mm, 257 parts, among them J1601 AUDIO, J1602 V_IN, J1603 15_V_IN, J201 +15/A_GND/-15 out, J202 PD module in (1=GND 2=+12V), Q401 BSS138, Q402 BSS138, SW1601 DEST sense (3PDT 3rd pole, sa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, SW402 PWR SW, SW501 DEST L (PHONE/MUTE/LINE), SW502 DEST R (PHONE/MUTE/LINE), U1601 OPA1656, U1602 OPA1656, U1603 LT1763-3.3, U1605 TPS3307-33, U1606 LT1763-5, U1607 BP5293-50, U1608 OPA1656, U1609 XC8107AC20MR-G, U1610 MCP23017 (UI 0x22), U1611 OPA1656, U201 REC20K-2415DZ, U202 L7809CV +9V, U311 TMUX7612, U312 TMUX7612, U402 PT2314E, U403 BP5293-50 +5V, U501 OPA1652, Y1601 ASFL1-12.288MHZ-EC-T

Commit message: ch1
Parts:
- R610: moved to B.Cu
- moved C311 36.4 mm to (345.2, 219.5)
- moved C313 31.5 mm to (377.0, 202.0)
- moved R607 16.1 mm to (370.5, 168.5), turned to 180 degrees
- moved C605 15.6 mm to (372.0, 176.9), turned to 90 degrees
- moved R603 12.2 mm to (348.0, 177.5)
- moved C312 12.1 mm to (345.0, 214.8)
- moved R609 11.0 mm to (385.0, 172.5), turned to 0 degrees
- moved C601 9.85 mm to (348.0, 167.5)
- moved R601 9.74 mm to (354.5, 163.0)
- moved R610 8.43 mm to (376.2, 167.8)
- moved R612 7.59 mm to (376.1, 161.8)
- moved R602 7.49 mm to (356.0, 159.3)
- moved R604 7.49 mm to (359.7, 160.4)
- moved AMP601 7.49 mm to (364.4, 157.8)
- moved R608 7.49 mm to (380.1, 161.8)
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Routing:
- net /AMP_SEL_L: track 11.3 -> 110.8 mm, vias 1 -> 2
- net /AMP_SEL_R: track 12.1 -> 101.8 mm
- net /-15V: track 168.2 -> 197.2 mm
- net /+15V: track 147.0 -> 175.9 mm
- net /AmpBankSwitch/CH1_OUT_L: track 11.6 -> 33.5 mm, vias 1 -> 0
- net Net-(AMP601B-+): track 27.8 -> 6.49 mm
- net Net-(AMP601A-+): track 30.2 -> 17.3 mm
- net Net-(C601-Pad1): track 0.00 -> 10.8 mm
- net /AmpBankSwitch/SEL_CH1: track 51.6 -> 60.1 mm
- net /AmpBankSwitch/CH1_OUT_R: track 15.0 -> 23.5 mm
- net Net-(AMP601-Pad1): track 0.00 -> 8.41 mm
- net Net-(AMP601-Pad7): track 0.00 -> 8.07 mm
- net Net-(AMP601A--): track 0.00 -> 7.60 mm
- net Net-(AMP601B--): track 0.00 -> 7.15 mm
- net Net-(C604-Pad2): track 0.07 -> 4.14 mm
