File: AudioV2/AudioV2Case.kicad_pcb (KiCad board)
At the start: 2 copper layers, 110 x 110 mm, 257 parts, among them J1601 AUDIO, J1602 V_IN, J1603 15_V_IN, J201 +15/A_GND/-15 out, J202 PD module in (1=GND 2=+12V), Q401 BSS138, Q402 BSS138, SW1601 DEST sense (3PDT 3rd pole, sa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, SW402 PWR SW, SW501 DEST L (PHONE/MUTE/LINE), SW502 DEST R (PHONE/MUTE/LINE), U1601 OPA1656, U1602 OPA1656, U1603 LT1763-3.3, U1605 TPS3307-33, U1606 LT1763-5, U1607 BP5293-50, U1608 OPA1656, U1609 XC8107AC20MR-G, U1610 MCP23017 (UI 0x22), U1611 OPA1656, U201 REC20K-2415DZ, U202 L7809CV +9V, U311 TMUX7612, U312 TMUX7612, U402 PT2314E, U403 BP5293-50 +5V, U501 OPA1652, Y1601 ASFL1-12.288MHZ-EC-T

Commit message: AudioV2: 娘 CH1–4 配線を固め、親ラフと PCB 配線スキルを足す
偶数 DIP 0°／南辺 L=R 並びに合わせた TMUX_MAP と AmpBankSwitch、娘 PCB の配置配線、親外形＋再グリッド、メーカー資料スキルと査読メモをまとめる。

Co-authored-by: Cursor <cursoragent@cursor.com>
Parts:
- C311, C312, C313, C708, C709, C809, C908, C909, R704, R707, R801, R803, R804, R808, R809, R810, R812, R904, R907: moved to B.Cu
- C601, C604, C701, C704, C801, C804, C901, C904: footprint C_Rect_L7.2mm_W7.2mm_P5.00mm_FKS2_FKP2_MKS2_MKP2 -> Capacitor_THT:C_Rect_L7.2mm_W7.2mm_P5.00mm_FKS2_FKP2_MKS2_MKP2
- C602, C605, C702, C705, C802, C805, C902, C905: footprint C_Rect_L7.2mm_W4.5mm_P5.00mm_FKS2_FKP2_MKS2_MKP2 -> Capacitor_THT:C_Rect_L7.2mm_W4.5mm_P5.00mm_FKS2_FKP2_MKS2_MKP2
- R607: moved to F.Cu
- moved R807 156.7 mm to (443.8, 168.5), turned to 90 degrees
- moved R812 150.9 mm to (431.6, 166.2), turned to 90 degrees
- moved R808 150.8 mm to (435.6, 166.2), turned to 90 degrees
- moved C805 150.7 mm to (443.8, 177.8), turned to 90 degrees
- moved R810 147.4 mm to (431.7, 171.9), turned to -90 degrees
- moved C804 145.5 mm to (435.5, 177.7), turned to 90 degrees
- moved R809 141.4 mm to (428.2, 176.7), turned to 180 degrees
- moved C808 137.9 mm to (432.3, 162.3)
- moved R806 130.6 mm to (415.5, 163.4), turned to -90 degrees
- moved R804 128.2 mm to (414.1, 163.4), turned to 180 degrees
- moved C801 123.6 mm to (411.5, 172.8), turned to -90 degrees
- moved R802 123.5 mm to (411.5, 163.3), turned to -90 degrees
- moved R907 122.3 mm to (442.2, 208.7), turned to 180 degrees
- moved R803 121.0 mm to (413.0, 181.8)
- moved C905 120.7 mm to (443.8, 200.6), turned to -90 degrees
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Connections:
- U311 pad 10: /AMP_SEL_R -> /AMP_SEL_L
- U311 pad 11: /AmpBankSwitch/CH2_OUT_R -> /AmpBankSwitch/CH2_OUT_L
- U311 pad 14: /AmpBankSwitch/CH2_OUT_L -> /AmpBankSwitch/CH2_OUT_R
- U311 pad 15: /AMP_SEL_L -> /AMP_SEL_R
- U312 pad 10: /AMP_SEL_R -> /AMP_SEL_L
- U312 pad 11: /AmpBankSwitch/CH4_OUT_R -> /AmpBankSwitch/CH4_OUT_L
- U312 pad 14: /AmpBankSwitch/CH4_OUT_L -> /AmpBankSwitch/CH4_OUT_R
- U312 pad 15: /AMP_SEL_L -> /AMP_SEL_R
Routing:
- net /TONE_L: track 0.00 -> 177.1 mm, vias 0 -> 1
- net /TONE_R: track 0.00 -> 172.5 mm
- net /-15V: track 197.2 -> 351.0 mm
- net /AMP_SEL_L: track 110.8 -> 237.0 mm, vias 2 -> 7
- net /AMP_SEL_R: track 101.8 -> 220.2 mm, vias 2 -> 5
- net /AmpBankSwitch/SEL_CH4: track 7.24 -> 121.0 mm, vias 0 -> 4
- net /AmpBankSwitch/SEL_CH3: track 7.88 -> 102.1 mm, vias 0 -> 7
- net /+15V: track 175.9 -> 267.7 mm, vias 3 -> 4
- net Net-(AMP701B-+): track 103.8 -> 23.2 mm
- net Net-(AMP701A-+): track 99.7 -> 26.4 mm
- net /AmpBankSwitch/SEL_CH2: track 15.3 -> 72.7 mm, vias 0 -> 3
- net Net-(AMP901A-+): track 0.00 -> 26.4 mm
- net /AmpBankSwitch/CH3_OUT_L: track 0.00 -> 24.0 mm
- net Net-(AMP901B-+): track 0.00 -> 23.2 mm
- net Net-(AMP801A-+): track 0.00 -> 22.7 mm
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Other:
- board size 110 x 110 mm -> 450 x 450 mm
