File: AudioV2/AudioV2Case.kicad_pcb (KiCad board)
At the start: 2 copper layers, 450 x 450 mm, 257 parts, among them J1601 AUDIO, J1602 V_IN, J1603 15_V_IN, J201 +15/A_GND/-15 out, J202 PD module in (1=GND 2=+12V), Q401 BSS138, Q402 BSS138, SW1601 DEST sense (3PDT 3rd pole, sa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, SW402 PWR SW, SW501 DEST L (PHONE/MUTE/LINE), SW502 DEST R (PHONE/MUTE/LINE), U1601 OPA1656, U1602 OPA1656, U1603 LT1763-3.3, U1605 TPS3307-33, U1606 LT1763-5, U1607 BP5293-50, U1608 OPA1656, U1609 XC8107AC20MR-G, U1610 MCP23017 (UI 0x22), U1611 OPA1656, U201 REC20K-2415DZ, U202 L7809CV +9V, U311 TMUX7612, U312 TMUX7612, U402 PT2314E, U403 BP5293-50 +5V, U501 OPA1652, Y1601 ASFL1-12.288MHZ-EC-T

Commit message: re asighn pin
Parts:
- removed C_IO301: 100nF, Capacitor_SMD:C_1206_3216Metric_Pad1.33x1.80mm_HandSolder
- removed U_IO301: MCP23017, Package_DIP:DIP-28_W7.62mm
- added C_IO101: 100nF, Capacitor_SMD:C_1206_3216Metric_Pad1.33x1.80mm_HandSolder, F.Cu at (333.3, 114.2)
- added U_IO101: MCP23017 (SW SEL 0x23), Package_DIP:DIP-28_W7.62mm, F.Cu at (321.1, 114.6)
- J_PWR101, J_PWR102, J_PWR103: footprint Connector_PinSocket_2.54mm:PinSocket_2x06_P2.54mm_Vertical -> Connector_PinSocket_2.54mm:PinSocket_2x08_P2.54mm_Vertical
- J_PWR301: footprint Connector_PinHeader_2.54mm:PinHeader_2x06_P2.54mm_Vertical -> Connector_PinHeader_2.54mm:PinHeader_2x08_P2.54mm_Vertical
- moved R701 138.7 mm to (483.8, 197.7)
- moved H303 138.2 mm to (483.2, 136.1)
- moved R901 135.0 mm to (535.5, 198.2)
- moved R601 134.3 mm to (477.7, 150.9), turned to 90 degrees
- moved C602 132.4 mm to (475.0, 146.8)
- moved R801 130.6 mm to (529.4, 151.3), turned to 90 degrees
- moved C802 129.4 mm to (526.1, 142.4), turned to -90 degrees
- moved C702 128.3 mm to (474.6, 196.2), turned to 0 degrees
- moved C902 128.2 mm to (529.9, 201.4), turned to 90 degrees
- moved J_ANA301 125.7 mm to (515.0, 214.5)
- moved R702 125.7 mm to (479.4, 190.9)
- moved AMP601 125.7 mm to (488.8, 144.3)
- moved AMP701 125.7 mm to (488.4, 191.1)
- moved C311 125.7 mm to (499.5, 178.0)
- moved C312 125.7 mm to (498.9, 163.2)
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Connections:
- J_PWR301 pad 10: /3V3 -> unconnected-(J_PWR301-Pin_10-Pad10)
- J_PWR301 pad 11: /D_GND -> unconnected-(J_PWR301-Pin_11-Pad11)
- J_PWR301 pad 12: /D_GND -> unconnected-(J_PWR301-Pin_12-Pad12)
- J_PWR301 pad 7: /I2C_SDA -> unconnected-(J_PWR301-Pin_7-Pad7)
- J_PWR301 pad 8: /D_GND -> unconnected-(J_PWR301-Pin_8-Pad8)
- J_PWR301 pad 9: /I2C_SCL -> unconnected-(J_PWR301-Pin_9-Pad9)
- U311 pad 1: /AmpBankSwitch/SEL_CH1 -> /SLOT1_SEL_CH1
- U311 pad 16: /AmpBankSwitch/SEL_CH2 -> /SLOT1_SEL_CH2
- U311 pad 8: /AmpBankSwitch/SEL_CH1 -> /SLOT1_SEL_CH1
- U311 pad 9: /AmpBankSwitch/SEL_CH2 -> /SLOT1_SEL_CH2
- U312 pad 1: /AmpBankSwitch/SEL_CH3 -> /SLOT1_SEL_CH3
- U312 pad 16: /AmpBankSwitch/SEL_CH4 -> /SLOT1_SEL_CH4
- U312 pad 8: /AmpBankSwitch/SEL_CH3 -> /SLOT1_SEL_CH3
- U312 pad 9: /AmpBankSwitch/SEL_CH4 -> /SLOT1_SEL_CH4
Routing:
- net /AmpBankSwitch/SEL_CH4: track 121.0 -> 0.00 mm, vias 4 -> 0
- net /SLOT1_SEL_CH4: track 0.00 -> 108.5 mm, vias 0 -> 4
- net /AmpBankSwitch/SEL_CH3: track 102.1 -> 0.00 mm, vias 7 -> 0
- net /SLOT1_SEL_CH3: track 0.00 -> 99.4 mm, vias 0 -> 7
- net /SLOT1_SEL_CH2: track 0.00 -> 72.7 mm, vias 0 -> 3
- net /AmpBankSwitch/SEL_CH2: track 72.7 -> 0.00 mm, vias 3 -> 0
- net /SLOT1_SEL_CH1: track 0.00 -> 55.8 mm, vias 0 -> 2
- net /AmpBankSwitch/SEL_CH1: track 55.8 -> 0.00 mm, vias 2 -> 0
- net unconnected-(J_PWR301-Pin_7-Pad7): track 0.00 -> 45.3 mm
- net /I2C_SDA: track 45.3 -> 0.00 mm
- net unconnected-(J_PWR301-Pin_9-Pad9): track 0.00 -> 39.7 mm
- net /I2C_SCL: track 39.7 -> 0.00 mm
- net unconnected-(J_PWR301-Pin_10-Pad10): track 0.00 -> 37.5 mm
- net /3V3: track 47.8 -> 10.3 mm
- net /AMP_SEL_L: track 237.0 -> 212.1 mm, vias 7 -> 8
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Other:
- board size 450 x 450 mm -> 569.4 x 450 mm
