File: AudioV2/AmpBankSwitch.kicad_sch (KiCad schematic)
At the start: 16 parts, among them U311 TMUX7612, U312 TMUX7612

Commit message: AudioV2: TMUX 案C（90°+ピン再割当）と Amp 入力カップリング再配置
PCB 配置に合わせて S↔D・ch 組・SEL 結びを変え、U311 周りを引き出し配線。
C602/C605/C702/C705 はソケット脇へ移し、3層化は保留。

Co-authored-by: Cursor <cursoragent@cursor.com>
Connections:
- net AMP_SEL_L: now also U311.14 (S2), U311.6 (S4), U312.14 (S2), U312.6 (S4); no longer U311.10 (D3), U311.2 (D1), U312.10 (D3), U312.2 (D1)
- net AMP_SEL_R: now also U311.11 (S3), U311.3 (S1), U312.11 (S3), U312.3 (S1); no longer U311.15 (D2), U311.7 (D4), U312.15 (D2), U312.7 (D4)
- net CH1_OUT_L: now also U311.15 (D2); no longer U311.3 (S1)
- net CH1_OUT_R: now also U311.10 (D3); no longer U311.14 (S2)
- net CH2_OUT_L: now also U311.7 (D4); no longer U311.11 (S3)
- net CH2_OUT_R: now also U311.2 (D1); no longer U311.6 (S4)
- net CH3_OUT_L: now also U312.15 (D2); no longer U312.3 (S1)
- net CH3_OUT_R: now also U312.10 (D3); no longer U312.14 (S2)
- net CH4_OUT_L: now also U312.7 (D4); no longer U312.11 (S3)
- net CH4_OUT_R: now also U312.2 (D1); no longer U312.6 (S4)
- net SEL_CH1: now also U311.9 (SEL3); no longer U311.1 (SEL1)
- net SEL_CH2: now also U311.1 (SEL1); no longer U311.9 (SEL3)
- net SEL_CH3: now also U312.9 (SEL3); no longer U312.1 (SEL1)
- net SEL_CH4: now also U312.1 (SEL1); no longer U312.9 (SEL3)

Commit message: AudioV2: TMUX を 270°（ピン1側=CH1）にし、AmpChannel のスイッチ用デカップを外す
S=各ch出力・D=AMP_SEL に戻し、CH1 配線途中の PCB も取り込む。C607/C610 は D22 の残りなのでシートから削除した。

Co-authored-by: Cursor <cursoragent@cursor.com>
Connections:
- net AMP_SEL_L: now also U311.15 (D2), U311.7 (D4), U312.15 (D2), U312.7 (D4); no longer U311.14 (S2), U311.6 (S4), U312.14 (S2), U312.6 (S4)
- net AMP_SEL_R: now also U311.10 (D3), U311.2 (D1), U312.10 (D3), U312.2 (D1); no longer U311.11 (S3), U311.3 (S1), U312.11 (S3), U312.3 (S1)
- net CH1_OUT_L: now also U311.6 (S4); no longer U311.15 (D2)
- net CH1_OUT_R: now also U311.3 (S1); no longer U311.10 (D3)
- net CH2_OUT_L: now also U311.14 (S2); no longer U311.7 (D4)
- net CH2_OUT_R: now also U311.11 (S3); no longer U311.2 (D1)
- net CH3_OUT_L: now also U312.6 (S4); no longer U312.15 (D2)
- net CH3_OUT_R: now also U312.3 (S1); no longer U312.10 (D3)
- net CH4_OUT_L: now also U312.14 (S2); no longer U312.7 (D4)
- net CH4_OUT_R: now also U312.11 (S3); no longer U312.2 (D1)
- net SEL_CH1: now also U311.1 (SEL1), U311.8 (SEL4); no longer U311.16 (SEL2), U311.9 (SEL3)
- net SEL_CH2: now also U311.16 (SEL2), U311.9 (SEL3); no longer U311.1 (SEL1), U311.8 (SEL4)
- net SEL_CH3: now also U312.1 (SEL1), U312.8 (SEL4); no longer U312.16 (SEL2), U312.9 (SEL3)
- net SEL_CH4: now also U312.16 (SEL2), U312.9 (SEL3); no longer U312.1 (SEL1), U312.8 (SEL4)
Changed lines of the file:
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@@
 	)
 	(label "SEL_CH4"
-		(at 200.66 279.4 180)
+		(at 200.66 294.64 180)
 		(effects
 			(font
@@
 	)
 	(label "SEL_CH2"
-		(at 137.16 302.26 180)
+		(at 137.16 287.02 180)
 		(effects
 			(font
@@
 	)
 	(label "CH3_OUT_L"
+		(at 200.66 304.8 180)
+		(effects
+			(font
+				(size 1.27 1.27)
+			)
+			(justify right bottom)
+		)
+	)
+	(label "SEL_CH1"
+		(at 137.16 279.4 180)
+		(effects
+			(font
+				(size 1.27 1.27)
+			)
+			(justify right bottom)
+		)
+	)
+	(label "AMP_SEL_L"
+		(at 162.56 303.53 0)
+		(effects
+			(font
+				(size 1.27 1.27)
+			)
+			(justify left bottom)
+		)
+	)
+	(label "A_GND"
+		(at 38.1 157.48 180)
+		(effects
+			(font
+				(size 1.27 1.27)
+			)
+			(justify right bottom)
+		)
+	)
+	(label "AMP_SEL_L"
 		(at 226.06 288.29 0)
 		(effects
@@
 		)
 	)
-	(label "SEL_CH1"
-		(at 137.16 294.64 180)
-		(effects
-			(font
-				(size 1.27 1.27)
-			)
-			(justify right bottom)
-		)
-	)
-	(label "AMP_SEL_L"
-		(at 137.16 289.56 180)
-		(effects
-			(font
-				(size 1.27 1.27)
-			)
-			(justify right bottom)
-		)
-	)
-	(label "A_GND"
-		(at 38.1 157.48 180)
-		(effects
-			(font
-				(size 1.27 1.27)
-			)
-			(justify right bottom)
-		)
-	)
-	(label "AMP_SEL_L"
-		(at 200.66 304.8 180)
-		(effects
-			(font
-				(size 1.27 1.27)
-			)
-			(justify right bottom)
-		)
-	)
 	(label "AMP_SEL_R"
-		(at 200.66 297.18 180)
-		(effects
-			(font
-				(size 1.27 1.27)
-			)
-			(justify right bottom)
+		(at 226.06 280.67 0)
+		(effects
+			(font
+				(size 1.27 1.27)
+			)
+			(justify left bottom)
 		)
 	)
@@
 	)
 	(label "CH4_OUT_R"
-		(at 226.06 280.67 0)
-		(effects
-			(font
-				(size 1.27 1.27)
-			)
-			(justify left bottom)
+		(at 200.66 297.18 180)
+		(effects
+			(font
+				(size 1.27 1.27)
+			)
+			(justify right bottom)
 		)
 	)
@@
 	)
 	(label "AMP_SEL_R"
-		(at 200.66 281.94 180)
-		(effects
-			(font
-				(size 1.27 1.27)
-			)
-			(justify right bottom)
+		(at 226.06 295.91 0)
+		(effects
+			(font
+				(size 1.27 1.27)
+			)
+			(justify left bottom)
 		)
 	)
@@
 	)
 	(label "CH3_OUT_R"
-		(at 226.06 295.91 0)
-		(effects
-			(font
-				(size 1.27 1.27)
-			)
-			(justify left bottom)
+		(at 200.66 281.94 180)
+		(effects
+			(font
+				(size 1.27 1.27)
+			)
+			(justify right bottom)
 		)
 	)
 	(label "SEL_CH3"
-		(at 200.66 294.64 180)
+		(at 200.66 279.4 180)
 		(effects
 			(font
@@
 	)
 	(label "CH4_OUT_L"
-		(at 226.06 303.53 0)
-		(effects
-			(font
-				(size 1.27 1.27)
-			)
-			(justify left bottom)
+		(at 200.66 289.56 180)
+		(effects
+			(font
+				(size 1.27 1.27)
+			)
+			(justify right bottom)
 		)
 	)
@@
 	)
 	(label "CH1_OUT_R"
-		(at 162.56 295.91 0)
-		(effects
-			(font
-				(size 1.27 1.27)
-			)
-			(justify left bottom)
+		(at 137.16 281.94 180)
+		(effects
+			(font
+				(size 1.27 1.27)
+			)
+			(justify right bottom)
 		)
 	)
@@
 	)
 	(label "AMP_SEL_R"
-		(at 137.16 297.18 180)
-		(effects
-			(font
-				(size 1.27 1.27)
-			)
-			(justify right bottom)
+		(at 162.56 280.67 0)
+		(effects
+			(font
+				(size 1.27 1.27)
+			)
+			(justify left bottom)
 		)
 	)
@@
 	)
 	(label "AMP_SEL_L"
-		(at 200.66 289.56 180)
-		(effects
-			(font
-				(size 1.27 1.27)
-			)
-			(justify right bottom)
+		(at 226.06 303.53 0)
+		(effects
+			(font
+				(size 1.27 1.27)
+			)
+			(justify left bottom)
 		)
 	)
@@
 	)
 	(label "CH2_OUT_R"
-		(at 162.56 280.67 0)
-		(effects
-			(font
-				(size 1.27 1.27)
-			)
-			(justify left bottom)
+		(at 137.16 297.18 180)
+		(effects
+			(font
+				(size 1.27 1.27)
+			)
+			(justify right bottom)
 		)
 	)
@@
 	)
 	(label "AMP_SEL_L"
-		(at 137.16 304.8 180)
-		(effects
-			(font
-				(size 1.27 1.27)
-			)
-			(justify right bottom)
+		(at 162.56 288.29 0)
+		(effects
+			(font
+				(size 1.27 1.27)
+			)
+			(justify left bottom)
 		)
 	)
@@
 	)
 	(label "SEL_CH2"
-		(at 137.16 279.4 180)
+		(at 137.16 294.64 180)
 		(effects
 			(font
@@
 	)
 	(label "SEL_CH1"
-		(at 137.16 287.02 180)
+		(at 137.16 302.26 180)
 		(effects
 			(font
@@
 	)
 	(label "SEL_CH3"
-		(at 200.66 287.02 180)
+		(at 200.66 302.26 180)
 		(effects
 			(font
@@
 	)
 	(label "AMP_SEL_R"
-		(at 137.16 281.94 180)
-		(effects
-			(font
-				(size 1.27 1.27)
-			)
-			(justify right bottom)
+		(at 162.56 295.91 0)
+		(effects
+			(font
+				(size 1.27 1.27)
+			)
+			(justify left bottom)
 		)
 	)
@@
 	)
 	(label "CH1_OUT_L"
-		(at 162.56 288.29 0)
-		(effects
-			(font
-				(size 1.27 1.27)
-			)
-			(justify left bottom)
+		(at 137.16 304.8 180)
+		(effects
+			(font
+				(size 1.27 1.27)
+			)
+			(justify right bottom)
 		)
 	)
 	(label "CH2_OUT_L"
-		(at 162.56 303.53 0)
-		(effects
-			(font
-				(size 1.27 1.27)
-			)
-			(justify left bottom)
+		(at 137.16 289.56 180)
+		(effects
+			(font
+				(size 1.27 1.27)
+			)
+			(justify right bottom)
 		)
 	)
@@
 	)
 	(label "SEL_CH4"
-		(at 200.66 302.26 180)
-		(effects
-			(font
+		(at 200.66 287.02 180)
+		(effects
+			(font

Commit message: AudioV2: 娘 CH1–4 配線を固め、親ラフと PCB 配線スキルを足す
偶数 DIP 0°／南辺 L=R 並びに合わせた TMUX_MAP と AmpBankSwitch、娘 PCB の配置配線、親外形＋再グリッド、メーカー資料スキルと査読メモをまとめる。

Co-authored-by: Cursor <cursoragent@cursor.com>
Connections:
- net AMP_SEL_L: now also U311.10 (D3), U312.10 (D3); no longer U311.15 (D2), U312.15 (D2)
- net AMP_SEL_R: now also U311.15 (D2), U312.15 (D2); no longer U311.10 (D3), U312.10 (D3)
- net CH2_OUT_L: now also U311.11 (S3); no longer U311.14 (S2)
- net CH2_OUT_R: now also U311.14 (S2); no longer U311.11 (S3)
- net CH4_OUT_L: now also U312.11 (S3); no longer U312.14 (S2)
- net CH4_OUT_R: now also U312.14 (S2); no longer U312.11 (S3)
