File: AudioV2/FrontPanel.kicad_sch (KiCad schematic)
At the start: 31 parts, among them SW402 Cosland 2MS1 PWR, SW501 Cosland 2MD1 DEST, U1609 XC8107AC20MR-G, U1610 MCP23017 (UI 0x22)

Commit message: AudioV2: FrontPanel の 12V を電源 XH に分離し FP PCB を配線
音声 XH から PD を外し J_PNL_P* へ移す。A/D/PD の GND 同居を避け、
FrontPanel 側のデジ・音声・電源配線とベタ分けを進めた。

Co-authored-by: Cursor <cursoragent@cursor.com>
Parts:
- removed LCDDisplay1601: WAVESHARE-29318, Connector_JST:JST_XH_B15B-XH-A_1x15_P2.50mm_Vertical, symbol MeasurementADC_Extras:WAVESHARE-29318
- added J_PNL_P1611: FrontPanel 12V raw, Connector_JST:JST_XH_B3B-XH-A_1x03_P2.50mm_Vertical, symbol Connector_Generic:Conn_01x03
- added J_PNL_P1612: FrontPanel 12V switched, Connector_JST:JST_XH_B3B-XH-A_1x03_P2.50mm_Vertical, symbol Connector_Generic:Conn_01x03
- J_LCD1601: renamed from LCDDisplay1601_1; value FrontPanel analog B (even) -> LCD cable A (XH8)
- J_LCD1602: renamed from LCDDisplay1601_2; value FrontPanel analog B (even) -> LCD cable B (XH8)
- J_PNL_A1602_2: value FrontPanel analog B (even) -> LCD cable A (XH8)
Connections:
- net LED_DEST1: now also U1610.3 (GPB2); no longer U1610.2 (GPB1)
- net LED_DEST2: now also U1610.2 (GPB1); no longer U1610.3 (GPB2)
- net PD_12V: now also J_PNL_P1611.1 (Pin_1); no longer J_PNL_A1602_1.5 (Pin_5)
- net PD_12V_SW: now also J_PNL_P1612.1 (Pin_1); no longer J_PNL_A1602_2.5 (Pin_5)
- net PD_GND: now also J_PNL_P1611.2 (Pin_2), J_PNL_P1612.2 (Pin_2); no longer J_PNL_A1602_1.6 (Pin_6)
- no-connect marks 23 -> 28
Other:
- moved on the sheet: D403, R401, SW402, SW501A, SW501B
