File: AudioV2/AmpBankRelay.kicad_sch (KiCad schematic)
At the start: 17 parts, among them K301 AZ850P2-5, K302 AZ850P2-5, K303 AZ850P2-5, K304 AZ850P2-5, U321 TBD62083APG

Commit message: re asighn pin
Parts:
- removed H311: M3, MountingHole:MountingHole_3.2mm_M3, symbol Mechanical:MountingHole
- removed J_PWR302: SLOT PWR/CTRL (D18), Connector_PinHeader_2.54mm:PinHeader_2x06_P2.54mm_Vertical, symbol Connector_Generic:Conn_02x06_Odd_Even
- added C322: 100nF, Capacitor_SMD:C_1206_3216Metric_Pad1.33x1.80mm_HandSolder, symbol Device:C
- added J_PWR302: SLOT PWR/CTRL (D18), Connector_PinHeader_2.54mm:PinHeader_2x08_P2.54mm_Vertical, symbol Connector_Generic:Conn_02x08_Odd_Even
- H311: renamed from C322; value 100nF -> M3; footprint Capacitor_SMD:C_1206_3216Metric_Pad1.33x1.80mm_HandSolder -> MountingHole:MountingHole_3.2mm_M3; symbol Device:C -> Mechanical:MountingHole
Connections:
- net +15V: now also J_PWR302.1 (Pin_1)
- net +5V_COIL: now also C322.1, J_PWR302.5 (Pin_5); no longer H311.1
- net -15V: now also J_PWR302.3 (Pin_3)
- net 3V3: now also J_PWR302.10 (Pin_10)
- net ADDR0: now also J_PWR302.11 (Pin_11)
- net ADDR1: now also J_PWR302.12 (Pin_12)
- net A_GND: now also J_PWR302.2 (Pin_2), J_PWR302.4 (Pin_4)
- net D_GND: now also J_PWR302.8 (Pin_8)
- net GND_COIL: now also C322.2, J_PWR302.6 (Pin_6); no longer H311.2
- net I2C_SCL: now also J_PWR302.9 (Pin_9)
- net I2C_SDA: now also J_PWR302.7 (Pin_7)
- no-connect marks 20 -> 24

Commit message: AudioV2: AmpBank 番地をジャンパ 6 段へ（縦積み向け）
スロット側 ADDR（D21）をやめ、娘の A0/A1/A2 ソルダージャンパで
0x20/21/23/24/25/26 を選択。スイッチ版にも MCP を載せ SEL を現地駆動し、
親 U_IO101 を廃止。コネクタ pin11–16 は N.C.。

Co-authored-by: m_arino <indare@users.noreply.github.com>
Parts:
- added JP_ADDR_A0302: ADDR A0, Jumper:SolderJumper-3_P1.3mm_Bridged12_Pad1.0x1.5mm_NumberLabels, symbol Jumper:SolderJumper_3_Bridged12
- added JP_ADDR_A1302: ADDR A1, Jumper:SolderJumper-3_P1.3mm_Bridged12_Pad1.0x1.5mm_NumberLabels, symbol Jumper:SolderJumper_3_Bridged12
- added JP_ADDR_A2302: ADDR A2, Jumper:SolderJumper-3_P1.3mm_Bridged12_Pad1.0x1.5mm_NumberLabels, symbol Jumper:SolderJumper_3_Bridged12
Connections:
- net 3V3: now also JP_ADDR_A0302.3 (B), JP_ADDR_A1302.3 (B), JP_ADDR_A2302.3 (B)
- net D_GND: now also JP_ADDR_A0302.1 (A), JP_ADDR_A1302.1 (A), JP_ADDR_A2302.1 (A); no longer U_IO302.17 (A2)
- net ADDR0: no longer names the net of J_PWR302.11 (Pin_11)
- net ADDR0: no longer U_IO302.15 (A0)
- net ADDR1: no longer names the net of J_PWR302.12 (Pin_12)
- net ADDR1: no longer U_IO302.16 (A1)
- new net ADDR_A0: JP_ADDR_A0302.2 (C), U_IO302.15 (A0)
- new net ADDR_A1: JP_ADDR_A1302.2 (C), U_IO302.16 (A1)
- new net ADDR_A2: JP_ADDR_A2302.2 (C), U_IO302.17 (A2)
- no-connect marks 24 -> 26
Other:
- note added: "I2C ADDR jumpers (skip UI 0x22): tier1 000→0x20 tier2 001→0x21 tier3 011→0x23 tier4 100→0x24 tier5 101→0x25 tier6 110→0x26 (A2 A1 A0; Bridged12=GND=0, bridge 2-3 for 1)"
