File: AudioV2/AmpBankRelay.kicad_sch (KiCad schematic)
At the start: 20 parts, among them K301 AZ850P2-5, K302 AZ850P2-5, K303 AZ850P2-5, K304 AZ850P2-5, U321 TBD62083APG

Commit message: relay rework
Connections:
- net AMP_SEL_L: now also K301.7, K302.7, K303.7, K304.7; no longer K301.4, K302.4, K303.4, K304.4
- net AMP_SEL_R: now also K301.4, K302.4, K303.4, K304.4; no longer K301.7, K302.7, K303.7, K304.7
Changed lines of the file:
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@@
-		)
-	)
-	(label "AMP_SEL_R"
-		(at 208.28 281.94 0)
-		(effects
-			(font
-				(size 1.27 1.27)
-			)
-			(justify left bottom)
 		)
 	)
@@
 		)
 	)
+	(label "AMP_SEL_R"
+		(at 152.4 281.94 90)
+		(effects
+			(font
+				(size 1.27 1.27)
+			)
+			(justify left bottom)
+		)
+	)
 	(label "D_GND"
 		(at 200.66 238.76 0)
@@
 		)
 	)
+	(label "AMP_SEL_L"
+		(at 254 281.94 90)
+		(effects
+			(font
+				(size 1.27 1.27)
+			)
+			(justify left bottom)
+		)
+	)
 	(label "CH3_SETC"
 		(at 233.68 297.18 180)
@@
 		)
 	)
-	(label "AMP_SEL_R"
-		(at 299.72 281.94 0)
-		(effects
-			(font
-				(size 1.27 1.27)
-			)
-			(justify left bottom)
-		)
-	)
 	(label "ADDR_A2"
 		(at 210.82 194.31 0)
@@
 		)
 	)
-	(label "AMP_SEL_R"
-		(at 162.56 281.94 0)
-		(effects
-			(font
-				(size 1.27 1.27)
-			)
-			(justify left bottom)
-		)
-	)
 	(label "CH4_OUT_R"
 		(at 114.3 142.24 0)
@@
 		)
 	)
-	(label "AMP_SEL_L"
-		(at 289.56 281.94 0)
-		(effects
-			(font
-				(size 1.27 1.27)
-			)
-			(justify left bottom)
-		)
-	)
 	(label "CH1_RSTC"
 		(at 259.08 179.07 0)
@@
 		)
 	)
-	(label "AMP_SEL_L"
-		(at 243.84 281.94 0)
-		(effects
-			(font
-				(size 1.27 1.27)
-			)
-			(justify left bottom)
-		)
-	)
 	(label "-15V"
 		(at 38.1 152.4 180)
@@
 	)
 	(label "AMP_SEL_L"
+		(at 208.28 281.94 90)
+		(effects
+			(font
+				(size 1.27 1.27)
+			)
+			(justify left bottom)
+		)
+	)
+	(label "AMP_SEL_L"
 		(at 335.28 63.5 180)
 		(effects
@@
 		)
 	)
+	(label "AMP_SEL_R"
+		(at 289.56 281.94 90)
+		(effects
+			(font
+				(size 1.27 1.27)
+			)
+			(justify left bottom)
+		)
+	)
 	(label "-15V"
 		(at 38.1 81.28 180)
@@
 		)
 	)
+	(label "AMP_SEL_R"
+		(at 198.12 281.94 90)
+		(effects
+			(font
+				(size 1.27 1.27)
+			)
+			(justify left bottom)
+		)
+	)
 	(label "CH2_OUT_R"
 		(at 114.3 71.12 0)
@@
 		)
 	)
-	(label "AMP_SEL_L"
-		(at 152.4 281.94 0)
-		(effects
-			(font
-				(size 1.27 1.27)
-			)
-			(justify left bottom)
-		)
-	)
 	(label "-15V"
 		(at 38.1 116.84 180)
@@
 		)
 	)
-	(label "AMP_SEL_R"
-		(at 254 281.94 0)
-		(effects
-			(font
-				(size 1.27 1.27)
-			)
-			(justify left bottom)
-		)
-	)
 	(label "+15V"
 		(at 38.1 147.32 180)
@@
 		)
 	)
+	(label "AMP_SEL_L"
+		(at 162.56 281.94 90)
+		(effects
+			(font
+				(size 1.27 1.27)
+			)
+			(justify left bottom)
+		)
+	)
+	(label "AMP_SEL_L"
+		(at 299.72 281.94 90)
+		(effects
+			(font
+				(size 1.27 1.27)
+			)
+			(justify left bottom)
+		)
+	)
 	(label "GND_COIL"
 		(at 419.1 147.32 0)
@@
 		)
 	)
+	(label "AMP_SEL_R"
+		(at 243.84 281.94 90)
+		(effects
+			(font
+				(size 1.27 1.27)
+			)
+			(justify left bottom)
+		)
+	)
 	(label "-15V"
 		(at 335.28 111.76 180)
@@
 		(effects
 			(font
-				(size 1.27 1.27)
-			)
-			(justify left bottom)
-		)
-	)
-	(label "AMP_SEL_L"
-		(at 198.12 281.94 0)
-		(effects
-			(font
