File: AudioV2/AmpBankRelay.kicad_sch (KiCad schematic)
At the start: 20 parts, among them K301 AZ850P2-5, K302 AZ850P2-5, K303 AZ850P2-5, K304 AZ850P2-5, U321 TBD62083APG

Commit message: AudioV2: 娘基板（Switch/Relay）の AMP_SEL 配線・デカップを音質優先で追い込む (#42)
- Switch: AMP_SEL を1ホップずつ B.Cu へ、TMUX の南北 D を本体下で直結、TMUX に 1 µF（0603）追加・100 nF を足元の裏へ、J_ANA301 の L/R 交差を 90° に
- Relay: リレー列↔ドライバ間の帯を組み直し（コイル線・L バス・ドライバ 100 nF・+5V_COIL 近道）、AMP_SEL の L/R を別の通り道に分離（2 mm 以内並走 L↔R 18 → 0 mm）
- 共通: MCP23017 の 100 nF を 0603 で VDD/VSS の足の真上へ
- ルートを手編集所有に切替、ERC 残骸の片付け（59 → 5）、期待値と PARTS.md を実測に合わせる

DRC 新規違反 0・未接続不変・schematic parity 0。ERC 5。部品 355。

Co-Authored-By: Claude Opus 5.5 <noreply@anthropic.com>
Claude-Session: https://claude.ai/code/session_01NpwAm89hZpJTCZphnQ6odp
Parts:
- C322, C_IO302: footprint Capacitor_SMD:C_1206_3216Metric_Pad1.33x1.80mm_HandSolder -> Capacitor_SMD:C_0603_1608Metric_Pad1.08x0.95mm_HandSolder
Changed lines of the file:
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@@
 			)
 		)
-		(property "Footprint" "Capacitor_SMD:C_1206_3216Metric_Pad1.33x1.80mm_HandSolder"
+		(property "Footprint" "Capacitor_SMD:C_0603_1608Metric_Pad1.08x0.95mm_HandSolder"
 			(at 0 0 0)
 			(hide yes)
@@
 			)
 		)
-		(property "Footprint" "Capacitor_SMD:C_1206_3216Metric_Pad1.33x1.80mm_HandSolder"
+		(property "Footprint" "Capacitor_SMD:C_0603_1608Metric_Pad1.08x0.95mm_HandSolder"
 			(at 0 0 0)
 			(hide yes)
