File: AudioV2/legacy/OutputStage.kicad_sch (KiCad schematic)
At the start: 7 parts, among them SW501 DEST L (PHONE/MUTE/LINE), SW502 DEST R (PHONE/MUTE/LINE)

Commit message: AudioV2: パネル部品6個をヘッダのフットプリントにした（16 -> 10）
PARTS.md がヘッダ構成まで既に指定していた。それに従っただけで、新しい判断は
入れていない。

  PARTS.md:5    RV / SW_DEST / ENC / PWR SW は パネル実装。基板はヘッダ＋リード
  PARTS.md:173  RV は基板 6P ヘッダ（Device:R_Potentiometer_Dual ピン番号のまま）
  PARTS.md:141  SW_DEST は 現物端子 -> 基板ヘッダ（音声 2x4 + センス 1x3）

  RV501/502     PinHeader_1x06   シンボルのピン 1-6 がそのままヘッダのピン
  SW501/502     PinHeader_1x04   PARTS.md §2.1 の SW601-1..4 / SW602-1..4 に対応
  SW1601        PinHeader_1x04   同じ並び。pin2(MUTE) は基板側で未使用
  SW402         PinHeader_1x02   SPST

ポットの品種（Alps RK27 か RK097 か Alpha RD901 か）は決めていない。
PARTS.md が「RK097 でも回路は同一」「A50k デュアルならピン互換で可」と
書いており、電気的な要件は A カーブ・50k・2連だけ。**ヘッダなので基板側は
品種に依存しない**。入手性と性能で選ぶ調達判断として残す（ユーザー判断 2026-09-07）。

⚠ PARTS.md の「音声 2x4」は 2行4列ではなく「4ピンを2組」と読んだ。同 §2.1 の
ピン対応表が SW601-1..4 / SW602-1..4 と別々に並べており、シンボルも2つに
分かれているため。2行4列の1個を意図していたなら要修正。

副次的に、Cursor 査読の「DEST の 3PDT が自動 BOM 上で現物3個に見える」も解ける。
基板に載るのはヘッダ3個（実際に3個要る）で、スイッチ本体はパネル部品として
基板 BOM に出ないのが正しい形。

なお PARTS.md §2.1 のピン対応表は SW601-3 をコモン（AMP_SEL_L）としており、
今日 SW1601 で直した割り当て（pin3=コモン）と一致していた。

検証:
  未設定      16 -> 10（残りは D403・F201/202/203・J201/202・J_HP501・
              J_LINE501・J_RAIL501・U202。すべて調達判断待ち）
  netlist     部品 370 / 重複 0（変化なし）
  erc         17 件（変化なし）
  check_sexpr 13 ファイル / 問題 0
  roundtrip   6/6 OK
  再生成      2回目でバイト一致

Co-Authored-By: Claude Opus 5 <noreply@anthropic.com>
Claude-Session: https://claude.ai/code/session_01VCArLcCGbMGgxvWJ5HFJiY
Parts:
- RV501, RV502: footprint (none) -> Connector_PinHeader_2.54mm:PinHeader_1x06_P2.54mm_Vertical
- SW501, SW502: footprint (none) -> Connector_PinHeader_2.54mm:PinHeader_1x04_P2.54mm_Vertical
Changed lines of the file:
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@@
 			)
 		)
-		(property "Footprint" ""
+		(property "Footprint" "Connector_PinHeader_2.54mm:PinHeader_1x06_P2.54mm_Vertical"
 			(at 0 0 0)
 			(hide yes)
@@
 			)
 		)
-		(property "Footprint" ""
+		(property "Footprint" "Connector_PinHeader_2.54mm:PinHeader_1x04_P2.54mm_Vertical"
 			(at -26.67 1.27 0)
 			(hide yes)
@@
 			)
 		)
-		(property "Footprint" ""
+		(property "Footprint" "Connector_PinHeader_2.54mm:PinHeader_1x06_P2.54mm_Vertical"
 			(at 0 8.89 0)
 			(hide yes)
@@
 			)
 		)
-		(property "Footprint" ""
+		(property "Footprint" "Connector_PinHeader_2.54mm:PinHeader_1x04_P2.54mm_Vertical"
 			(at -26.67 2.54 0)
 			(hide yes)

Commit message: AudioV2: 端子台5個を Phoenix MKDS-1,5 にした（10 -> 5）
ユーザー判断（2026-09-07）。PARTS.md:211 が板間の端子台に Phoenix MKDS-1,5
系を指定しており、計測基板の J1601(2P) / J1603(3P) に既に同じ footprint が
入っている。その前例に合わせた。

  J201       1x03  +15/-15/A_GND out
  J202       1x02  PD module in
  J_HP501    1x02  to Audio HP Buffer
  J_LINE501  1x02  LINE OUT
  J_RAIL501  1x03  RAIL IN

J_HP501 / J_LINE501 / J_RAIL501 は元から Connector:Screw_Terminal_01xNN
シンボルなので端子台が自然。J201 / J202 は Conn_01xNN_Pin（汎用ピン）だが、
板間の電源なので同じ系に揃えた。

残り5個は性質が違うので手を付けていない:
  D403             12V パネル LED。直列抵抗の有無が未決（DECISIONS の既知項目）
  F201             T1.6A slow 5x20。ヒューズホルダの品種
  F202/F203        PPTC。MPN 未確定（直流抵抗とディレーティングが決まらない）
  U202             L7809CV TO-220。実装向き（垂直/水平・放熱器）が機構判断

検証:
  未設定      10 -> 5
  netlist     部品 370 / 重複 0（変化なし）
  erc         17 件（変化なし）
  check_sexpr 13 ファイル / 問題 0
  roundtrip   6/6 OK
  再生成      2回目でバイト一致

Co-Authored-By: Claude Opus 5 <noreply@anthropic.com>
Claude-Session: https://claude.ai/code/session_01VCArLcCGbMGgxvWJ5HFJiY
Parts:
- J_HP501, J_LINE501: footprint (none) -> TerminalBlock_Phoenix:TerminalBlock_Phoenix_MKDS-1,5-2-5.08_1x02_P5.08mm_Horizontal
- J_RAIL501: footprint (none) -> TerminalBlock_Phoenix:TerminalBlock_Phoenix_MKDS-1,5-3-5.08_1x03_P5.08mm_Horizontal
Changed lines of the file:
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@@
 			)
 		)
-		(property "Footprint" ""
+		(property "Footprint" "TerminalBlock_Phoenix:TerminalBlock_Phoenix_MKDS-1,5-2-5.08_1x02_P5.08mm_Horizontal"
 			(at 8.89 3.81 0)
 			(hide yes)
@@
 			)
 		)
-		(property "Footprint" ""
+		(property "Footprint" "TerminalBlock_Phoenix:TerminalBlock_Phoenix_MKDS-1,5-2-5.08_1x02_P5.08mm_Horizontal"
 			(at 8.89 0 0)
 			(hide yes)
@@
 			)
 		)
-		(property "Footprint" ""
+		(property "Footprint" "TerminalBlock_Phoenix:TerminalBlock_Phoenix_MKDS-1,5-3-5.08_1x03_P5.08mm_Horizontal"
 			(at -13.97 -62.23 0)
 			(hide yes)
