File: AudioV2/legacy/ControlPanelAnalog.kicad_sch (KiCad schematic)
At the start: 20 parts, among them SW402 PWR SW, U402 PT2314E, U403 BP5293-50 +5V

Commit message: AudioV2: HP バッファを移設し、PT2314E の DGND を A_GND へ寄せて I²C にレベルシフタを入れた
未実装のまま「確定」に留まっていた2件を回路図に入れ、注釈・BOM の腐りを直した。

- HP バッファ移設（2026-09-06 確定）: legacy/OutputStage に U501（DIP-8 ソケット、
  標準実装 OPA1652）+ R501/R502 10Ω + C501/C502 470µF NP + R503/R504 100k +
  C503-C506。RV501 ワイパー側のラベルを PHONE_BUF_L/R に改名し、PHONE_L/R は
  バッファ出力になった。J_HP501 / J_LINE501 を 01x03（L / A_GND / R）にして帰路を入れた
- DGND→A_GND ＋ I²C 境界（2026-09-07 確定）: U402.25 を A_GND へ。境界は BSS138 ×2 の
  双方向レベルシフタ（Q401/Q402、PT 側 R412/R413 10k → VCC_TONE）。P82B96 を使わない
  理由（Sx 側 VOL 0.8–1.0 V が PT2314E VIL 1.0 V / RP2350 VIL 0.8 V を食い切る）は
  DECISIONS の実装節に一次資料の数字で置いた
- MeasureControl の注釈: 上書きしてしまった Pico ピン配置ノートを復元（GP9=NC）、
  R1605 / 3.3k の旧記述を消し、U1611 Description を実値（約30k・−115.5 dB）に直した
- NT1603 を in_bom no に揃え、PARTS.md は 385（ネットリスト 389 − NetTie 4）
- DECISIONS: PPTC「戻さない」の理由を言い直し（1・2行目は判定材料にならない、
  3行目の条件は X7R 割れに限らない、U201 の OCP は 230 % max @ nom. VIN 24 V）、
  ヘッドルーム −0.4 dBFS は typ 基準で余裕の確定ではないと追記（7.5k 案を併記）、
  U1611 の 47Ω 省略に CL 100 pF の根拠を足した

検証: check_sexpr 0 / roundtrip 全 OK / 再生成は冪等（バイト一致）/ ERC 11 件（型・件数とも
変化なし）/ ネットリスト 389 個・重複 0・フットプリント未設定 0 / 母板で座標の偶然一致なし

Co-Authored-By: Claude Fable 5.1 <noreply@anthropic.com>
Claude-Session: https://claude.ai/code/session_01VCArLcCGbMGgxvWJ5HFJiY
Parts:
- added Q401, Q402: BSS138, Package_TO_SOT_SMD:SOT-23, symbol Transistor_FET:BSS138
- added R412, R413: 10k, Resistor_SMD:R_1206_3216Metric_Pad1.30x1.75mm_HandSolder, symbol Device:R
Connections:
- net A_GND: now also U402.25 (DGND)
- net D_GND: no longer U402.25 (DGND)
- net I2C_SCL: now also Q402.2 (S); no longer U402.27 (CLK)
- net I2C_SDA: now also Q401.2 (S); no longer U402.26 (DATA)
- net VCC_TONE: now also R412.1, R413.1
- new net 3V3: Q401.1 (G), Q402.1 (G)
- new net I2C_SCL_9V: Q402.3 (D), R413.2, U402.27 (CLK)
- new net I2C_SDA_9V: Q401.3 (D), R412.2, U402.26 (DATA)
Other:
- note added: "I²C レベルシフタ（2026-09-08）: Pico 側 3V3 バス I2C_SDA/SCL（プルアップは MeasureControl の R1653/R1654 4.7k）↔ PT2314E 側 9V バス I2C_SDA_9V/SCL_9V（R412/R413 10k → VCC_TONE）。BSS138 ゲート=3V3。同時に U402 pin25 DGND をチップの足元で A_GND へ（旧 D_GND）。片方だけでは成立しない（DECISIONS「DGND はチップの足元で A_GND へ」）。"
